File: ram.kicad_sch (KiCad schematic)
At the start: 2 parts, among them U28 74LS138

Commit message: more pcb routing, implementing learnings from the prototype board
Parts:
- removed C40: 0.1uF 20% Ceramic, Capacitor_SMD:C_0805_2012Metric, symbol Device:C
- removed U28: 74LS138, Package_DIP:DIP-16_W7.62mm_Socket, symbol 74xx:74LS138
Connections:
- no-connect marks 4 -> 0
Other:
- note removed: "A17..A18: 00 = 0x00000 -> 0x20000 01 = 0x20000 -> 0x40000 10 = 0x40000 -> 0x60000 11 = 0x60000 -> 0x80000"
