File: 8088_databus.kicad_sch (KiCad schematic)
At the start: 2 parts, among them U6 74HC245

Commit message: bringing over learnings/improvements from prototype board
Parts:
- added RN3: 10k, Resistor_THT:R_Array_SIP9, symbol Device:R_Network08
Connections:
- net +5V: now also RN3.1 (common)
- net D0: now also RN3.2 (R1)
- net D1: now also RN3.3 (R2)
- net D2: now also RN3.4 (R3)
- net D3: now also RN3.5 (R4)
- net D4: now also RN3.6 (R5)
- net D5: now also RN3.7 (R6)
- net D6: now also RN3.8 (R7)
- net D7: now also RN3.9 (R8)

Commit message: pcb is fully routed, working on power capacitor tweaks, some ROM testing
Parts:
- renumbered C6 to C28, RN3 to RN4, U6 to U15
Changed lines of the file:
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@@
 		(dnp no)
 		(fields_autoplaced yes)
-		(property "Reference" "RN3"
+		(property "Reference" "RN4"
 			(at 237.49 100.5839 0)
 			(effects
@@
 			(project "sbc_8088"
 				(path "/5e468d94-0319-44d1-a77f-2adc451eed13/e0da2df2-77fd-4360-b71c-7e802397f430"
-					(reference "RN3")
+					(reference "RN4")
 					(unit 1)
 				)
@@
 		(dnp no)
 		(fields_autoplaced yes)
-		(property "Reference" "C6"
+		(property "Reference" "C28"
 			(at 148.59 71.12 90)
 			(effects
@@
 			(project "sbc_8088"
 				(path "/5e468d94-0319-44d1-a77f-2adc451eed13/e0da2df2-77fd-4360-b71c-7e802397f430"
-					(reference "C6")
+					(reference "C28")
 					(unit 1)
 				)
@@
 		(dnp no)
 		(fields_autoplaced yes)
-		(property "Reference" "U6"
+		(property "Reference" "U15"
 			(at 141.8941 81.28 0)
 			(effects
@@
 			(project "sbc_8088"
 				(path "/5e468d94-0319-44d1-a77f-2adc451eed13/e0da2df2-77fd-4360-b71c-7e802397f430"
-					(reference "U6")
-					(unit 1)
-				)
+					(reference "U15")
+					(unit 1)
+				)

Commit message: added ATtiny for SMC, added PC speaker
Parts:
- renumbered C28 to C33, U15 to U16
Changed lines of the file:
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@@
 		(dnp no)
 		(fields_autoplaced yes)
-		(property "Reference" "C28"
+		(property "Reference" "C33"
 			(at 148.59 71.12 90)
 			(effects
@@
 			(project "sbc_8088"
 				(path "/5e468d94-0319-44d1-a77f-2adc451eed13/e0da2df2-77fd-4360-b71c-7e802397f430"
-					(reference "C28")
+					(reference "C33")
 					(unit 1)
 				)
@@
 		(dnp no)
 		(fields_autoplaced yes)
-		(property "Reference" "U15"
+		(property "Reference" "U16"
 			(at 141.8941 81.28 0)
 			(effects
@@
 			(project "sbc_8088"
 				(path "/5e468d94-0319-44d1-a77f-2adc451eed13/e0da2df2-77fd-4360-b71c-7e802397f430"
-					(reference "U15")
+					(reference "U16")
 					(unit 1)
 				)
