File: biosrom.kicad_sch (KiCad schematic)
At the start: 2 parts, among them U7 W27C512 BIOS ROM

Commit message: pcb is fully routed, working on power capacitor tweaks, some ROM testing
Parts:
- renumbered C7 to C53, U7 to U34
Changed lines of the file:
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@@
 		(dnp no)
 		(fields_autoplaced yes)
-		(property "Reference" "C7"
+		(property "Reference" "C53"
 			(at 163.8363 52.07 90)
 			(effects
@@
 			(project "sbc_8088"
 				(path "/5e468d94-0319-44d1-a77f-2adc451eed13/7c2a67e3-de61-4656-9956-d7abc8589104"
-					(reference "C7")
+					(reference "C53")
 					(unit 1)
 				)
@@
 		(dnp no)
 		(fields_autoplaced yes)
-		(property "Reference" "U7"
+		(property "Reference" "U34"
 			(at 158.4041 64.77 0)
 			(effects
@@
 			(project "sbc_8088"
 				(path "/5e468d94-0319-44d1-a77f-2adc451eed13/7c2a67e3-de61-4656-9956-d7abc8589104"
-					(reference "U7")
+					(reference "U34")
 					(unit 1)
 				)

Commit message: added ATtiny for SMC, added PC speaker
Parts:
- renumbered C53 to C58, U34 to U38
Changed lines of the file:
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@@
 		(dnp no)
 		(fields_autoplaced yes)
-		(property "Reference" "C53"
+		(property "Reference" "C58"
 			(at 163.8363 52.07 90)
 			(effects
@@
 			(project "sbc_8088"
 				(path "/5e468d94-0319-44d1-a77f-2adc451eed13/7c2a67e3-de61-4656-9956-d7abc8589104"
-					(reference "C53")
+					(reference "C58")
 					(unit 1)
 				)
@@
 		(dnp no)
 		(fields_autoplaced yes)
-		(property "Reference" "U34"
+		(property "Reference" "U38"
 			(at 158.4041 64.77 0)
 			(effects
@@
 			(project "sbc_8088"
 				(path "/5e468d94-0319-44d1-a77f-2adc451eed13/7c2a67e3-de61-4656-9956-d7abc8589104"
-					(reference "U34")
+					(reference "U38")
 					(unit 1)
 				)
