File: biosrom.kicad_sch (KiCad schematic)
At the start: 2 parts, among them U38 W27C512 BIOS ROM

Commit message: fixes, prep for final production run
Parts:
- C58: LCSC Part # (none) -> C1853649
- U38: LCSC Part # (none) -> C72121
Changed lines of the file:
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@@
 			)
 		)
-		(property "Description" ""
+		(property "Description" "LCSC #C1853649"
+			(at 163.83 58.42 0)
+			(effects
+				(font
+					(size 1.27 1.27)
+				)
+				(hide yes)
+			)
+		)
+		(property "Height" ""
+			(at 163.83 58.42 0)
+			(effects
+				(font
+					(size 1.27 1.27)
+				)
+				(hide yes)
+			)
+		)
+		(property "Manufacturer_Name" ""
+			(at 163.83 58.42 0)
+			(effects
+				(font
+					(size 1.27 1.27)
+				)
+				(hide yes)
+			)
+		)
+		(property "Manufacturer_Part_Number" ""
+			(at 163.83 58.42 0)
+			(effects
+				(font
+					(size 1.27 1.27)
+				)
+				(hide yes)
+			)
+		)
+		(property "Mouser Part Number" ""
+			(at 163.83 58.42 0)
+			(effects
+				(font
+					(size 1.27 1.27)
+				)
+				(hide yes)
+			)
+		)
+		(property "Mouser Price/Stock" ""
+			(at 163.83 58.42 0)
+			(effects
+				(font
+					(size 1.27 1.27)
+				)
+				(hide yes)
+			)
+		)
+		(property "LCSC Part #" "C1853649"
 			(at 163.83 58.42 0)
 			(effects
@@
 			)
 		)
-		(property "Description" ""
-			(at 156.21 88.9 0)
-			(effects
+		(property "Description" "LCSC #C72121 "
+			(at 156.21 88.9 0)
+			(effects
+				(font
+					(size 1.27 1.27)
+				)
+				(hide yes)
+			)
+		)
+		(property "Height" ""
+			(at 156.21 88.9 0)
+			(effects
+				(font
+					(size 1.27 1.27)
+				)
+				(hide yes)
+			)
+		)
+		(property "Manufacturer_Name" ""
+			(at 156.21 88.9 0)
+			(effects
+				(font
+					(size 1.27 1.27)
+				)
+				(hide yes)
+			)
+		)
+		(property "Manufacturer_Part_Number" ""
+			(at 156.21 88.9 0)
+			(effects
+				(font
+					(size 1.27 1.27)
+				)
+				(hide yes)
+			)
+		)
+		(property "Mouser Part Number" ""
+			(at 156.21 88.9 0)
+			(effects
+				(font
+					(size 1.27 1.27)
+				)
+				(hide yes)
+			)
+		)
+		(property "Mouser Price/Stock" ""
+			(at 156.21 88.9 0)
+			(effects
+				(font
+					(size 1.27 1.27)
+				)
+				(hide yes)
+			)
+		)
+		(property "LCSC Part #" "C72121 "
+			(at 156.21 88.9 0)
+			(effects

Commit message: m88: use round-hole socket for BIOS ROM by default
Parts:
- U38: LCSC Part # C72121 -> C2874016
Changed lines of the file:
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@@
 			)
 		)
-		(property "Description" "LCSC #C72121"
+		(property "Description" "Use LCSC #C2874016 for round hole, LCSC #C72121 for standard DIP"
 			(at 156.21 88.9 0)
 			(effects
@@
 			)
 		)
-		(property "LCSC Part #" "C72121 "
+		(property "LCSC Part #" "C2874016"
 			(at 156.21 88.9 0)
 			(effects

Commit message: motherboard tweaks for manufacturing run, i2c card tweaks for manufacturing run, de9 -> stemma adapter idea for the i2c card
Parts:
- C58: LCSC Part # C1853649 -> C49678
Changed lines of the file:
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@@
 			)
 		)
-		(property "Description" "LCSC #C1853649"
+		(property "Description" "LCSC #C49678"
 			(at 163.83 58.42 0)
 			(effects
@@
 			)
 		)
-		(property "LCSC Part #" "C1853649"
+		(property "LCSC Part #" "C49678"
 			(at 163.83 58.42 0)
 			(effects
