File: isa.kicad_sch (KiCad schematic)
At the start: 9 parts, among them J4 Bus_ISA_8bit, J5 Bus_ISA_8bit, J6 Bus_ISA_8bit

Commit message: more pcb routing
Connections:
- removed net IRQ2: J4.4 (IRQ2), J5.4 (IRQ2), J6.4 (IRQ2)
- no-connect marks 6 -> 9
Other:
- note added: "IRQ2 is reserved by PIC cascade ISA BUS may not use it."
- moved on the sheet: C33, C35, C37, C38, J4, J5, J6

Commit message: pcb is fully routed, working on power capacitor tweaks, some ROM testing
Parts:
- removed C33, C34, C35, C36, C37, C38: 10 uF 10% 10V Tantalum Kemet T landing (3528-12 E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, Capacitor_Tantalum_SMD:CP_EIA-3528-12_Kemet-T, symbol Device:C_Polarized_Small_US
- added C10, C11, C27, C29, C7, C8: 10UF 16V 20%, Capacitor_SMD:CP_Elec_5x4.5, symbol Device:C_Polarized_Small_US
- added R1, R3: 10k, Resistor_SMD:R_0805_2012Metric, symbol Device:R_US
- renumbered J6 to J3, J5 to J4, J4 to J5
Connections:
- net +5V: now also C10.1, C11.1, C27.1, C29.1, C7.1, C8.1, R1.1, R3.1
- net GND: now also C10.2, C11.2, C27.2, C29.2, C7.2, C8.2
- net IO_CH_CHK: now also R1.2
- net IO_READY: now also R3.2

Commit message: added ATtiny for SMC, added PC speaker
Parts:
- renumbered C27 to C32, C29 to C34, J3 to J4, J4 to J5, J5 to J6
Changed lines of the file:
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@@
 		(dnp no)
 		(fields_autoplaced yes)
-		(property "Reference" "C29"
+		(property "Reference" "C34"
 			(at 104.14 174.8282 0)
 			(effects
@@
 			(project "sbc_8088"
 				(path "/5e468d94-0319-44d1-a77f-2adc451eed13/7e9ec34b-a562-42ca-aed5-ced2fee0dbf0"
-					(reference "C29")
+					(reference "C34")
 					(unit 1)
 				)
@@
 		(dnp no)
 		(fields_autoplaced yes)
-		(property "Reference" "J5"
+		(property "Reference" "J6"
 			(at 69.85 61.595 0)
 			(effects
@@
 			(project "sbc_8088"
 				(path "/5e468d94-0319-44d1-a77f-2adc451eed13/7e9ec34b-a562-42ca-aed5-ced2fee0dbf0"
-					(reference "J5")
+					(reference "J6")
 					(unit 1)
 				)
@@
 		(dnp no)
 		(fields_autoplaced yes)
-		(property "Reference" "J4"
+		(property "Reference" "J5"
 			(at 157.48 61.595 0)
 			(effects
@@
 			(project "sbc_8088"
 				(path "/5e468d94-0319-44d1-a77f-2adc451eed13/7e9ec34b-a562-42ca-aed5-ced2fee0dbf0"
-					(reference "J4")
+					(reference "J5")
 					(unit 1)
 				)
@@
 		(dnp no)
 		(fields_autoplaced yes)
-		(property "Reference" "C27"
+		(property "Reference" "C32"
 			(at 66.04 174.8282 0)
 			(effects
@@
 			(project "sbc_8088"
 				(path "/5e468d94-0319-44d1-a77f-2adc451eed13/7e9ec34b-a562-42ca-aed5-ced2fee0dbf0"
-					(reference "C27")
+					(reference "C32")
 					(unit 1)
 				)
@@
 		(dnp no)
 		(fields_autoplaced yes)
-		(property "Reference" "J3"
+		(property "Reference" "J4"
 			(at 243.84 61.595 0)
 			(effects
@@
 			(project "sbc_8088"
 				(path "/5e468d94-0319-44d1-a77f-2adc451eed13/7e9ec34b-a562-42ca-aed5-ced2fee0dbf0"
-					(reference "J3")
-					(unit 1)
-				)
+					(reference "J4")
+					(unit 1)
+				)
