File: isa.kicad_sch (KiCad schematic)
At the start: 11 parts, among them J4 Bus_ISA_8bit, J5 Bus_ISA_8bit, J6 Bus_ISA_8bit

Commit message: fix KBC/PPI CS# schematic bugs, add ISA expansion header for adding more cards
Parts:
- added J11: Conn_02x31_Top_Bottom, Connector_PinSocket_2.54mm:PinSocket_2x31_P2.54mm_Horizontal, symbol Connector_Generic:Conn_02x31_Odd_Even
Connections:
- net +12V: now also J11.17 (Pin_17)
- net +5V: now also J11.5 (Pin_5), J11.57 (Pin_57)
- net -12V: now also J11.13 (Pin_13)
- net A0: now also J11.62 (Pin_62)
- net A1: now also J11.60 (Pin_60)
- net A10: now also J11.42 (Pin_42)
- net A11: now also J11.40 (Pin_40)
- net A12: now also J11.38 (Pin_38)
- net A13: now also J11.36 (Pin_36)
- net A14: now also J11.34 (Pin_34)
- net A15: now also J11.32 (Pin_32)
- net A16: now also J11.30 (Pin_30)
- net A17: now also J11.28 (Pin_28)
- net A18: now also J11.26 (Pin_26)
- net A19: now also J11.24 (Pin_24)
- net A2: now also J11.58 (Pin_58)
- net A3: now also J11.56 (Pin_56)
- net A4: now also J11.54 (Pin_54)
- net A5: now also J11.52 (Pin_52)
- net A6: now also J11.50 (Pin_50)
- net A7: now also J11.48 (Pin_48)
- net A8: now also J11.46 (Pin_46)
- net A9: now also J11.44 (Pin_44)
- net AEN: now also J11.22 (Pin_22)
- net ALE: now also J11.55 (Pin_55)
- net CLK: now also J11.39 (Pin_39)
- net D0: now also J11.18 (Pin_18)
- net D1: now also J11.16 (Pin_16)
- net D2: now also J11.14 (Pin_14)
- net D3: now also J11.12 (Pin_12)
- net D4: now also J11.10 (Pin_10)
- net D5: now also J11.8 (Pin_8)
- net D6: now also J11.6 (Pin_6)
- net D7: now also J11.4 (Pin_4)
- net DRQ1: now also J11.35 (Pin_35)
- net DRQ2: now also J11.11 (Pin_11)
- net DRQ3: now also J11.31 (Pin_31)
- net GND: now also J11.1 (Pin_1), J11.19 (Pin_19), J11.61 (Pin_61)
- net IO_CH_CHK: now also J11.2 (Pin_2)
- net IO_READY: now also J11.20 (Pin_20)
- net IRQ3: now also J11.49 (Pin_49)
- net IRQ4: now also J11.47 (Pin_47)
- net IRQ5: now also J11.45 (Pin_45)
- net IRQ6: now also J11.43 (Pin_43)
- net IRQ7: now also J11.41 (Pin_41)
- net OSC: now also J11.59 (Pin_59)
- net RESET: now also J11.3 (Pin_3)
- net TC: now also J11.53 (Pin_53)
- net ~{DACK}0: now also J11.37 (Pin_37)
- net ~{DACK}1: now also J11.33 (Pin_33)
- net ~{DACK}2: now also J11.51 (Pin_51)
- net ~{DACK}3: now also J11.29 (Pin_29)
- net ~{IOR}: now also J11.27 (Pin_27)
- net ~{IOW}: now also J11.25 (Pin_25)
- net ~{MEMR}: now also J11.23 (Pin_23)
- net ~{MEMW}: now also J11.21 (Pin_21)
- no-connect marks 9 -> 12
Other:
- note added: "ISA Expansion connector For extending ISA bus beyond mainboard"

Commit message: fixes, prep for final production run
Parts:
- removed J11: Conn_02x31_Top_Bottom, Connector_PinSocket_2.54mm:PinSocket_2x31_P2.54mm_Horizontal, symbol Connector_Generic:Conn_02x31_Odd_Even
- removed R1, R3: 10k, Resistor_SMD:R_0805_2012Metric, symbol Device:R_US
- added C36, C41: 10UF 16V 20%, Capacitor_SMD:CP_Elec_5x4.5, symbol Device:C_Polarized_Small_US
- added J11: Bus_ISA_8bit, SamacSys_Parts:755308430_ISA, symbol Custom:Bus_ISA_8bit_Host
- added R50, R51, R52, R53, R54, R55, R56, R57, R58: 10k, Resistor_SMD:R_0805_2012Metric, symbol Device:R_US
- C10, C11, C32, C34, C7, C8: LCSC Part # (none) -> C20607181
- J4, J5, J6: LCSC Part # (none) -> C5173311
Connections:
- net +12V: now also J11.9 (+12V)
- net +5V: now also C36.1, C41.1, J11.29 (VCC), J11.3 (VCC), R50.2, R51.2, R52.2, R53.2
- net -12V: now also J11.7 (-12V)
- net A0: now also J11.62 (BA00)
- net A1: now also J11.61 (BA01)
- net A10: now also J11.52 (BA10)
- net A11: now also J11.51 (BA11)
- net A12: now also J11.50 (BA12)
- net A13: now also J11.49 (BA13)
- net A14: now also J11.48 (BA14)
- net A15: now also J11.47 (BA15)
- net A16: now also J11.46 (BA16)
- net A17: now also J11.45 (BA17)
- net A18: now also J11.44 (BA18)
- net A19: now also J11.43 (BA19)
- net A2: now also J11.60 (BA02)
- net A3: now also J11.59 (BA03)
- net A4: now also J11.58 (BA04)
- net A5: now also J11.57 (BA05)
- net A6: now also J11.56 (BA06)
- net A7: now also J11.55 (BA07)
- net A8: now also J11.54 (BA08)
- net A9: now also J11.53 (BA09)
- net AEN: now also J11.42 (AEN), R54.1
- net ALE: now also J11.28 (ALE)
- net CLK: now also J11.20 (CLK)
- net D0: now also J11.40 (DB0)
- net D1: now also J11.39 (DB1)
- net D2: now also J11.38 (DB2)
- net D3: now also J11.37 (DB3)
- net D4: now also J11.36 (DB4)
- net D5: now also J11.35 (DB5)
- net D6: now also J11.34 (DB6)
- net D7: now also J11.33 (DB7)
- net DRQ1: now also J11.18 (DRQ1), R56.1
- net DRQ2: now also J11.6 (DRQ2), R57.1
- net DRQ3: now also J11.16 (DRQ3), R58.1
- net GND: now also C36.2, C41.2, J11.1 (GND), J11.10 (GND), J11.31 (GND), R54.2, R55.2, R56.2, R57.2, R58.2
- net IO_CH_CHK: now also J11.32 (IO_CH_CHK)
- net IO_READY: now also J11.41 (IO_CH_READY)
- net IRQ3: now also J11.25 (IRQ3)
- net IRQ4: now also J11.24 (IRQ4)
- net IRQ5: now also J11.23 (IRQ5)
- net IRQ6: now also J11.22 (IRQ6)
- net IRQ7: now also J11.21 (IRQ7)
- net OSC: now also J11.30 (OSC)
- net RESET: now also J11.2 (RESET)
- net TC: now also J11.27 (TC), R55.1
- net ~{DACK}0: now also J11.19 (~{DACK0}), R52.1
- net ~{DACK}1: now also J11.17 (~{DACK1}), R51.1
- net ~{DACK}2: now also J11.26 (~{DACK2}), R53.1
- net ~{DACK}3: now also J11.15 (~{DACK3}), R50.1
- net ~{IOR}: now also J11.14 (~{IOR})
- net ~{IOW}: now also J11.13 (~{IOW})
- net ~{MEMR}: now also J11.12 (~{SMEMR})
- net ~{MEMW}: now also J11.11 (~{SMEMW})
Other:
- note added: "Don't allow DMA signals to float if DMAC not installed"
- note removed: "ISA Expansion connector For extending ISA bus beyond mainboard"

Commit message: part tweaks, BOM is pretty much finalized, use 0.5W resistors for bleeders
Parts:
- C10, C11, C32, C34, C36, C41, C7, C8: LCSC Part # C20607181 -> C72486
- J11, J4, J5, J6: value Bus_ISA_8bit -> 8-bit ISA Bus connector; LCSC Part # C5173311 -> C4874769; Manufacturer_Name (none) -> TE Connectivity; Manufacturer_Part_Number (none) -> 7-5530843-0
Changed lines of the file:
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@@
 			)
 		)
-		(property "Description" "LCSC #C20607181"
+		(property "Description" "LCSC #C72486"
 			(at 72.39 176.53 0)
 			(effects
@@
 			)
 		)
-		(property "LCSC Part #" "C20607181"
+		(property "LCSC Part #" "C72486"
 			(at 72.39 176.53 0)
 			(effects
@@
 			)
 		)
-		(property "Description" "LCSC #C20607181"
+		(property "Description" "LCSC #C72486"
 			(at 101.6 176.53 0)
 			(effects
@@
 			)
 		)
-		(property "LCSC Part #" "C20607181"
+		(property "LCSC Part #" "C72486"
 			(at 101.6 176.53 0)
 			(effects
@@
 			)
 		)
-		(property "Description" "LCSC #C20607181"
+		(property "Description" "LCSC #C72486"
 			(at 82.55 176.53 0)
 			(effects
@@
 			)
 		)
-		(property "LCSC Part #" "C20607181"
+		(property "LCSC Part #" "C72486"
 			(at 82.55 176.53 0)
 			(effects
@@
 			)
 		)
-		(property "Description" "LCSC #C20607181"
+		(property "Description" "LCSC #C72486"
 			(at 110.49 176.53 0)
 			(effects
@@
 			)
 		)
-		(property "LCSC Part #" "C20607181"
+		(property "LCSC Part #" "C72486"
 			(at 110.49 176.53 0)
 			(effects
@@
 			)
 		)
-		(property "Value" "Bus_ISA_8bit"
+		(property "Value" "8-bit ISA Bus connector"
 			(at 341.63 64.135 0)
 			(effects
@@
 			)
 		)
-		(property "Description" "LCSC #C5173311"
+		(property "Description" "LCSC #C4874769"
 			(at 341.63 106.68 0)
 			(effects
@@
 			)
 		)
-		(property "Manufacturer_Name" ""
+		(property "Manufacturer_Name" "TE Connectivity"
 			(at 341.63 106.68 0)
 			(effects
@@
 			)
 		)
-		(property "Manufacturer_Part_Number" ""
+		(property "Manufacturer_Part_Number" "7-5530843-0"
 			(at 341.63 106.68 0)
 			(effects
@@
 			)
 		)
-		(property "LCSC Part #" "C5173311"
+		(property "LCSC Part #" "C4874769"
 			(at 341.63 106.68 0)
 			(effects
@@
 			)
 		)
-		(property "Description" "LCSC #C20607181"
+		(property "Description" "LCSC #C72486"
 			(at 128.27 176.53 0)
 			(effects
@@
 			)
 		)
-		(property "LCSC Part #" "C20607181"
+		(property "LCSC Part #" "C72486"
 			(at 128.27 176.53 0)
 			(effects
@@
 			)
 		)
-		(property "Description" "LCSC #C20607181"
+		(property "Description" "LCSC #C72486"
 			(at 119.38 176.53 0)
 			(effects
@@
 			)
 		)
-		(property "LCSC Part #" "C20607181"
+		(property "LCSC Part #" "C72486"
 			(at 119.38 176.53 0)
 			(effects
@@
 			)
 		)
-		(property "Value" "Bus_ISA_8bit"
+		(property "Value" "8-bit ISA Bus connector"
 			(at 69.85 64.135 0)
 			(effects
@@
 			)
 		)
-		(property "Description" "LCSC #C5173311"
+		(property "Description" "LCSC #C4874769"
 			(at 69.85 106.68 0)
 			(effects
@@
 			)
 		)
-		(property "Manufacturer_Name" ""
+		(property "Manufacturer_Name" "TE Connectivity"
 			(at 69.85 106.68 0)
 			(effects
@@
 			)
 		)
-		(property "Manufacturer_Part_Number" ""
+		(property "Manufacturer_Part_Number" "7-5530843-0"
 			(at 69.85 106.68 0)
 			(effects
@@
 			)
 		)
-		(property "LCSC Part #" "C5173311"
+		(property "LCSC Part #" "C4874769"
 			(at 69.85 106.68 0)
 			(effects
@@
 			)
 		)
-		(property "Description" "LCSC #C20607181"
+		(property "Description" "LCSC #C72486"
 			(at 91.44 176.53 0)
 			(effects
@@
 			)
 		)
-		(property "LCSC Part #" "C20607181"
+		(property "LCSC Part #" "C72486"
 			(at 91.44 176.53 0)
 			(effects
@@
 			)
 		)
-		(property "Value" "Bus_ISA_8bit"
+		(property "Value" "8-bit ISA Bus connector"
 			(at 157.48 64.135 0)
 			(effects
@@
 			)
 		)
-		(property "Description" "LCSC #C5173311"
+		(property "Description" "LCSC #C4874769"
 			(at 157.48 106.68 0)
 			(effects
@@
 			)
 		)
-		(property "Manufacturer_Name" ""
+		(property "Manufacturer_Name" "TE Connectivity"
 			(at 157.48 106.68 0)
 			(effects
@@
 			)
 		)
-		(property "Manufacturer_Part_Number" ""
+		(property "Manufacturer_Part_Number" "7-5530843-0"
 			(at 157.48 106.68 0)
 			(effects
@@
 			)
 		)
-		(property "LCSC Part #" "C5173311"
+		(property "LCSC Part #" "C4874769"
 			(at 157.48 106.68 0)
 			(effects
@@
 			)
 		)
-		(property "Description" "LCSC #C20607181"
+		(property "Description" "LCSC #C72486"
 			(at 63.5 176.53 0)
 			(effects
@@
 			)
 		)
-		(property "LCSC Part #" "C20607181"
+		(property "LCSC Part #" "C72486"
 			(at 63.5 176.53 0)
 			(effects
@@
 			)
 		)
-		(property "Value" "Bus_ISA_8bit"
+		(property "Value" "8-bit ISA Bus connector"
 			(at 243.84 64.135 0)
 			(effects
@@
 			)
 		)
-		(property "Description" "LCSC #C5173311"
+		(property "Description" "LCSC #C4874769"
 			(at 243.84 106.68 0)
 			(effects
@@
 			)
 		)
-		(property "Manufacturer_Name" ""
+		(property "Manufacturer_Name" "TE Connectivity"
 			(at 243.84 106.68 0)
 			(effects
@@
 			)
 		)
-		(property "Manufacturer_Part_Number" ""
+		(property "Manufacturer_Part_Number" "7-5530843-0"
 			(at 243.84 106.68 0)
 			(effects
@@
 			)
 		)
-		(property "LCSC Part #" "C5173311"
+		(property "LCSC Part #" "C4874769"
 			(at 243.84 106.68 0)
 			(effects

Commit message: no more SMT for isa_i2c, tweak motherboard multiplex logic, handful of other tweaks
Parts:
- removed R50, R51, R54, R56, R57, R58: 10k, Resistor_SMD:R_0805_2012Metric, symbol Device:R_US
- added RN7, RN8: 10k, Resistor_THT:R_Array_SIP5, symbol Device:R_Network04
- R52: value 10k -> 22; LCSC Part # C84376 -> (none)
- R53: value 10k -> 27; LCSC Part # C84376 -> (none)
Connections:
- net +5V: now also RN7.1 (common); no longer R52.2, R53.2
- net AEN: now also RN8.2 (R1)
- net CLK: now also R53.1; no longer J11.20 (CLK), J4.20 (CLK), J5.20 (CLK), J6.20 (CLK)
- net DRQ1: now also RN8.3 (R2)
- net DRQ2: now also RN8.4 (R3)
- net DRQ3: now also RN8.5 (R4)
- net GND: now also RN8.1 (common)
- net OSC: now also R52.1; no longer J11.30 (OSC), J4.30 (OSC), J5.30 (OSC), J6.30 (OSC)
- net ~{DACK}0: now also RN7.4 (R3); no longer R52.1
- net ~{DACK}1: now also RN7.5 (R4)
- net ~{DACK}2: now also RN7.3 (R2); no longer R53.1
- net ~{DACK}3: now also RN7.2 (R1)
- net IRQ2: now reaches J11.4 (IRQ2)
- net IRQ2: now also J4.4 (IRQ2), J5.4 (IRQ2), J6.4 (IRQ2)
- new net 84OSC: J11.30 (OSC), J4.30 (OSC), J5.30 (OSC), J6.30 (OSC), R52.2
- new net SYSCLK: J11.20 (CLK), J4.20 (CLK), J5.20 (CLK), J6.20 (CLK), R53.2
- no-connect marks 12 -> 8
Other:
- note added: "CLK = Pin B20 = "SYSCLK""
- note added: "OSC = Pin B30 = "84OSC""
- note removed: "IRQ2 is reserved by PIC cascade ISA BUS may not use it."
- moved on the sheet: R55

Commit message: simplify m88 logic further, reduce ICs, reorient the POST display, use an oscillator for 14.31818 MHz, update isa-i2c bridge BOM
Parts:
- R52: LCSC Part # (none) -> C2933536
- R53: LCSC Part # (none) -> C2889599
Changed lines of the file:
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@@
 			)
 		)
-		(property "Description" ""
+		(property "Description" "LCSC #C2889599"
 			(at 104.14 24.13 0)
 			(effects
@@
 			)
 		)
-		(property "LCSC Part #" ""
+		(property "LCSC Part #" "C2889599"
 			(at 104.14 24.13 0)
 			(effects
@@
 			)
 		)
-		(property "Description" ""
+		(property "Description" "LCSC #C2933536"
 			(at 104.14 36.83 0)
 			(effects
@@
 			)
 		)
-		(property "LCSC Part #" ""
+		(property "LCSC Part #" "C2933536"
 			(at 104.14 36.83 0)
 			(effects

Commit message: motherboard tweaks for manufacturing run, i2c card tweaks for manufacturing run, de9 -> stemma adapter idea for the i2c card
Parts:
- R52: LCSC Part # C2933536 -> C17561
- R53: LCSC Part # C2889599 -> C17594
- R55: LCSC Part # C84376 -> C17414
- RN7, RN8: value 10k -> 10k (bussed)
Changed lines of the file:
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@@
 			)
 		)
-		(property "Description" "LCSC #C84376"
+		(property "Description" "LCSC #C17414"
 			(at 143.51 208.28 0)
 			(effects
@@
 			)
 		)
-		(property "LCSC Part #" "C84376 "
+		(property "LCSC Part #" "C17414"
 			(at 143.51 208.28 0)
 			(effects
@@
 			)
 		)
-		(property "Description" "LCSC #C2889599"
+		(property "Description" "LCSC #C17594"
 			(at 104.14 24.13 0)
 			(effects
@@
 			)
 		)
-		(property "LCSC Part #" "C2889599"
+		(property "LCSC Part #" "C17594"
 			(at 104.14 24.13 0)
 			(effects
@@
 			)
 		)
-		(property "Value" "10k"
+		(property "Value" "10k (bussed)"
 			(at 178.816 203.2 90)
 			(effects
@@
 			)
 		)
-		(property "Description" "LCSC #C2933536"
+		(property "Description" "LCSC #C17561"
 			(at 104.14 36.83 0)
 			(effects
@@
 			)
 		)
-		(property "LCSC Part #" "C2933536"
+		(property "LCSC Part #" "C17561"
 			(at 104.14 36.83 0)
 			(effects
@@
 			)
 		)
-		(property "Value" "10k"
+		(property "Value" "10k (bussed)"
 			(at 210.566 203.2 90)
 			(effects
