File: post_7seg.kicad_sch (KiCad schematic)
At the start: 8 parts, among them U11 74LS02, U35 74LS248, U36 HDSP-A151, U37 74LS77

Commit message: bringing over learnings/improvements from prototype board
Parts:
- removed R61, R62: 150, Resistor_SMD:R_0805_2012Metric, symbol Device:R_US
- removed U37: 74LS77, Package_DIP:DIP-14_W7.62mm_Socket, symbol 74xx:74LS77
- added C48: 0.1uF 20% Ceramic, Capacitor_SMD:C_0805_2012Metric, symbol Device:C_Small
- added RN1, RN10, RN11, RN2: 10k, Resistor_THT:R_Array_SIP8, symbol Device:R_Pack04_SIP_Split
- added U13: 74LS573, Package_DIP:DIP-20_W7.62mm_Socket, symbol 74xx:74LS573
- added U34: HDSP-A151, Display_7Segment:HDSP-A151, symbol Display_Character:HDSP-A151
- added U37: 74LS247, Package_DIP:DIP-16_W7.62mm_Socket, symbol 74xx:74LS248
- U35: value 74LS248 -> 74LS247
Connections:
- net +5V: now also U36.1 (CA), U36.6 (CA), C48.1, U13.20 (VCC), U34.1 (CA), U34.6 (CA), U37.16 (VCC), U37.3 (~{LT}), U37.5 (~{RBI})
- net D0: now also U13.2 (D0)
- net D1: now also U13.3 (D1)
- net D2: now also U13.4 (D2)
- net D3: now also U13.5 (D3)
- net GND: now also C48.2, U13.1 (OE), U13.10 (GND), U34.7 (DP), U37.8 (GND)
- net LATCH_EN: now also U13.11 (Load)
- net a: now also RN10.2 (R1.2), RN2.2 (R1.2), U34.10 (A); no longer U35.13 (a)
- net b: now also RN1.8 (R4.2), RN10.4 (R2.2), U34.9 (B); no longer U35.12 (b)
- net c: now also RN1.6 (R3.2), RN10.6 (R3.2), U34.8 (C); no longer U35.11 (c)
- net d: now also RN1.4 (R2.2), RN10.8 (R4.2), U34.5 (D); no longer U35.10 (d)
- net e: now also RN1.2 (R1.2), RN11.2 (R1.2), U34.4 (E); no longer U35.9 (e)
- net f: now also RN11.4 (R2.2), RN2.6 (R3.2), U34.2 (F); no longer U35.15 (f)
- net g: now also RN11.6 (R3.2), RN2.4 (R2.2), U34.3 (G); no longer U35.14 (g)
- net DISPA_B: now reaches U35.1 (B)
- net DISPA_B: now also U13.18 (Q1)
- net DISPA_A: now reaches U35.7 (A)
- net DISPA_A: now also U13.19 (Q0)
- net DISPA_D: now reaches U35.6 (D)
- net DISPA_D: now also U13.16 (Q3)
- net DISPA_C: now reaches U35.2 (C)
- net DISPA_C: now also U13.17 (Q2)
- new net: RN10.5 (R3.1), U37.11 (c)
- new net: RN1.1 (R1.1), U35.9 (e)
- new net: RN11.1 (R1.1), U37.9 (e)
- new net: RN11.5 (R3.1), U37.14 (g)
- new net: RN10.1 (R1.1), U37.13 (a)
- new net: RN1.7 (R4.1), U35.12 (b)
- new net: RN1.3 (R2.1), U35.10 (d)
- new net: RN1.5 (R3.1), U35.11 (c)
- new net: RN2.1 (R1.1), U35.13 (a)
- new net: RN2.3 (R2.1), U35.14 (g)
- new net: RN2.5 (R3.1), U35.15 (f)
- new net: RN10.7 (R4.1), U37.10 (d)
- new net: RN10.3 (R2.1), U37.12 (b)
- new net: RN11.3 (R2.1), U37.15 (f)
- new net D4: U13.6 (D4)
- new net D5: U13.7 (D5)
- new net D6: U13.8 (D6)
- new net D7: U13.9 (D7)
- new net DISPB_A: U13.15 (Q4), U37.7 (A)
- new net DISPB_B: U13.14 (Q5), U37.1 (B)
- new net DISPB_C: U13.13 (Q6), U37.2 (C)
- new net DISPB_D: U13.12 (Q7), U37.6 (D)
- no-connect marks 1 -> 6
Other:
- note removed: "consider LS77 (less pins due no ~{Q} outs)"
- moved on the sheet: U11A, U36

Commit message: more pcb routing, implementing learnings from the prototype board
Parts:
- RN1, RN10, RN11, RN2: footprint Resistor_THT:R_Array_SIP8 -> Resistor_SMD:R_Array_Convex_4x0603; symbol Device:R_Pack04_SIP_Split -> Device:R_Pack04_Split
- RN1: renamed from RN2; footprint Resistor_THT:R_Array_SIP8 -> Resistor_SMD:R_Array_Convex_4x0603; symbol Device:R_Pack04_SIP_Split -> Device:R_Pack04_Split
- RN2: renamed from RN1; footprint Resistor_THT:R_Array_SIP8 -> Resistor_SMD:R_Array_Convex_4x0603; symbol Device:R_Pack04_SIP_Split -> Device:R_Pack04_Split
Connections:
- net +5V: now also U34.7 (DP), U36.7 (DP)
- net D0: now also U13.9 (D7); no longer U13.2 (D0)
- net D1: now also U13.8 (D6); no longer U13.3 (D1)
- net D2: now also U13.7 (D5); no longer U13.4 (D2)
- net D3: now also U13.6 (D4); no longer U13.5 (D3)
- net D4: now also U13.5 (D3); no longer U13.6 (D4)
- net D5: now also U13.4 (D2); no longer U13.7 (D5)
- net D6: now also U13.3 (D1); no longer U13.8 (D6)
- net D7: now also U13.2 (D0); no longer U13.9 (D7)
- net DISPA_A: now also U13.12 (Q7); no longer U13.19 (Q0)
- net DISPA_B: now also U13.13 (Q6); no longer U13.18 (Q1)
- net DISPA_C: now also U13.14 (Q5); no longer U13.17 (Q2)
- net DISPA_D: now also U13.15 (Q4); no longer U13.16 (Q3)
- net DISPB_A: now also U13.16 (Q3); no longer U13.15 (Q4)
- net DISPB_B: now also U13.17 (Q2); no longer U13.14 (Q5)
- net DISPB_C: now also U13.18 (Q1); no longer U13.13 (Q6)
- net DISPB_D: now also U13.19 (Q0); no longer U13.12 (Q7)
- net GND: no longer U34.7 (DP), U36.7 (DP)
- net at U37.11 (c): now also RN10.4 (R4.1); no longer RN10.5 (R3.1)
- net at RN2.1 (R1.1): now also U35.10 (d); no longer U35.9 (e)
- net at U37.9 (e): now also RN11.4 (R4.1); no longer RN11.1 (R1.1)
- net at U37.14 (g): now also RN11.3 (R3.1); no longer RN11.5 (R3.1)
- net at U37.13 (a): now also RN10.2 (R2.1); no longer RN10.1 (R1.1)
- net at U35.12 (b): now also RN1.2 (R2.1); no longer RN1.7 (R4.1)
- net at U35.11 (c): now also RN1.1 (R1.1); no longer RN1.5 (R3.1)
- net at U35.13 (a): now also RN1.3 (R3.1); no longer RN1.1 (R1.1)
- net at U35.15 (f): now also RN2.4 (R4.1); no longer RN2.5 (R3.1)
- net at U37.10 (d): now also RN10.1 (R1.1); no longer RN10.7 (R4.1)
- net at U37.15 (f): now also RN11.2 (R2.1); no longer RN11.3 (R2.1)
- removed net a: RN1.2 (R1.2), RN10.2 (R1.2), U34.10 (A), U36.10 (A)
- removed net b: RN1.8 (R4.2), RN10.4 (R2.2), U34.9 (B), U36.9 (B)
- removed net c: RN1.6 (R3.2), RN10.6 (R3.2), U34.8 (C), U36.8 (C)
- net d renamed Bd
- net Bd: no longer RN1.4 (R2.2), U36.5 (D)
- removed net e: RN11.2 (R1.2), RN2.2 (R1.2), U34.4 (E), U36.4 (E)
- removed net f: RN11.4 (R2.2), RN2.6 (R3.2), U34.2 (F), U36.2 (F)
- net g renamed Bg
- net Bg: no longer RN2.4 (R2.2), U36.3 (G)
- new net: RN2.2 (R2.1), U35.9 (e)
- new net Aa: RN1.6 (R3.2), U36.10 (A)
- new net Ab: RN1.7 (R2.2), U36.9 (B)
- new net Ac: RN1.8 (R1.2), U36.8 (C)
- new net Ad: RN2.8 (R1.2), U36.5 (D)
- new net Ae: RN2.7 (R2.2), U36.4 (E)
- new net Af: RN2.5 (R4.2), U36.2 (F)
- new net Ag: RN2.6 (R3.2), U36.3 (G)
- new net Ba: RN10.7 (R2.2), U34.10 (A)
- new net Bb: RN10.6 (R3.2), U34.9 (B)
- new net Bc: RN10.5 (R4.2), U34.8 (C)
- new net Be: RN11.5 (R4.2), U34.4 (E)
- new net Bf: RN11.7 (R2.2), U34.2 (F)

Commit message: pcb is fully routed, working on power capacitor tweaks, some ROM testing
Parts:
- renumbered C46 to C32, C48 to C38, C47 to C40, RN1 to RN6, RN2 to RN7, RN10 to RN8, RN11 to RN9, U36 to U12, U34 to U13, U37 to U19, U11 to U23, U13 to U24, U35 to U25
Connections:
- net D0: now also U24.5 (D3); no longer U24.9 (D7)
- net D1: now also U24.4 (D2); no longer U24.8 (D6)
- net D2: now also U24.3 (D1); no longer U24.7 (D5)
- net D3: now also U24.2 (D0); no longer U24.6 (D4)
- net D4: now also U24.9 (D7); no longer U24.5 (D3)
- net D5: now also U24.8 (D6); no longer U24.4 (D2)
- net D6: now also U24.7 (D5); no longer U24.3 (D1)
- net D7: now also U24.6 (D4); no longer U24.2 (D0)

Commit message: added ATtiny for SMC, added PC speaker
Parts:
- removed RN6, RN7, RN8, RN9: 10k, Resistor_SMD:R_Array_Convex_4x0603, symbol Device:R_Pack04_Split
- added R10, R11, R12, R13, R14, R15, R16, R17, R18, R19, R20, R21, R22, R23: 220, Resistor_SMD:R_0805_2012Metric, symbol Device:R_US
- renumbered C32 to C37, C38 to C43, C40 to C45, U19 to U21, U13 to U22, U12 to U26, U23 to U27, U25 to U28, U24 to U29
Connections:
- net Aa: now also R19.1
- net Ab: now also R20.1
- net Ac: now also R21.1
- net Ad: now also R22.1
- net Ae: now also R23.1
- net Af: now also R17.1
- net Ag: now also R18.1
- net Ba: now also R12.1
- net Bb: now also R13.1
- net Bc: now also R14.1
- net Bd: now also R15.1
- net Be: now also R16.1
- net Bf: now also R10.1
- net Bg: now also R11.1
- net at U21.11 (c): now also R14.2
- net at U28.10 (d): now also R22.2
- net at U21.9 (e): now also R16.2
- net at U21.14 (g): now also R11.2
- net at U21.13 (a): now also R12.2
- net at U28.12 (b): now also R20.2
- net at U28.11 (c): now also R21.2
- net at U28.13 (a): now also R19.2
- net at U28.14 (g): now also R18.2
- net at U28.15 (f): now also R17.2
- net at U28.9 (e): now also R23.2
- net at U21.10 (d): now also R15.2
- net at U21.12 (b): now also R13.2
- net at U21.15 (f): now also R10.2
- no-connect marks 6 -> 2
