File: post_7seg.kicad_sch (KiCad schematic)
At the start: 23 parts, among them U21 74LS247, U22 HDSP-A151, U26 HDSP-A151, U27 74LS02, U28 74LS247, U29 74LS573

Commit message: fix KBC/PPI CS# schematic bugs, add ISA expansion header for adding more cards
Connections:
- net DISPA_A: now also U21.7 (A); no longer U28.7 (A)
- net DISPA_B: now also U21.1 (B); no longer U28.1 (B)
- net DISPA_C: now also U21.2 (C); no longer U28.2 (C)
- net DISPA_D: now also U21.6 (D); no longer U28.6 (D)
- net DISPB_A: now also U28.7 (A); no longer U21.7 (A)
- net DISPB_B: now also U28.1 (B); no longer U21.1 (B)
- net DISPB_C: now also U28.2 (C); no longer U21.2 (C)
- net DISPB_D: now also U28.6 (D); no longer U21.6 (D)
Changed lines of the file:
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@@
+	(wire
+		(pts
+			(xy 85.09 124.46) (xy 76.2 124.46)
+		)
+		(stroke
+			(width 0)
+			(type default)
+		)
+	)
 	(wire
 		(pts
@@
 	(wire
 		(pts
+			(xy 85.09 66.04) (xy 73.66 66.04)
+		)
+		(stroke
+			(width 0)
+			(type default)
+		)
+	)
+	(wire
+		(pts
 			(xy 48.26 44.45) (xy 48.26 49.53)
 		)
@@
 	(wire
 		(pts
-			(xy 85.09 60.96) (xy 76.2 60.96)
-		)
-		(stroke
-			(width 0)
-			(type default)
-		)
-	)
-	(wire
-		(pts
 			(xy 139.7 132.08) (xy 158.75 132.08)
 		)
@@
 		)
 	)
-	(wire
-		(pts
-			(xy 85.09 121.92) (xy 73.66 121.92)
-		)
-		(stroke
-			(width 0)
-			(type default)
-		)
-	)
 	(bus
 		(pts
@@
 	(wire
 		(pts
-			(xy 85.09 66.04) (xy 76.2 66.04)
-		)
-		(stroke
-			(width 0)
-			(type default)
-		)
-	)
-	(wire
-		(pts
 			(xy 48.26 49.53) (xy 52.07 49.53)
 		)
@@
 	(wire
 		(pts
-			(xy 85.09 129.54) (xy 73.66 129.54)
-		)
-		(stroke
-			(width 0)
-			(type default)
-		)
-	)
-	(wire
-		(pts
 			(xy 158.75 60.96) (xy 138.43 60.96)
 		)
@@
 	(wire
 		(pts
+			(xy 85.09 63.5) (xy 73.66 63.5)
+		)
+		(stroke
+			(width 0)
+			(type default)
+		)
+	)
+	(wire
+		(pts
 			(xy 100.33 149.86) (xy 100.33 153.67)
 		)
@@
 	(wire
 		(pts
+			(xy 85.09 68.58) (xy 73.66 68.58)
+		)
+		(stroke
+			(width 0)
+			(type default)
+		)
+	)
+	(wire
+		(pts
 			(xy 81.28 74.93) (xy 81.28 76.2)
 		)
@@
 	(wire
 		(pts
-			(xy 85.09 127) (xy 73.66 127)
+			(xy 85.09 127) (xy 76.2 127)
 		)
 		(stroke
@@
 	(wire
 		(pts
-			(xy 85.09 63.5) (xy 76.2 63.5)
-		)
-		(stroke
-			(width 0)
-			(type default)
-		)
-	)
-	(wire
-		(pts
 			(xy 115.57 63.5) (xy 130.81 63.5)
 		)
@@
 	(wire
 		(pts
+			(xy 85.09 60.96) (xy 73.66 60.96)
+		)
+		(stroke
+			(width 0)
+			(type default)
+		)
+	)
+	(wire
+		(pts
 			(xy 100.33 45.72) (xy 100.33 48.895)
 		)
@@
 	(wire
 		(pts
+			(xy 85.09 121.92) (xy 76.2 121.92)
+		)
+		(stroke
+			(width 0)
+			(type default)
+		)
+	)
+	(wire
+		(pts
 			(xy 158.75 71.12) (xy 138.43 71.12)
 		)
@@
 	(wire
 		(pts
-			(xy 85.09 68.58) (xy 76.2 68.58)
-		)
-		(stroke
-			(width 0)
-			(type default)
-		)
-	)
-	(wire
-		(pts
 			(xy 185.42 132.08) (xy 185.42 137.16)
 		)
@@
 	(wire
 		(pts
+			(xy 85.09 129.54) (xy 76.2 129.54)
+		)
+		(stroke
+			(width 0)
+			(type default)
+		)
+	)
+	(wire
+		(pts
 			(xy 48.26 49.53) (xy 48.26 53.34)
-		)
-		(stroke
-			(width 0)
-			(type default)
-		)
-	)
-	(wire
-		(pts
-			(xy 85.09 124.46) (xy 73.66 124.46)
 		)
 		(stroke
@@
 		)
 	)
-	(label "DISPA_A"
-		(at 76.2 60.96 0)
-		(fields_autoplaced yes)
-		(effects
-			(font
-				(size 1.27 1.27)
-			)
-			(justify left bottom)
-		)
-	)
 	(label "Be"
 		(at 152.4 132.08 0)
@@
 		)
 	)
-	(label "DISPB_A"
-		(at 73.66 121.92 0)
-		(fields_autoplaced yes)
-		(effects
-			(font
-				(size 1.27 1.27)
-			)
-			(justify left bottom)
-		)
-	)
 	(label "DISPB_C"
 		(at 72.39 63.5 180)
@@
 		)
 	)
+	(label "DISPB_A"
+		(at 73.66 60.96 0)
+		(fields_autoplaced yes)
+		(effects
+			(font
+				(size 1.27 1.27)
+			)
+			(justify left bottom)
+		)
+	)
 	(label "DISPA_B"
 		(at 72.39 76.2 180)
@@
 		)
 	)
+	(label "DISPB_D"
+		(at 73.66 68.58 0)
+		(fields_autoplaced yes)
+		(effects
+			(font
+				(size 1.27 1.27)
+			)
+			(justify left bottom)
+		)
+	)
 	(label "DISPA_D"
 		(at 72.39 71.12 180)
@@
 		)
 	)
+	(label "DISPA_B"
+		(at 76.2 124.46 0)
+		(fields_autoplaced yes)
+		(effects
+			(font
+				(size 1.27 1.27)
+			)
+			(justify left bottom)
+		)
+	)
 	(label "LATCH_EN"
 		(at 26.67 83.82 0)
@@
 		)
 	)
+	(label "DISPB_B"
+		(at 73.66 63.5 0)
+		(fields_autoplaced yes)
+		(effects
+			(font
+				(size 1.27 1.27)
+			)
+			(justify left bottom)
+		)
+	)
 	(label "D7"
 		(at 34.29 71.12 180)
@@
 		)
 	)
+	(label "DISPB_C"
+		(at 73.66 66.04 0)
+		(fields_autoplaced yes)
+		(effects
+			(font
+				(size 1.27 1.27)
+			)
+			(justify left bottom)
+		)
+	)
 	(label "D2"
 		(at 34.29 63.5 180)
@@
 		)
 	)
+	(label "DISPA_C"
+		(at 76.2 127 0)
+		(fields_autoplaced yes)
+		(effects
+			(font
+				(size 1.27 1.27)
+			)
+			(justify left bottom)
+		)
+	)
 	(label "Ba"
 		(at 152.4 121.92 0)
@@
 		)
 	)
-	(label "DISPB_B"
-		(at 73.66 124.46 0)
-		(fields_autoplaced yes)
-		(effects
-			(font
-				(size 1.27 1.27)
-			)
-			(justify left bottom)
-		)
-	)
 	(label "Ag"
 		(at 152.4 76.2 0)
@@
 		)
 	)
-	(label "DISPB_C"
-		(at 73.66 127 0)
-		(fields_autoplaced yes)
-		(effects
-			(font
-				(size 1.27 1.27)
-			)
-			(justify left bottom)
-		)
-	)
-	(label "DISPA_B"
-		(at 76.2 63.5 0)
-		(fields_autoplaced yes)
-		(effects
-			(font
-				(size 1.27 1.27)
-			)
-			(justify left bottom)
-		)
-	)
 	(label "LATCH_EN"
 		(at 113.03 22.86 180)
@@
 	)
 	(label "DISPA_D"
-		(at 76.2 68.58 0)
+		(at 76.2 129.54 0)
+		(fields_autoplaced yes)
+		(effects
+			(font
+				(size 1.27 1.27)
+			)
+			(justify left bottom)
+		)
+	)
+	(label "DISPA_A"
+		(at 76.2 121.92 0)
 		(fields_autoplaced yes)
 		(effects
@@
 		)
 	)
-	(label "DISPB_D"
-		(at 73.66 129.54 0)
-		(fields_autoplaced yes)
-		(effects
-			(font
-				(size 1.27 1.27)
-			)
-			(justify left bottom)
-		)
-	)
 	(label "D0"
 		(at 34.29 68.58 180)
@@
 		)
 	)
-	(label "DISPA_C"
-		(at 76.2 66.04 0)
-		(fields_autoplaced yes)
-		(effects
-			(font
-				(size 1.27 1.27)
-			)
-			(justify left bottom)
-		)
-	)

Commit message: fixes, prep for final production run
Parts:
- C37, C43, C45: LCSC Part # (none) -> C1853649
- R10, R11, R12, R13, R14, R15, R16, R17, R18, R19, R20, R21, R22, R23: LCSC Part # (none) -> C114519
- U21, U28: LCSC Part # (none) -> C72115
- U22, U26: LCSC Part # (none) -> C252196
- U27: LCSC Part # (none) -> C72114
- U29: LCSC Part # (none) -> C72118

Commit message: no more SMT for isa_i2c, tweak motherboard multiplex logic, handful of other tweaks
Parts:
- added C15: 0.1uF 20% Ceramic, Capacitor_SMD:C_0805_2012Metric, symbol Device:C
- added unit 4 of U27
- added unit 3 of U27
- added unit 2 of U27
- added unit 5 of U27
Connections:
- net +5V: now also C15.1, U27.14 (VCC)
- net GND: now also C15.2, U27.11, U27.12, U27.5, U27.6, U27.7 (GND), U27.8, U27.9
- no-connect marks 2 -> 5
Other:
- moved on the sheet: C37, C45

Commit message: simplify m88 logic further, reduce ICs, reorient the POST display, use an oscillator for 14.31818 MHz, update isa-i2c bridge BOM
Parts:
- removed R10, R11, R12, R13, R14, R15, R16, R17, R18, R19, R20, R21, R22, R23: 220, Resistor_SMD:R_0805_2012Metric, symbol Device:R_US
- added R1, R3: 220, Resistor_SMD:R_0805_2012Metric, symbol Device:R_US
- U22: value HDSP-A151 -> Low Nibble - HDSP-A151
- U26: value HDSP-A151 -> High Nibble - HDSP-A151
Connections:
- net +5V: now also R1.2, R3.2; no longer U22.1 (CA), U22.6 (CA), U26.1 (CA), U26.6 (CA)
- net Aa: now also U21.13 (a), U22.10 (A); no longer U26.10 (A)
- net Ab: now also U21.12 (b), U22.9 (B); no longer U26.9 (B)
- net Ac: now also U21.11 (c), U22.8 (C); no longer U26.8 (C)
- net Ad: now also U21.10 (d), U22.5 (D); no longer U26.5 (D)
- net Ae: now also U21.9 (e), U22.4 (E); no longer U26.4 (E)
- net Af: now also U21.15 (f), U22.2 (F); no longer U26.2 (F)
- net Ag: now also U21.14 (g), U22.3 (G); no longer U26.3 (G)
- net Ba: now also U26.10 (A), U28.13 (a); no longer U22.10 (A)
- net Bb: now also U26.9 (B), U28.12 (b); no longer U22.9 (B)
- net Bc: now also U26.8 (C), U28.11 (c); no longer U22.8 (C)
- net Bd: now also U26.5 (D), U28.10 (d); no longer U22.5 (D)
- net Be: now also U26.4 (E), U28.9 (e); no longer U22.4 (E)
- net Bf: now also U26.2 (F), U28.15 (f); no longer U22.2 (F)
- net Bg: now also U26.3 (G), U28.14 (g); no longer U22.3 (G)
- net D1: now also U29.2 (D0); no longer U29.4 (D2)
- net D3: now also U29.4 (D2); no longer U29.2 (D0)
- net D5: now also U29.6 (D4); no longer U29.8 (D6)
- net D7: now also U29.8 (D6); no longer U29.6 (D4)
- net DISPA_B: now also U29.15 (Q4); no longer U29.13 (Q6)
- net DISPA_D: now also U29.13 (Q6); no longer U29.15 (Q4)
- net DISPB_B: now also U29.19 (Q0); no longer U29.17 (Q2)
- net DISPB_D: now also U29.17 (Q2); no longer U29.19 (Q0)
- new net: R3.1, U22.1 (CA), U22.6 (CA)
- new net: R1.1, U26.1 (CA), U26.6 (CA)
Other:
- moved on the sheet: C15, U22, U26, U27B, U27C, U27D, U27E

Commit message: motherboard tweaks for manufacturing run, i2c card tweaks for manufacturing run, de9 -> stemma adapter idea for the i2c card
Parts:
- C15, C37, C43, C45: LCSC Part # C1853649 -> C49678
- R1, R3: LCSC Part # C114519 -> C17557
Changed lines of the file:
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@@
 			)
 		)
-		(property "Description" "LCSC #C114519"
+		(property "Description" "LCSC #C17557"
 			(at 162.56 69.85 0)
 			(effects
@@
 			)
 		)
-		(property "LCSC Part #" "C114519"
+		(property "LCSC Part #" "C17557"
 			(at 162.56 69.85 0)
 			(effects
@@
 			)
 		)
-		(property "Description" "LCSC #C1853649"
+		(property "Description" "LCSC #C49678"
 			(at 110.49 48.26 0)
 			(effects
@@
 			)
 		)
-		(property "LCSC Part #" "C1853649"
+		(property "LCSC Part #" "C49678"
 			(at 110.49 48.26 0)
 			(effects
@@
 			)
 		)
-		(property "Description" "LCSC #C1853649"
+		(property "Description" "LCSC #C49678"
 			(at 54.61 49.53 0)
 			(effects
@@
 			)
 		)
-		(property "LCSC Part #" "C1853649"
+		(property "LCSC Part #" "C49678"
 			(at 54.61 49.53 0)
 			(effects
@@
 			)
 		)
-		(property "Description" "LCSC #C1853649"
+		(property "Description" "LCSC #C49678"
 			(at 110.49 110.49 0)
 			(effects
@@
 			)
 		)
-		(property "LCSC Part #" "C1853649"
+		(property "LCSC Part #" "C49678"
 			(at 110.49 110.49 0)
 			(effects
@@
 			)
 		)
-		(property "Description" "LCSC #C1853649"
+		(property "Description" "LCSC #C49678"
 			(at 240.03 31.75 0)
 			(effects
@@
 			)
 		)
-		(property "LCSC Part #" "C1853649"
+		(property "LCSC Part #" "C49678"
 			(at 240.03 31.75 0)
 			(effects
@@
 			)
 		)
-		(property "Description" "LCSC #C114519"
+		(property "Description" "LCSC #C17557"
 			(at 165.1 129.54 0)
 			(effects
@@
 			)
 		)
-		(property "LCSC Part #" "C114519"
+		(property "LCSC Part #" "C17557"
 			(at 165.1 129.54 0)
 			(effects
