File: sbc_buttons.kicad_sch (KiCad schematic)
At the start: 16 parts, among them SW1 SMD_4.6x2.8mm_h2.5mm

Commit message: bringing over learnings/improvements from prototype board
Parts:
- H1, H2, H3, H4, H5, H6, H7, H8, H9: footprint MountingHole:MountingHole_4mm_Pad -> MountingHole:MountingHole_4mm_Pad_Via
- SW1: footprint SparkFun-Switch:Momentary_SMD_4.6x2.8mm_h2.5mm -> Button_Switch_THT:SW_PUSH_6mm_H4.3mm
Changed lines of the file:
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@@
 	(wire
 		(pts
-			(xy 205.74 58.42) (xy 205.74 65.405)
+			(xy 199.39 60.96) (xy 199.39 65.405)
 		)
 		(stroke
@@
 	(wire
 		(pts
-			(xy 205.74 65.405) (xy 207.645 65.405)
+			(xy 199.39 65.405) (xy 207.645 65.405)
 		)
 		(stroke
@@
 			)
 		)
-		(property "Footprint" "MountingHole:MountingHole_4mm_Pad"
+		(property "Footprint" "MountingHole:MountingHole_4mm_Pad_Via"
 			(at 36.83 69.85 0)
 			(effects
@@
 			)
 		)
-		(property "Footprint" "MountingHole:MountingHole_4mm_Pad"
+		(property "Footprint" "MountingHole:MountingHole_4mm_Pad_Via"
 			(at 36.83 125.095 0)
 			(effects
@@
 			)
 		)
-		(property "Footprint" "MountingHole:MountingHole_4mm_Pad"
+		(property "Footprint" "MountingHole:MountingHole_4mm_Pad_Via"
 			(at 36.83 114.3 0)
 			(effects
@@
 			)
 		)
-		(property "Footprint" "MountingHole:MountingHole_4mm_Pad"
+		(property "Footprint" "MountingHole:MountingHole_4mm_Pad_Via"
 			(at 36.83 80.645 0)
 			(effects
@@
 			)
 		)
-		(property "Footprint" "MountingHole:MountingHole_4mm_Pad"
+		(property "Footprint" "MountingHole:MountingHole_4mm_Pad_Via"
 			(at 36.83 102.87 0)
 			(effects
@@
 			)
 		)
-		(property "Footprint" "MountingHole:MountingHole_4mm_Pad"
+		(property "Footprint" "MountingHole:MountingHole_4mm_Pad_Via"
 			(at 36.83 91.44 0)
 			(effects
@@
 	(symbol
 		(lib_id "power:+5V")
-		(at 205.74 58.42 0)
+		(at 199.39 60.96 0)
 		(unit 1)
 		(exclude_from_sim no)
@@
 		(fields_autoplaced yes)
 		(property "Reference" "#PWR091"
-			(at 205.74 62.23 0)
+			(at 199.39 64.77 0)
 			(effects
 				(font
@@
 		)
 		(property "Value" "+5V"
-			(at 205.74 53.34 0)
-			(effects
-				(font
-					(size 1.27 1.27)
-				)
+			(at 201.93 59.6899 0)
+			(effects
+				(font
+					(size 1.27 1.27)
+				)
+				(justify left)
 			)
 		)
 		(property "Footprint" ""
-			(at 205.74 58.42 0)
+			(at 199.39 60.96 0)
 			(effects
 				(font
@@
 		)
 		(property "Datasheet" ""
-			(at 205.74 58.42 0)
-			(effects
-				(font
-					(size 1.27 1.27)
-				)
-				(hide yes)
-			)
-		)
-		(property "Description" ""
-			(at 205.74 58.42 0)
+			(at 199.39 60.96 0)
+			(effects
+				(font
+					(size 1.27 1.27)
+				)
+				(hide yes)
+			)
+		)
+		(property "Description" ""
+			(at 199.39 60.96 0)
 			(effects
 				(font
@@
 			)
 		)
-		(property "Footprint" "MountingHole:MountingHole_4mm_Pad"
+		(property "Footprint" "MountingHole:MountingHole_4mm_Pad_Via"
 			(at 36.83 135.89 0)
 			(effects
@@
 			)
 		)
-		(property "Footprint" "MountingHole:MountingHole_4mm_Pad"
+		(property "Footprint" "MountingHole:MountingHole_4mm_Pad_Via"
 			(at 36.83 158.115 0)
 			(effects
@@
 			)
 		)
-		(property "Footprint" "MountingHole:MountingHole_4mm_Pad"
+		(property "Footprint" "MountingHole:MountingHole_4mm_Pad_Via"
 			(at 36.83 147.32 0)
 			(effects
@@
 			)
 		)
-		(property "Footprint" "SparkFun-Switch:Momentary_SMD_4.6x2.8mm_h2.5mm"
+		(property "Footprint" "Button_Switch_THT:SW_PUSH_6mm_H4.3mm"
 			(at 151.13 67.31 0)
 			(effects

Commit message: pcb is fully routed, working on power capacitor tweaks, some ROM testing
Parts:
- renumbered C16 to C14, D1 to D3, H5 to H1, H1 to H2, H4 to H3, H7 to H4, H6 to H5, H8 to H6, H9 to H7, H3 to H8, H2 to H9, R5 to R10, R7 to R2, R6 to R9
Changed lines of the file:
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@@
 		(dnp no)
 		(fields_autoplaced yes)
-		(property "Reference" "H1"
+		(property "Reference" "H2"
 			(at 35.56 63.5 90)
 			(effects
@@
 			(project "sbc_8088"
 				(path "/5e468d94-0319-44d1-a77f-2adc451eed13/4898bb81-eb43-46b2-921b-826de7c22e53"
-					(reference "H1")
+					(reference "H2")
 					(unit 1)
 				)
@@
 		(dnp no)
 		(fields_autoplaced yes)
-		(property "Reference" "H6"
+		(property "Reference" "H5"
 			(at 35.56 118.745 90)
 			(effects
@@
 			(project "sbc_8088"
 				(path "/5e468d94-0319-44d1-a77f-2adc451eed13/4898bb81-eb43-46b2-921b-826de7c22e53"
-					(reference "H6")
+					(reference "H5")
 					(unit 1)
 				)
@@
 		(dnp no)
 		(fields_autoplaced yes)
-		(property "Reference" "D1"
+		(property "Reference" "D3"
 			(at 219.6465 34.925 0)
 			(effects
@@
 			(project "sbc_8088"
 				(path "/5e468d94-0319-44d1-a77f-2adc451eed13/4898bb81-eb43-46b2-921b-826de7c22e53"
-					(reference "D1")
+					(reference "D3")
 					(unit 1)
 				)
@@
 		(dnp no)
 		(fields_autoplaced yes)
-		(property "Reference" "H5"
+		(property "Reference" "H1"
 			(at 35.56 107.95 90)
 			(effects
@@
 			(project "sbc_8088"
 				(path "/5e468d94-0319-44d1-a77f-2adc451eed13/4898bb81-eb43-46b2-921b-826de7c22e53"
-					(reference "H5")
+					(reference "H1")
 					(unit 1)
 				)
@@
 		(dnp no)
 		(fields_autoplaced yes)
-		(property "Reference" "H2"
+		(property "Reference" "H9"
 			(at 35.56 74.295 90)
 			(effects
@@
 			(project "sbc_8088"
 				(path "/5e468d94-0319-44d1-a77f-2adc451eed13/4898bb81-eb43-46b2-921b-826de7c22e53"
-					(reference "H2")
+					(reference "H9")
 					(unit 1)
 				)
@@
 		(dnp no)
 		(fields_autoplaced yes)
-		(property "Reference" "R6"
+		(property "Reference" "R9"
 			(at 211.455 59.055 90)
 			(effects
@@
 			(project "sbc_8088"
 				(path "/5e468d94-0319-44d1-a77f-2adc451eed13/4898bb81-eb43-46b2-921b-826de7c22e53"
-					(reference "R6")
+					(reference "R9")
 					(unit 1)
 				)
@@
 		(dnp no)
 		(fields_autoplaced yes)
-		(property "Reference" "H4"
+		(property "Reference" "H3"
 			(at 35.56 96.52 90)
 			(effects
@@
 			(project "sbc_8088"
 				(path "/5e468d94-0319-44d1-a77f-2adc451eed13/4898bb81-eb43-46b2-921b-826de7c22e53"
-					(reference "H4")
+					(reference "H3")
 					(unit 1)
 				)
@@
 		(dnp no)
 		(fields_autoplaced yes)
-		(property "Reference" "C16"
+		(property "Reference" "C14"
 			(at 137.16 66.04 0)
 			(effects
@@
 			(project "sbc_8088"
 				(path "/5e468d94-0319-44d1-a77f-2adc451eed13/4898bb81-eb43-46b2-921b-826de7c22e53"
-					(reference "C16")
+					(reference "C14")
 					(unit 1)
 				)
@@
 		(dnp no)
 		(fields_autoplaced yes)
-		(property "Reference" "R5"
+		(property "Reference" "R10"
 			(at 210.185 34.29 90)
 			(effects
@@
 			(project "sbc_8088"
 				(path "/5e468d94-0319-44d1-a77f-2adc451eed13/4898bb81-eb43-46b2-921b-826de7c22e53"
-					(reference "R5")
+					(reference "R10")
 					(unit 1)
 				)
@@
 		(dnp no)
 		(fields_autoplaced yes)
-		(property "Reference" "H3"
+		(property "Reference" "H8"
 			(at 35.56 85.09 90)
 			(effects
@@
 			(project "sbc_8088"
 				(path "/5e468d94-0319-44d1-a77f-2adc451eed13/4898bb81-eb43-46b2-921b-826de7c22e53"
-					(reference "H3")
+					(reference "H8")
 					(unit 1)
 				)
@@
 		(dnp no)
 		(fields_autoplaced yes)
-		(property "Reference" "R7"
+		(property "Reference" "R2"
 			(at 148.59 82.55 0)
 			(effects
@@
 			(project "sbc_8088"
 				(path "/5e468d94-0319-44d1-a77f-2adc451eed13/4898bb81-eb43-46b2-921b-826de7c22e53"
-					(reference "R7")
+					(reference "R2")
 					(unit 1)
 				)
@@
 		(dnp no)
 		(fields_autoplaced yes)
-		(property "Reference" "H7"
+		(property "Reference" "H4"
 			(at 35.56 129.54 90)
 			(effects
@@
 			(project "sbc_8088"
 				(path "/5e468d94-0319-44d1-a77f-2adc451eed13/4898bb81-eb43-46b2-921b-826de7c22e53"
-					(reference "H7")
+					(reference "H4")
 					(unit 1)
 				)
@@
 		(dnp no)
 		(fields_autoplaced yes)
-		(property "Reference" "H9"
+		(property "Reference" "H7"
 			(at 35.56 151.765 90)
 			(effects
@@
 			(project "sbc_8088"
 				(path "/5e468d94-0319-44d1-a77f-2adc451eed13/4898bb81-eb43-46b2-921b-826de7c22e53"
-					(reference "H9")
+					(reference "H7")
 					(unit 1)
 				)
@@
 		(dnp no)
 		(fields_autoplaced yes)
-		(property "Reference" "H8"
+		(property "Reference" "H6"
 			(at 35.56 140.97 90)
 			(effects
@@
 			(project "sbc_8088"
 				(path "/5e468d94-0319-44d1-a77f-2adc451eed13/4898bb81-eb43-46b2-921b-826de7c22e53"
-					(reference "H8")
-					(unit 1)
-				)
+					(reference "H6")
+					(unit 1)
+				)

Commit message: added ATtiny for SMC, added PC speaker
Parts:
- added J8: FP Power Switch, Connector_PinHeader_2.54mm:PinHeader_1x02_P2.54mm_Vertical, symbol Connector_Generic:Conn_01x02
- added R32: 10k, Resistor_SMD:R_0805_2012Metric, symbol Device:R_US
- renumbered D3 to D2, D2 to D3, R10 to R31, R9 to R33
Connections:
- net +5VSB: now also J8.1 (Pin_1)
- net GND: now also R32.2
- new net FP_PWR_SWITCH: J8.2 (Pin_2), R32.1
