File: sbc_buttons.kicad_sch (KiCad schematic)
At the start: 18 parts, among them J8 FP Power Switch, SW1 SMD_4.6x2.8mm_h2.5mm

Commit message: rev A3 pcb, added a fun logo to the BIOS startup
Parts:
- added J12: FP Power LED, Connector_PinHeader_2.54mm:PinHeader_1x02_P2.54mm_Vertical, symbol Connector_Generic:Conn_01x02
- added R49: 300, Resistor_SMD:R_0805_2012Metric, symbol Device:R_US
Connections:
- net +5V: now also R49.1
- net GND: now also J12.1 (Pin_1)
- new net: J12.2 (Pin_2), R49.2
Other:
- moved on the sheet: D3, R31, R33

Commit message: fixes, prep for final production run
Parts:
- C14: LCSC Part # (none) -> C1952580
- D2: LCSC Part # (none) -> C779431
- D3: LCSC Part # (none) -> C779429
- J12, J8: LCSC Part # (none) -> C124375
- R2, R32: LCSC Part # (none) -> C84376
- R31, R33, R49: LCSC Part # (none) -> C114529
- SW1: value SMD_4.6x2.8mm_h2.5mm -> ~; LCSC Part # (none) -> C7470126

Commit message: motherboard tweaks for manufacturing run, i2c card tweaks for manufacturing run, de9 -> stemma adapter idea for the i2c card
Parts:
- C14: LCSC Part # C1952580 -> C15850
- R2, R32: LCSC Part # C84376 -> C17414
- R31, R33, R49: LCSC Part # C114529 -> C17617
Changed lines of the file:
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@@
 			)
 		)
-		(property "Description" "LCSC #C84376"
+		(property "Description" "LCSC #C17414"
 			(at 133.35 138.43 0)
 			(effects
@@
 			)
 		)
-		(property "LCSC Part #" "C84376 "
+		(property "LCSC Part #" "C17414"
 			(at 133.35 138.43 0)
 			(effects
@@
 			)
 		)
-		(property "Description" "LCSC #C114529"
+		(property "Description" "LCSC #C17617"
 			(at 212.09 66.04 0)
 			(effects
@@
 			)
 		)
-		(property "LCSC Part #" "C114529 "
+		(property "LCSC Part #" "C17617"
 			(at 212.09 66.04 0)
 			(effects
@@
 			)
 		)
-		(property "Description" "LCSC #C1952580"
+		(property "Description" "LCSC #C15850"
 			(at 133.35 67.31 0)
 			(effects
@@
 			)
 		)
-		(property "LCSC Part #" "C1952580"
+		(property "LCSC Part #" "C15850"
 			(at 133.35 67.31 0)
 			(effects
@@
 			)
 		)
-		(property "Description" "LCSC #C114529"
+		(property "Description" "LCSC #C17617"
 			(at 210.82 40.64 0)
 			(effects
@@
 			)
 		)
-		(property "LCSC Part #" "C114529 "
+		(property "LCSC Part #" "C17617"
 			(at 210.82 40.64 0)
 			(effects
@@
 			)
 		)
-		(property "Description" "LCSC #C84376"
+		(property "Description" "LCSC #C17414"
 			(at 146.05 83.82 0)
 			(effects
@@
 			)
 		)
-		(property "LCSC Part #" "C84376 "
+		(property "LCSC Part #" "C17414"
 			(at 146.05 83.82 0)
 			(effects
@@
 			)
 		)
-		(property "Description" "LCSC #C114529"
+		(property "Description" "LCSC #C17617"
 			(at 212.09 76.2 0)
 			(effects
@@
 			)
 		)
-		(property "LCSC Part #" "C114529 "
+		(property "LCSC Part #" "C17617"
 			(at 212.09 76.2 0)
 			(effects
