File: sbc_pic.kicad_sch (KiCad schematic)
At the start: 21 parts, among them U16 8259 PIC SLAVE, U17 8259 PIC MASTER

Commit message: bringing over learnings/improvements from prototype board
Parts:
- removed R10, R11, R12, R13, R14, R15, R16, R17, R18, R19, R20, R21, R22, R23, R24, R8, R9: 10k, Resistor_SMD:R_0805_2012Metric, symbol Device:R_US
- added RN7, RN8: 10k, Resistor_THT:R_Array_SIP9, symbol Device:R_Network08
Connections:
- net +5V: now also U17.16 (~{SP}/~{EN})
- net GND: now also U16.16 (~{SP}/~{EN}), RN7.1 (common), RN8.1 (common)
- net IR0: now also RN8.9 (R8)
- net IR1: now also RN8.8 (R7)
- net IR10: now also RN7.7 (R6)
- net IR11: now also RN7.6 (R5)
- net IR12: now also RN7.5 (R4)
- net IR13: now also RN7.4 (R3)
- net IR14: now also RN7.3 (R2)
- net IR15: now also RN7.2 (R1)
- net IR3: now also RN8.6 (R5)
- net IR4: now also RN8.5 (R4)
- net IR5: now also RN8.4 (R3)
- net IR6: now also RN8.3 (R2)
- net IR7: now also RN8.2 (R1)
- net IR8: now also RN7.9 (R8)
- net IR9: now also RN7.8 (R7)
- no-connect marks 0 -> 1

Commit message: pcb is fully routed, working on power capacitor tweaks, some ROM testing
Parts:
- renumbered C18 to C33, C17 to C34, RN8 to RN10, RN7 to RN11, U16 to U18
Changed lines of the file:
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@@
 		(dnp no)
 		(fields_autoplaced yes)
-		(property "Reference" "C17"
+		(property "Reference" "C34"
 			(at 168.9163 46.99 90)
 			(effects
@@
 			(project "sbc_8088"
 				(path "/5e468d94-0319-44d1-a77f-2adc451eed13/3cc0661d-bb7d-4aa8-8cb0-0145893b26d4"
-					(reference "C17")
+					(reference "C34")
 					(unit 1)
 				)
@@
 		(on_board yes)
 		(dnp no)
-		(property "Reference" "RN7"
+		(property "Reference" "RN11"
 			(at 244.856 27.94 90)
 			(effects
@@
 			(project "sbc_8088"
 				(path "/5e468d94-0319-44d1-a77f-2adc451eed13/3cc0661d-bb7d-4aa8-8cb0-0145893b26d4"
-					(reference "RN7")
+					(reference "RN11")
 					(unit 1)
 				)
@@
 		(dnp no)
 		(fields_autoplaced yes)
-		(property "Reference" "U16"
+		(property "Reference" "U18"
 			(at 163.4841 62.23 0)
 			(effects
@@
 			(project "sbc_8088"
 				(path "/5e468d94-0319-44d1-a77f-2adc451eed13/3cc0661d-bb7d-4aa8-8cb0-0145893b26d4"
-					(reference "U16")
+					(reference "U18")
 					(unit 1)
 				)
@@
 		(on_board yes)
 		(dnp no)
-		(property "Reference" "RN8"
+		(property "Reference" "RN10"
 			(at 244.856 55.88 90)
 			(effects
@@
 			(project "sbc_8088"
 				(path "/5e468d94-0319-44d1-a77f-2adc451eed13/3cc0661d-bb7d-4aa8-8cb0-0145893b26d4"
-					(reference "RN8")
+					(reference "RN10")
 					(unit 1)
 				)
@@
 		(dnp no)
 		(fields_autoplaced yes)
-		(property "Reference" "C18"
+		(property "Reference" "C33"
 			(at 101.6063 49.53 90)
 			(effects
@@
 			(project "sbc_8088"
 				(path "/5e468d94-0319-44d1-a77f-2adc451eed13/3cc0661d-bb7d-4aa8-8cb0-0145893b26d4"
-					(reference "C18")
-					(unit 1)
-				)
+					(reference "C33")
+					(unit 1)
+				)

Commit message: added ATtiny for SMC, added PC speaker
Parts:
- renumbered C33 to C38, C34 to C39, RN10 to RN6, RN11 to RN7, U17 to U19, U18 to U20
Connections:
- net GND: now also RN6.7 (R6)
- no-connect marks 1 -> 0
Other:
- note added: "IR2 is used for cascade; no pull-down needed."
Changed lines of the file:
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@@
 		(color 0 0 0 0)
 	)
-	(no_connect
-		(at 240.03 74.93)
-	)
 	(bus_entry
 		(at 115.57 87.63)
@@
 	(wire
 		(pts
+			(xy 236.22 74.93) (xy 236.22 87.63)
+		)
+		(stroke
+			(width 0)
+			(type default)
+		)
+	)
+	(wire
+		(pts
 			(xy 74.93 85.09) (xy 69.85 85.09)
 		)
@@
 		)
 	)
+	(wire
+		(pts
+			(xy 240.03 74.93) (xy 236.22 74.93)
+		)
+		(stroke
+			(width 0)
+			(type default)
+		)
+	)
 	(bus
 		(pts
@@
 		)
 	)
+	(text "IR2 is used for cascade; no pull-down needed."
+		(exclude_from_sim no)
+		(at 226.568 95.504 0)
+		(effects
+			(font
+				(size 1.27 1.27)
+			)
+			(justify left top)
+		)
+	)
 	(label "CAS0"
 		(at 185.42 93.98 180)
@@
 	(symbol
 		(lib_id "power:GND")
+		(at 236.22 87.63 0)
+		(unit 1)
+		(exclude_from_sim no)
+		(in_bom yes)
+		(on_board yes)
+		(dnp no)
+		(fields_autoplaced yes)
+		(property "Reference" "#PWR0323"
+			(at 236.22 93.98 0)
+			(effects
+				(font
+					(size 1.27 1.27)
+				)
+				(hide yes)
+			)
+		)
+		(property "Value" "GND"
+			(at 236.22 92.71 0)
+			(effects
+				(font
+					(size 1.27 1.27)
+				)
+			)
+		)
+		(property "Footprint" ""
+			(at 236.22 87.63 0)
+			(effects
+				(font
+					(size 1.27 1.27)
+				)
+				(hide yes)
+			)
+		)
+		(property "Datasheet" ""
+			(at 236.22 87.63 0)
+			(effects
+				(font
+					(size 1.27 1.27)
+				)
+				(hide yes)
+			)
+		)
+		(property "Description" ""
+			(at 236.22 87.63 0)
+			(effects
+				(font
+					(size 1.27 1.27)
+				)
+				(hide yes)
+			)
+		)
+		(pin "1"
+		)
+		(instances
+			(project "sbc_8088"
+				(path "/5e468d94-0319-44d1-a77f-2adc451eed13/3cc0661d-bb7d-4aa8-8cb0-0145893b26d4"
+					(reference "#PWR0323")
+					(unit 1)
+				)
+			)
+		)
+	)
+	(symbol
+		(lib_id "power:GND")
 		(at 255.27 86.36 0)
 		(unit 1)
@@
 		(dnp no)
 		(fields_autoplaced yes)
-		(property "Reference" "C34"
+		(property "Reference" "C39"
 			(at 168.9163 46.99 90)
 			(effects
@@
 			(project "sbc_8088"
 				(path "/5e468d94-0319-44d1-a77f-2adc451eed13/3cc0661d-bb7d-4aa8-8cb0-0145893b26d4"
-					(reference "C34")
+					(reference "C39")
 					(unit 1)
 				)
@@
 		(on_board yes)
 		(dnp no)
-		(property "Reference" "RN11"
+		(property "Reference" "RN7"
 			(at 244.856 27.94 90)
 			(effects
@@
 			(project "sbc_8088"
 				(path "/5e468d94-0319-44d1-a77f-2adc451eed13/3cc0661d-bb7d-4aa8-8cb0-0145893b26d4"
-					(reference "RN11")
+					(reference "RN7")
 					(unit 1)
 				)
@@
 		(dnp no)
 		(fields_autoplaced yes)
-		(property "Reference" "U18"
+		(property "Reference" "U20"
 			(at 163.4841 62.23 0)
 			(effects
@@
 			(project "sbc_8088"
 				(path "/5e468d94-0319-44d1-a77f-2adc451eed13/3cc0661d-bb7d-4aa8-8cb0-0145893b26d4"
-					(reference "U18")
+					(reference "U20")
 					(unit 1)
 				)
@@
 		(on_board yes)
 		(dnp no)
-		(property "Reference" "RN10"
+		(property "Reference" "RN6"
 			(at 244.856 55.88 90)
 			(effects
@@
 			(project "sbc_8088"
 				(path "/5e468d94-0319-44d1-a77f-2adc451eed13/3cc0661d-bb7d-4aa8-8cb0-0145893b26d4"
-					(reference "RN10")
+					(reference "RN6")
 					(unit 1)
 				)
@@
 		(dnp no)
 		(fields_autoplaced yes)
-		(property "Reference" "C33"
+		(property "Reference" "C38"
 			(at 101.6063 49.53 90)
 			(effects
@@
 			(project "sbc_8088"
 				(path "/5e468d94-0319-44d1-a77f-2adc451eed13/3cc0661d-bb7d-4aa8-8cb0-0145893b26d4"
-					(reference "C33")
+					(reference "C38")
 					(unit 1)
 				)
@@
 		(dnp no)
 		(fields_autoplaced yes)
-		(property "Reference" "U17"
+		(property "Reference" "U19"
 			(at 92.3641 63.5 0)
 			(effects
@@
 			(project "sbc_8088"
 				(path "/5e468d94-0319-44d1-a77f-2adc451eed13/3cc0661d-bb7d-4aa8-8cb0-0145893b26d4"
-					(reference "U17")
+					(reference "U19")
 					(unit 1)
 				)
