File: sbc_pic.kicad_sch (KiCad schematic)
At the start: 6 parts, among them U19 8259 PIC MASTER, U20 8259 PIC SLAVE

Commit message: fixes, prep for final production run
Parts:
- C38, C39: LCSC Part # (none) -> C1853649
- RN6, RN7: LCSC Part # (none) -> C8692
- U19, U20: LCSC Part # (none) -> C72121

Commit message: no more SMT for isa_i2c, tweak motherboard multiplex logic, handful of other tweaks
Parts:
- removed C39: 0.1uF 20% Ceramic, Capacitor_SMD:C_0805_2012Metric, symbol Device:C_Small
- removed RN7: 10k, Resistor_THT:R_Array_SIP9, symbol Device:R_Network08
- removed U20: 8259 PIC SLAVE, Package_DIP:DIP-28_W15.24mm_Socket, symbol Interface:8259
Connections:
- net GND: no longer RN6.7 (R6)
- net IR2: now also RN6.7 (R6)
- net CAS0: no longer names the net of U19.12 (CAS0)
- net CAS1: no longer names the net of U19.13 (CAS1)
- net CAS2: no longer names the net of U19.15 (CAS2)
- no-connect marks 0 -> 3
Other:
- note removed: "IR2 is used for cascade; no pull-down needed."
- moved on the sheet: RN6

Commit message: motherboard tweaks for manufacturing run, i2c card tweaks for manufacturing run, de9 -> stemma adapter idea for the i2c card
Parts:
- C38: LCSC Part # C1853649 -> C49678
- RN6: value 10k -> 10k (bussed)
Changed lines of the file:
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@@
 			)
 		)
-		(property "Value" "10k"
+		(property "Value" "10k (bussed)"
 			(at 166.116 60.96 90)
 			(effects
@@
 			)
 		)
-		(property "Description" "LCSC #C1853649"
+		(property "Description" "LCSC #C49678"
 			(at 101.6 55.88 0)
 			(effects
@@
 			)
 		)
-		(property "LCSC Part #" "C1853649"
-			(at 101.6 55.88 0)
-			(effects
+		(property "LCSC Part #" "C49678"
+			(at 101.6 55.88 0)
+			(effects
