File: sbc_pit.kicad_sch (KiCad schematic)
At the start: 4 parts, among them U18 8254 PIT

Commit message: bringing over learnings/improvements from prototype board
Parts:
- removed R25, R26: 10k, Resistor_SMD:R_0805_2012Metric, symbol Device:R_US
Connections:
- net G0 is gone; now on net +5V: U18.11 (G0)
- net G1 is gone; now on net +5V: U18.14 (G1)
Changed lines of the file:
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@@
-	(wire
-		(pts
-			(xy 209.55 73.66) (xy 209.55 71.12)
-		)
-		(stroke
-			(width 0)
-			(type default)
-		)
-	)
 	(wire
 		(pts
@@
 	(wire
 		(pts
-			(xy 199.39 73.66) (xy 199.39 71.12)
+			(xy 199.39 57.15) (xy 199.39 73.66)
 		)
 		(stroke
@@
 	(wire
 		(pts
-			(xy 209.55 63.5) (xy 209.55 57.15)
-		)
-		(stroke
-			(width 0)
-			(type default)
-		)
-	)
-	(wire
-		(pts
-			(xy 199.39 63.5) (xy 199.39 57.15)
+			(xy 209.55 57.15) (xy 209.55 73.66)
 		)
 		(stroke
@@
 					(unit 1)
 				)
-			)
-		)
-	)
-	(symbol
-		(lib_id "Device:R_US")
-		(at 209.55 67.31 0)
-		(mirror y)
-		(unit 1)
-		(exclude_from_sim no)
-		(in_bom yes)
-		(on_board yes)
-		(dnp no)
-		(fields_autoplaced yes)
-		(property "Reference" "R26"
-			(at 212.09 68.58 0)
-			(effects
-				(font
-					(size 1.27 1.27)
-				)
-				(justify right)
-			)
-		)
-		(property "Value" "10k"
-			(at 212.09 66.04 0)
-			(effects
-				(font
-					(size 1.27 1.27)
-				)
-				(justify right)
-			)
-		)
-		(property "Footprint" "Resistor_SMD:R_0805_2012Metric"
-			(at 208.534 67.564 90)
-			(effects
-				(font
-					(size 1.27 1.27)
-				)
-				(hide yes)
-			)
-		)
-		(property "Datasheet" "~"
-			(at 209.55 67.31 0)
-			(effects
-				(font
-					(size 1.27 1.27)
-				)
-				(hide yes)
-			)
-		)
-		(property "Description" ""
-			(at 209.55 67.31 0)
-			(effects
-				(font
-					(size 1.27 1.27)
-				)
-				(hide yes)
-			)
-		)
-		(pin "2"
-		)
-		(pin "1"
-		)
-		(instances
-			(project "sbc_8088"
-				(path "/5e468d94-0319-44d1-a77f-2adc451eed13/dc082762-fe67-486b-b56c-72b8eb99ff93"
-					(reference "R26")
-					(unit 1)
-				)
-			)
-		)
-	)
-	(symbol
-		(lib_id "Device:R_US")
-		(at 199.39 67.31 0)
-		(mirror y)
-		(unit 1)
-		(exclude_from_sim no)
-		(in_bom yes)
-		(on_board yes)
-		(dnp no)
-		(fields_autoplaced yes)
-		(property "Reference" "R25"
-			(at 201.93 68.58 0)
-			(effects
-				(font
-					(size 1.27 1.27)
-				)
-				(justify right)
-			)
-		)
-		(property "Value" "10k"
-			(at 201.93 66.04 0)
-			(effects
-				(font
-					(size 1.27 1.27)
-				)
-				(justify right)
-			)
-		)
-		(property "Footprint" "Resistor_SMD:R_0805_2012Metric"
-			(at 198.374 67.564 90)
-			(effects
-				(font
-					(size 1.27 1.27)
-				)
-				(hide yes)
-			)
-		)
-		(property "Datasheet" "~"
-			(at 199.39 67.31 0)
-			(effects
-				(font
-					(size 1.27 1.27)
-				)
-				(hide yes)
-			)
-		)
-		(property "Description" ""
-			(at 199.39 67.31 0)
-			(effects
-				(font
-					(size 1.27 1.27)
-				)
-				(hide yes)
-			)
-		)
-		(pin "2"
-		)
-		(pin "1"
-		)
-		(instances
-			(project "sbc_8088"
-				(path "/5e468d94-0319-44d1-a77f-2adc451eed13/dc082762-fe67-486b-b56c-72b8eb99ff93"
-					(reference "R25")
-					(unit 1)
-				)

Commit message: pcb is fully routed, working on power capacitor tweaks, some ROM testing
Parts:
- renumbered C19 to C35, U18 to U20
Changed lines of the file:
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@@
 		(dnp no)
 		(fields_autoplaced yes)
-		(property "Reference" "C19"
+		(property "Reference" "C35"
 			(at 151.1363 60.96 90)
 			(effects
@@
 			(project "sbc_8088"
 				(path "/5e468d94-0319-44d1-a77f-2adc451eed13/dc082762-fe67-486b-b56c-72b8eb99ff93"
-					(reference "C19")
+					(reference "C35")
 					(unit 1)
 				)
@@
 		(dnp no)
 		(fields_autoplaced yes)
-		(property "Reference" "U18"
+		(property "Reference" "U20"
 			(at 141.8941 73.66 0)
 			(effects
@@
 			(project "sbc_8088"
 				(path "/5e468d94-0319-44d1-a77f-2adc451eed13/dc082762-fe67-486b-b56c-72b8eb99ff93"
-					(reference "U18")
+					(reference "U20")
 					(unit 1)
 				)

Commit message: added ATtiny for SMC, added PC speaker
Parts:
- renumbered C35 to C40, U20 to U23
Changed lines of the file:
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@@
 		(dnp no)
 		(fields_autoplaced yes)
-		(property "Reference" "C35"
+		(property "Reference" "C40"
 			(at 151.1363 60.96 90)
 			(effects
@@
 			(project "sbc_8088"
 				(path "/5e468d94-0319-44d1-a77f-2adc451eed13/dc082762-fe67-486b-b56c-72b8eb99ff93"
-					(reference "C35")
+					(reference "C40")
 					(unit 1)
 				)
@@
 		(dnp no)
 		(fields_autoplaced yes)
-		(property "Reference" "U20"
+		(property "Reference" "U23"
 			(at 141.8941 73.66 0)
 			(effects
@@
 			(project "sbc_8088"
 				(path "/5e468d94-0319-44d1-a77f-2adc451eed13/dc082762-fe67-486b-b56c-72b8eb99ff93"
-					(reference "U20")
+					(reference "U23")
 					(unit 1)
 				)
