File: sram.kicad_sch (KiCad schematic)
At the start: 3 parts, among them U30 AS6C1008-55PCN

Commit message: bringing over learnings/improvements from prototype board
Parts:
- removed R56: 10k, Resistor_SMD:R_0805_2012Metric, symbol Device:R_US
Connections:
- net +5V: now also U30.30 (CS2)
Changed lines of the file:
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@@
+		)
+	)
+	(wire
+		(pts
+			(xy 175.26 91.44) (xy 175.26 105.41)
+		)
+		(stroke
+			(width 0)
+			(type default)
 		)
 	)
@@
 	(wire
 		(pts
-			(xy 175.26 105.41) (xy 175.26 101.6)
-		)
-		(stroke
-			(width 0)
-			(type default)
-		)
-	)
-	(wire
-		(pts
 			(xy 129.54 113.03) (xy 135.89 113.03)
 		)
@@
 		(pts
 			(xy 167.64 85.09) (xy 167.64 87.63)
-		)
-		(stroke
-			(width 0)
-			(type default)
-		)
-	)
-	(wire
-		(pts
-			(xy 175.26 93.98) (xy 175.26 91.44)
 		)
 		(stroke
@@
 		)
 	)
-	(symbol
-		(lib_id "Device:R_US")
-		(at 175.26 97.79 0)
-		(unit 1)
-		(exclude_from_sim no)
-		(in_bom yes)
-		(on_board yes)
-		(dnp no)
-		(fields_autoplaced yes)
-		(property "Reference" "R56"
-			(at 177.8 96.52 0)
-			(effects
-				(font
-					(size 1.27 1.27)
-				)
-				(justify left)
-			)
-		)
-		(property "Value" "10k"
-			(at 177.8 99.06 0)
-			(effects
-				(font
-					(size 1.27 1.27)
-				)
-				(justify left)
-			)
-		)
-		(property "Footprint" "Resistor_SMD:R_0805_2012Metric"
-			(at 176.276 98.044 90)
-			(effects
-				(font
-					(size 1.27 1.27)
-				)
-				(hide yes)
-			)
-		)
-		(property "Datasheet" "~"
-			(at 175.26 97.79 0)
-			(effects
-				(font
-					(size 1.27 1.27)
-				)
-				(hide yes)
-			)
-		)
-		(property "Description" ""
-			(at 175.26 97.79 0)
-			(effects
-				(font
-					(size 1.27 1.27)
-				)
-				(hide yes)
-			)
-		)
-		(pin "2"
-		)
-		(pin "1"
-		)
-		(instances
-			(project "sbc_8088"
-				(path "/5e468d94-0319-44d1-a77f-2adc451eed13/60e3f5cc-e9a1-4c51-8079-4abea41f3ef6/d8ffe6c7-769b-4cc5-aca4-7a87a4c90d3d"
-					(reference "R56")
-					(unit 1)
-				)
-				(path "/5e468d94-0319-44d1-a77f-2adc451eed13/60e3f5cc-e9a1-4c51-8079-4abea41f3ef6/e6292733-ef24-480c-87ef-102058650c41"
-					(reference "R57")
-					(unit 1)
-				)
-				(path "/5e468d94-0319-44d1-a77f-2adc451eed13/60e3f5cc-e9a1-4c51-8079-4abea41f3ef6/3295199e-1d64-463f-a9c7-137d49446518"
-					(reference "R58")
-					(unit 1)
-				)
-				(path "/5e468d94-0319-44d1-a77f-2adc451eed13/60e3f5cc-e9a1-4c51-8079-4abea41f3ef6/27cb51fc-351a-4f47-9680-d3bd1524539b"
-					(reference "R59")
-					(unit 1)
-				)
-			)
-		)
-	)

Commit message: pcb is fully routed, working on power capacitor tweaks, some ROM testing
Parts:
- renumbered C41 to C49, U30 to U32
Changed lines of the file:
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@@
 		(dnp no)
 		(fields_autoplaced yes)
-		(property "Reference" "C41"
+		(property "Reference" "C49"
 			(at 153.67 62.23 90)
 			(effects
@@
 			(project "sbc_8088"
 				(path "/5e468d94-0319-44d1-a77f-2adc451eed13/60e3f5cc-e9a1-4c51-8079-4abea41f3ef6/d8ffe6c7-769b-4cc5-aca4-7a87a4c90d3d"
-					(reference "C41")
+					(reference "C49")
 					(unit 1)
 				)
 				(path "/5e468d94-0319-44d1-a77f-2adc451eed13/60e3f5cc-e9a1-4c51-8079-4abea41f3ef6/e6292733-ef24-480c-87ef-102058650c41"
-					(reference "C42")
+					(reference "C47")
 					(unit 1)
 				)
 				(path "/5e468d94-0319-44d1-a77f-2adc451eed13/60e3f5cc-e9a1-4c51-8079-4abea41f3ef6/3295199e-1d64-463f-a9c7-137d49446518"
-					(reference "C43")
+					(reference "C48")
 					(unit 1)
 				)
 				(path "/5e468d94-0319-44d1-a77f-2adc451eed13/60e3f5cc-e9a1-4c51-8079-4abea41f3ef6/27cb51fc-351a-4f47-9680-d3bd1524539b"
-					(reference "C44")
+					(reference "C46")
 					(unit 1)
 				)
@@
 		(on_board yes)
 		(dnp no)
-		(property "Reference" "U30"
+		(property "Reference" "U32"
 			(at 148.59 76.2 0)
 			(effects
@@
 			(project "sbc_8088"
 				(path "/5e468d94-0319-44d1-a77f-2adc451eed13/60e3f5cc-e9a1-4c51-8079-4abea41f3ef6/d8ffe6c7-769b-4cc5-aca4-7a87a4c90d3d"
+					(reference "U32")
+					(unit 1)
+				)
+				(path "/5e468d94-0319-44d1-a77f-2adc451eed13/60e3f5cc-e9a1-4c51-8079-4abea41f3ef6/e6292733-ef24-480c-87ef-102058650c41"
 					(reference "U30")
 					(unit 1)
 				)
-				(path "/5e468d94-0319-44d1-a77f-2adc451eed13/60e3f5cc-e9a1-4c51-8079-4abea41f3ef6/e6292733-ef24-480c-87ef-102058650c41"
+				(path "/5e468d94-0319-44d1-a77f-2adc451eed13/60e3f5cc-e9a1-4c51-8079-4abea41f3ef6/3295199e-1d64-463f-a9c7-137d49446518"
 					(reference "U31")
 					(unit 1)
 				)
-				(path "/5e468d94-0319-44d1-a77f-2adc451eed13/60e3f5cc-e9a1-4c51-8079-4abea41f3ef6/3295199e-1d64-463f-a9c7-137d49446518"
-					(reference "U32")
-					(unit 1)
-				)
 				(path "/5e468d94-0319-44d1-a77f-2adc451eed13/60e3f5cc-e9a1-4c51-8079-4abea41f3ef6/27cb51fc-351a-4f47-9680-d3bd1524539b"
-					(reference "U33")
-					(unit 1)
-				)
+					(reference "U29")
+					(unit 1)
+				)

Commit message: added ATtiny for SMC, added PC speaker
Parts:
- renumbered C49 to C54, U32 to U36
Changed lines of the file:
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@@
 		(dnp no)
 		(fields_autoplaced yes)
-		(property "Reference" "C49"
+		(property "Reference" "C54"
 			(at 153.67 62.23 90)
 			(effects
@@
 			(project "sbc_8088"
 				(path "/5e468d94-0319-44d1-a77f-2adc451eed13/60e3f5cc-e9a1-4c51-8079-4abea41f3ef6/d8ffe6c7-769b-4cc5-aca4-7a87a4c90d3d"
-					(reference "C49")
+					(reference "C54")
 					(unit 1)
 				)
 				(path "/5e468d94-0319-44d1-a77f-2adc451eed13/60e3f5cc-e9a1-4c51-8079-4abea41f3ef6/e6292733-ef24-480c-87ef-102058650c41"
-					(reference "C47")
+					(reference "C52")
 					(unit 1)
 				)
 				(path "/5e468d94-0319-44d1-a77f-2adc451eed13/60e3f5cc-e9a1-4c51-8079-4abea41f3ef6/3295199e-1d64-463f-a9c7-137d49446518"
-					(reference "C48")
+					(reference "C53")
 					(unit 1)
 				)
 				(path "/5e468d94-0319-44d1-a77f-2adc451eed13/60e3f5cc-e9a1-4c51-8079-4abea41f3ef6/27cb51fc-351a-4f47-9680-d3bd1524539b"
-					(reference "C46")
+					(reference "C51")
 					(unit 1)
 				)
@@
 		(on_board yes)
 		(dnp no)
-		(property "Reference" "U32"
+		(property "Reference" "U36"
 			(at 148.59 76.2 0)
 			(effects
@@
 			(project "sbc_8088"
 				(path "/5e468d94-0319-44d1-a77f-2adc451eed13/60e3f5cc-e9a1-4c51-8079-4abea41f3ef6/d8ffe6c7-769b-4cc5-aca4-7a87a4c90d3d"
-					(reference "U32")
+					(reference "U36")
 					(unit 1)
 				)
 				(path "/5e468d94-0319-44d1-a77f-2adc451eed13/60e3f5cc-e9a1-4c51-8079-4abea41f3ef6/e6292733-ef24-480c-87ef-102058650c41"
-					(reference "U30")
+					(reference "U34")
 					(unit 1)
 				)
 				(path "/5e468d94-0319-44d1-a77f-2adc451eed13/60e3f5cc-e9a1-4c51-8079-4abea41f3ef6/3295199e-1d64-463f-a9c7-137d49446518"
-					(reference "U31")
+					(reference "U35")
 					(unit 1)
 				)
 				(path "/5e468d94-0319-44d1-a77f-2adc451eed13/60e3f5cc-e9a1-4c51-8079-4abea41f3ef6/27cb51fc-351a-4f47-9680-d3bd1524539b"
-					(reference "U29")
-					(unit 1)
-				)
+					(reference "U33")
+					(unit 1)
+				)
