File: sram.kicad_sch (KiCad schematic)
At the start: 2 parts, among them U36 AS6C1008-55PCN

Commit message: fixes, prep for final production run
Parts:
- C54: LCSC Part # (none) -> C1853649
- U36: LCSC Part # (none) -> C2874017
Changed lines of the file:
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@@
 			)
 		)
-		(property "Description" ""
+		(property "Description" "LCSC #C1853649"
+			(at 153.67 69.85 0)
+			(effects
+				(font
+					(size 1.27 1.27)
+				)
+				(hide yes)
+			)
+		)
+		(property "Height" ""
+			(at 153.67 69.85 0)
+			(effects
+				(font
+					(size 1.27 1.27)
+				)
+				(hide yes)
+			)
+		)
+		(property "Manufacturer_Name" ""
+			(at 153.67 69.85 0)
+			(effects
+				(font
+					(size 1.27 1.27)
+				)
+				(hide yes)
+			)
+		)
+		(property "Manufacturer_Part_Number" ""
+			(at 153.67 69.85 0)
+			(effects
+				(font
+					(size 1.27 1.27)
+				)
+				(hide yes)
+			)
+		)
+		(property "Mouser Part Number" ""
+			(at 153.67 69.85 0)
+			(effects
+				(font
+					(size 1.27 1.27)
+				)
+				(hide yes)
+			)
+		)
+		(property "Mouser Price/Stock" ""
+			(at 153.67 69.85 0)
+			(effects
+				(font
+					(size 1.27 1.27)
+				)
+				(hide yes)
+			)
+		)
+		(property "LCSC Part #" "C1853649"
 			(at 153.67 69.85 0)
 			(effects
@@
 			)
 		)
-		(property "Description" ""
-			(at 148.59 100.33 0)
-			(effects
+		(property "Description" "LCSC #C2874017 "
+			(at 148.59 100.33 0)
+			(effects
+				(font
+					(size 1.27 1.27)
+				)
+				(hide yes)
+			)
+		)
+		(property "Height" ""
+			(at 148.59 100.33 0)
+			(effects
+				(font
+					(size 1.27 1.27)
+				)
+				(hide yes)
+			)
+		)
+		(property "Manufacturer_Name" ""
+			(at 148.59 100.33 0)
+			(effects
+				(font
+					(size 1.27 1.27)
+				)
+				(hide yes)
+			)
+		)
+		(property "Manufacturer_Part_Number" ""
+			(at 148.59 100.33 0)
+			(effects
+				(font
+					(size 1.27 1.27)
+				)
+				(hide yes)
+			)
+		)
+		(property "Mouser Part Number" ""
+			(at 148.59 100.33 0)
+			(effects
+				(font
+					(size 1.27 1.27)
+				)
+				(hide yes)
+			)
+		)
+		(property "Mouser Price/Stock" ""
+			(at 148.59 100.33 0)
+			(effects
+				(font
+					(size 1.27 1.27)
+				)
+				(hide yes)
+			)
+		)
+		(property "LCSC Part #" "C2874017 "
+			(at 148.59 100.33 0)
+			(effects

Commit message: no more SMT for isa_i2c, tweak motherboard multiplex logic, handful of other tweaks
Other:
- moved on the sheet: C54
Changed lines of the file:
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@@
 	(paper "A4")
 	(junction
-		(at 148.59 69.85)
+		(at 148.59 67.31)
 		(diameter 0)
 		(color 0 0 0 0)
@@
 	(wire
 		(pts
-			(xy 148.59 67.31) (xy 148.59 69.85)
+			(xy 148.59 60.96) (xy 148.59 67.31)
 		)
 		(stroke
@@
 	(wire
 		(pts
-			(xy 148.59 69.85) (xy 149.86 69.85)
-		)
-		(stroke
-			(width 0)
-			(type default)
-		)
-	)
-	(wire
-		(pts
-			(xy 148.59 69.85) (xy 148.59 74.93)
+			(xy 148.59 67.31) (xy 156.21 67.31)
+		)
+		(stroke
+			(width 0)
+			(type default)
+		)
+	)
+	(wire
+		(pts
+			(xy 148.59 67.31) (xy 148.59 74.93)
 		)
 		(stroke
@@
 	(wire
 		(pts
-			(xy 158.75 69.85) (xy 158.75 71.12)
+			(xy 168.91 67.31) (xy 168.91 69.85)
 		)
 		(stroke
@@
 	(wire
 		(pts
-			(xy 157.48 69.85) (xy 158.75 69.85)
+			(xy 163.83 67.31) (xy 168.91 67.31)
 		)
 		(stroke
@@
 					(unit 1)
 				)
+				(path "/5e468d94-0319-44d1-a77f-2adc451eed13/60e3f5cc-e9a1-4c51-8079-4abea41f3ef6/efb6cba0-5032-4bc5-b666-40ce2e18a9bb"
+					(reference "#PWR0331")
+					(unit 1)
+				)
 			)
 		)
@@
 					(unit 1)
 				)
+				(path "/5e468d94-0319-44d1-a77f-2adc451eed13/60e3f5cc-e9a1-4c51-8079-4abea41f3ef6/efb6cba0-5032-4bc5-b666-40ce2e18a9bb"
+					(reference "#PWR0389")
+					(unit 1)
+				)
 			)
 		)
@@
 					(unit 1)
 				)
+				(path "/5e468d94-0319-44d1-a77f-2adc451eed13/60e3f5cc-e9a1-4c51-8079-4abea41f3ef6/efb6cba0-5032-4bc5-b666-40ce2e18a9bb"
+					(reference "#PWR0259")
+					(unit 1)
+				)
 			)
 		)
@@
 	(symbol
 		(lib_id "Device:C")
-		(at 153.67 69.85 90)
+		(at 160.02 67.31 90)
 		(unit 1)
 		(exclude_from_sim no)
@@
 		(fields_autoplaced yes)
 		(property "Reference" "C54"
-			(at 153.67 62.23 90)
+			(at 160.02 59.69 90)
 			(effects
 				(font
@@
 		)
 		(property "Value" "0.1uF 20% Ceramic"
-			(at 153.67 64.77 90)
+			(at 160.02 62.23 90)
 			(effects
 				(font
@@
 		)
 		(property "Footprint" "Capacitor_SMD:C_0805_2012Metric"
-			(at 157.48 68.8848 0)
+			(at 163.83 66.3448 0)
 			(effects
 				(font
@@
 		)
 		(property "Datasheet" "~"
-			(at 153.67 69.85 0)
+			(at 160.02 67.31 0)
 			(effects
 				(font
@@
 		)
 		(property "Description" "LCSC #C1853649"
-			(at 153.67 69.85 0)
+			(at 160.02 67.31 0)
 			(effects
 				(font
@@
 		)
 		(property "Height" ""
-			(at 153.67 69.85 0)
+			(at 160.02 67.31 0)
 			(effects
 				(font
@@
 		)
 		(property "Manufacturer_Name" ""
-			(at 153.67 69.85 0)
+			(at 160.02 67.31 0)
 			(effects
 				(font
@@
 		)
 		(property "Manufacturer_Part_Number" ""
-			(at 153.67 69.85 0)
+			(at 160.02 67.31 0)
 			(effects
 				(font
@@
 		)
 		(property "Mouser Part Number" ""
-			(at 153.67 69.85 0)
+			(at 160.02 67.31 0)
 			(effects
 				(font
@@
 		)
 		(property "Mouser Price/Stock" ""
-			(at 153.67 69.85 0)
+			(at 160.02 67.31 0)
 			(effects
 				(font
@@
 		)
 		(property "LCSC Part #" "C1853649"
-			(at 153.67 69.85 0)
+			(at 160.02 67.31 0)
 			(effects
 				(font
@@
 				(path "/5e468d94-0319-44d1-a77f-2adc451eed13/60e3f5cc-e9a1-4c51-8079-4abea41f3ef6/9b1546e1-77e5-4750-8a58-354545442f58"
 					(reference "C70")
+					(unit 1)
+				)
+				(path "/5e468d94-0319-44d1-a77f-2adc451eed13/60e3f5cc-e9a1-4c51-8079-4abea41f3ef6/efb6cba0-5032-4bc5-b666-40ce2e18a9bb"
+					(reference "C31")
 					(unit 1)
 				)
@@
 					(unit 1)
 				)
+				(path "/5e468d94-0319-44d1-a77f-2adc451eed13/60e3f5cc-e9a1-4c51-8079-4abea41f3ef6/efb6cba0-5032-4bc5-b666-40ce2e18a9bb"
+					(reference "#PWR0278")
+					(unit 1)
+				)
 			)
 		)
@@
 	(symbol
 		(lib_id "power:GND")
-		(at 158.75 71.12 0)
+		(at 168.91 69.85 0)
 		(unit 1)
 		(exclude_from_sim no)
@@
 		(fields_autoplaced yes)
 		(property "Reference" "#PWR0227"
-			(at 158.75 77.47 0)
+			(at 168.91 76.2 0)
 			(effects
 				(font
@@
 		)
 		(property "Value" "GND"
-			(at 158.75 76.2 0)
+			(at 168.91 74.93 0)
 			(effects
 				(font
@@
 		)
 		(property "Footprint" ""
-			(at 158.75 71.12 0)
+			(at 168.91 69.85 0)
 			(effects
 				(font
@@
 		)
 		(property "Datasheet" ""
-			(at 158.75 71.12 0)
+			(at 168.91 69.85 0)
 			(effects
 				(font
@@
 		)
 		(property "Description" ""
-			(at 158.75 71.12 0)
+			(at 168.91 69.85 0)
 			(effects
 				(font
@@
 					(unit 1)
 				)
+				(path "/5e468d94-0319-44d1-a77f-2adc451eed13/60e3f5cc-e9a1-4c51-8079-4abea41f3ef6/efb6cba0-5032-4bc5-b666-40ce2e18a9bb"
+					(reference "#PWR0387")
+					(unit 1)
+				)
 			)
 		)
@@
 	(symbol
 		(lib_id "power:+5V")
-		(at 148.59 67.31 0)
+		(at 148.59 60.96 0)
 		(unit 1)
 		(exclude_from_sim no)
@@
 		(fields_autoplaced yes)
 		(property "Reference" "#PWR0226"
-			(at 148.59 71.12 0)
+			(at 148.59 64.77 0)
 			(effects
 				(font
@@
 		)
 		(property "Value" "+5V"
-			(at 148.59 62.23 0)
+			(at 148.59 55.88 0)
 			(effects
 				(font
@@
 		)
 		(property "Footprint" ""
-			(at 148.59 67.31 0)
+			(at 148.59 60.96 0)
 			(effects
 				(font
@@
 		)
 		(property "Datasheet" ""
-			(at 148.59 67.31 0)
+			(at 148.59 60.96 0)
 			(effects
 				(font
@@
 		)
 		(property "Description" ""
-			(at 148.59 67.31 0)
+			(at 148.59 60.96 0)
 			(effects
 				(font
@@
 				(path "/5e468d94-0319-44d1-a77f-2adc451eed13/60e3f5cc-e9a1-4c51-8079-4abea41f3ef6/9b1546e1-77e5-4750-8a58-354545442f58"
 					(reference "#PWR0346")
+					(unit 1)
+				)
+				(path "/5e468d94-0319-44d1-a77f-2adc451eed13/60e3f5cc-e9a1-4c51-8079-4abea41f3ef6/efb6cba0-5032-4bc5-b666-40ce2e18a9bb"
+					(reference "#PWR0328")
 					(unit 1)
 				)
@@
 					(unit 1)
 				)
+				(path "/5e468d94-0319-44d1-a77f-2adc451eed13/60e3f5cc-e9a1-4c51-8079-4abea41f3ef6/efb6cba0-5032-4bc5-b666-40ce2e18a9bb"
+					(reference "U14")
+					(unit 1)
+				)

Commit message: motherboard tweaks for manufacturing run, i2c card tweaks for manufacturing run, de9 -> stemma adapter idea for the i2c card
Parts:
- C51: renamed from C54; LCSC Part # C1853649 -> C49678
- renumbered U36 to U33
Changed lines of the file:
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@@
 		(dnp no)
 		(fields_autoplaced yes)
-		(property "Reference" "#PWR0229"
+		(property "Reference" "#PWR0257"
 			(at 148.59 134.62 0)
 			(effects
@@
 		(dnp no)
 		(fields_autoplaced yes)
-		(property "Reference" "#PWR0228"
+		(property "Reference" "#PWR0256"
 			(at 175.26 95.25 0)
 			(effects
@@
 		(dnp no)
 		(fields_autoplaced yes)
-		(property "Reference" "#PWR0230"
+		(property "Reference" "#PWR0252"
 			(at 97.79 58.42 0)
 			(effects
@@
 		(dnp no)
 		(fields_autoplaced yes)
-		(property "Reference" "C54"
+		(property "Reference" "C51"
 			(at 160.02 59.69 90)
 			(effects
@@
 			)
 		)
-		(property "Description" "LCSC #C1853649"
+		(property "Description" "LCSC #C49678"
 			(at 160.02 67.31 0)
 			(effects
@@
 			)
 		)
-		(property "LCSC Part #" "C1853649"
+		(property "LCSC Part #" "C49678"
 			(at 160.02 67.31 0)
 			(effects
@@
 		(dnp no)
 		(fields_autoplaced yes)
-		(property "Reference" "#PWR0231"
+		(property "Reference" "#PWR0253"
 			(at 97.79 66.04 0)
 			(effects
@@
 		(dnp no)
 		(fields_autoplaced yes)
-		(property "Reference" "#PWR0227"
+		(property "Reference" "#PWR0255"
 			(at 168.91 76.2 0)
 			(effects
@@
 		(dnp no)
 		(fields_autoplaced yes)
-		(property "Reference" "#PWR0226"
+		(property "Reference" "#PWR0254"
 			(at 148.59 64.77 0)
 			(effects
@@
 		(on_board yes)
 		(dnp no)
-		(property "Reference" "U36"
+		(property "Reference" "U33"
 			(at 148.59 76.2 0)
 			(effects
