File: clockgen.kicad_sch (KiCad schematic)
At the start: 9 parts, among them U32 8284 CLOCK GENERATOR, U37 74HC74, Y1 14.31818 MHz Crystal

Commit message: fixes, prep for final production run
Parts:
- added C71: 0.1uF 20% Ceramic, Capacitor_SMD:C_0805_2012Metric, symbol Device:C
- added C73: 30 pF 1% 10V Ceramic, Capacitor_SMD:C_0805_2012Metric, symbol Device:C
- added R1, R3: 510, Resistor_SMD:R_0805_2012Metric, symbol Device:R_US
- added U1: 8284 CLOCK GENERATOR, Package_DIP:DIP-18_W7.62mm_Socket, symbol Timer:8284
- added Y2: 14.31818 MHz Crystal, Crystal:Crystal_HC49-4H_Vertical, symbol PCM_SL_Devices:Crystal_24MHz
- C55, C57: LCSC Part # (none) -> C1853649
- C56: LCSC Part # (none) -> C527184
- R24, R25: LCSC Part # (none) -> C114563
- R26: LCSC Part # (none) -> C84376
- U32: LCSC Part # (none) -> C72116
- U37: LCSC Part # (none) -> C72114
- Y1: value 14.31818 MHz Crystal -> 24 MHz Crystal; LCSC Part # (none) -> C240917
Connections:
- net +5V: now also C71.1, C73.2, U1.18 (VCC), U1.4 (RDY1)
- net GND: now also C71.2, R1.2, R3.2, U1.1 (CSYNC), U1.13 (F/~{C}), U1.15 (~{ASYNC}), U1.3 (~{AEN1}), U1.6 (RDY2), U1.7 (~{AEN2}), U1.9 (GND)
- net PCLK: now also U1.2 (PCLK)
- net ~{RESET}: now also U1.11 (~{RES})
- new net: R3.1, U1.16 (X2), Y2.1
- new net: C73.1, R1.1, U1.17 (X1), Y2.2
- new net ISA_OSC: U1.12 (OSC)
- no-connect marks 3 -> 7
Other:
- note added: "14.318 MHz Clock Generator (ISA OSC, PIT ticks) No READY logic."
- note added: "8284 Clock/Reset/Ready Generator For 8088"
- note removed: "8284 Clock/Reset/Ready Generator"

Commit message: bump cpu to 8mhz, add second clock gen for ISA bus and PIT
Connections:
- net PCLK: no longer U1.2 (PCLK), U37.3 (C)
- new net PIT_CLK: U1.2 (PCLK), U37.3 (C)
Changed lines of the file:
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@@
 	(wire
 		(pts
-			(xy 53.34 115.57) (xy 59.69 115.57)
+			(xy 53.34 115.57) (xy 63.5 115.57)
 		)
 		(stroke
@@
 	(wire
 		(pts
+			(xy 58.42 120.65) (xy 72.39 120.65)
+		)
+		(stroke
+			(width 0)
+			(type default)
+		)
+	)
+	(wire
+		(pts
+			(xy 161.29 106.68) (xy 175.26 106.68)
+		)
+		(stroke
+			(width 0)
+			(type default)
+		)
+	)
+	(wire
+		(pts
+			(xy 203.2 54.61) (xy 208.28 54.61)
+		)
+		(stroke
+			(width 0)
+			(type default)
+		)
+	)
+	(wire
+		(pts
+			(xy 58.42 125.73) (xy 58.42 120.65)
+		)
+		(stroke
+			(width 0)
+			(type default)
+		)
+	)
+	(wire
+		(pts
+			(xy 189.23 40.64) (xy 189.23 46.99)
+		)
+		(stroke
+			(width 0)
+			(type default)
+		)
+	)
+	(wire
+		(pts
+			(xy 21.59 105.41) (xy 21.59 95.25)
+		)
+		(stroke
+			(width 0)
+			(type default)
+		)
+	)
+	(wire
+		(pts
+			(xy 175.26 106.68) (xy 179.07 106.68)
+		)
+		(stroke
+			(width 0)
+			(type default)
+		)
+	)
+	(wire
+		(pts
+			(xy 203.2 68.58) (xy 203.2 54.61)
+		)
+		(stroke
+			(width 0)
+			(type default)
+		)
+	)
+	(wire
+		(pts
+			(xy 242.57 80.01) (xy 246.38 80.01)
+		)
+		(stroke
+			(width 0)
+			(type default)
+		)
+	)
+	(wire
+		(pts
+			(xy 135.89 99.06) (xy 114.3 99.06)
+		)
+		(stroke
+			(width 0)
+			(type default)
+		)
+	)
+	(wire
+		(pts
 			(xy 156.21 101.6) (xy 158.75 101.6)
-		)
-		(stroke
-			(width 0)
-			(type default)
-		)
-	)
-	(wire
-		(pts
-			(xy 58.42 120.65) (xy 72.39 120.65)
-		)
-		(stroke
-			(width 0)
-			(type default)
-		)
-	)
-	(wire
-		(pts
-			(xy 161.29 106.68) (xy 175.26 106.68)
-		)
-		(stroke
-			(width 0)
-			(type default)
-		)
-	)
-	(wire
-		(pts
-			(xy 203.2 54.61) (xy 208.28 54.61)
-		)
-		(stroke
-			(width 0)
-			(type default)
-		)
-	)
-	(wire
-		(pts
-			(xy 58.42 125.73) (xy 58.42 120.65)
-		)
-		(stroke
-			(width 0)
-			(type default)
-		)
-	)
-	(wire
-		(pts
-			(xy 189.23 40.64) (xy 189.23 46.99)
-		)
-		(stroke
-			(width 0)
-			(type default)
-		)
-	)
-	(wire
-		(pts
-			(xy 21.59 105.41) (xy 21.59 95.25)
-		)
-		(stroke
-			(width 0)
-			(type default)
-		)
-	)
-	(wire
-		(pts
-			(xy 175.26 106.68) (xy 179.07 106.68)
-		)
-		(stroke
-			(width 0)
-			(type default)
-		)
-	)
-	(wire
-		(pts
-			(xy 203.2 68.58) (xy 203.2 54.61)
-		)
-		(stroke
-			(width 0)
-			(type default)
-		)
-	)
-	(wire
-		(pts
-			(xy 242.57 80.01) (xy 246.38 80.01)
-		)
-		(stroke
-			(width 0)
-			(type default)
-		)
-	)
-	(wire
-		(pts
-			(xy 135.89 99.06) (xy 114.3 99.06)
 		)
 		(stroke
@@
 		)
 	)
-	(label "PCLK"
-		(at 59.69 115.57 180)
+	(label "PIT_CLK"
+		(at 63.5 115.57 180)
 		(fields_autoplaced yes)
 		(effects
@@
 		)
 	)
-	(label "PCLK"
+	(label "PIT_CLK"
 		(at 194.31 57.15 0)
 		(fields_autoplaced yes)
@@
 		)
 	)
+	(hierarchical_label "PCLK"
+		(shape output)
+		(at 158.75 101.6 0)
+		(fields_autoplaced yes)
+		(effects
+			(font
+				(size 1.27 1.27)
+			)
+			(justify left)
+		)
+	)
 	(hierarchical_label "~{RESET}"
 		(shape input)
@@
 		)
 	)
-	(hierarchical_label "PCLK"
-		(shape output)
-		(at 158.75 101.6 0)
-		(fields_autoplaced yes)
-		(effects
-			(font
-				(size 1.27 1.27)
-			)
-			(justify left)
-		)
-	)

Commit message: part tweaks, BOM is pretty much finalized, use 0.5W resistors for bleeders
Parts:
- R1, R24, R25, R3: LCSC Part # C114563 -> C309660
Changed lines of the file:
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@@
 			)
 		)
-		(property "Description" "LCSC #C114563 "
+		(property "Description" "LCSC #C309660"
 			(at 86.36 120.65 0)
 			(effects
@@
 			)
 		)
-		(property "LCSC Part #" "C114563 "
+		(property "LCSC Part #" "C309660"
 			(at 86.36 120.65 0)
 			(effects
@@
 			)
 		)
-		(property "Description" "LCSC #C114563 "
+		(property "Description" "LCSC #C309660"
 			(at 86.36 140.97 0)
 			(effects
@@
 			)
 		)
-		(property "LCSC Part #" "C114563 "
+		(property "LCSC Part #" "C309660"
 			(at 86.36 140.97 0)
 			(effects
@@
 			)
 		)
-		(property "Description" "LCSC #C114563 "
+		(property "Description" "LCSC #C309660"
 			(at 189.23 106.68 0)
 			(effects
@@
 			)
 		)
-		(property "LCSC Part #" "C114563 "
+		(property "LCSC Part #" "C309660"
 			(at 189.23 106.68 0)
 			(effects
@@
 			)
 		)
-		(property "Description" "LCSC #C114563 "
+		(property "Description" "LCSC #C309660"
 			(at 189.23 127 0)
 			(effects
@@
 			)
 		)
-		(property "LCSC Part #" "C114563 "
+		(property "LCSC Part #" "C309660"
 			(at 189.23 127 0)
 			(effects

Commit message: no more SMT for isa_i2c, tweak motherboard multiplex logic, handful of other tweaks
Parts:
- removed C56: 30 pF 1% 10V Ceramic, Capacitor_SMD:C_0805_2012Metric, symbol Device:C
- added C16: 30 pF 1% 10V Ceramic, Capacitor_SMD:C_0805_2012Metric, symbol Device:C
- R26: value 10k -> 1k; LCSC Part # C84376 -> (none)
Connections:
- net +5V: no longer C73.2
- net GND: now also R1.1, R24.1, R25.1, R3.1; no longer R1.2, R24.2, R25.2, R3.2
- net at U32.16 (X2), Y1.1: now also R25.2; no longer R25.1
- new net: R3.2, U1.16 (X2), Y2.2
- new net: C73.2, R1.2, U1.17 (X1)
- new net: C16.2, R24.2, U32.17 (X1)
- new net: C16.1, Y1.2
- new net: C73.1, Y2.1
Other:
- moved on the sheet: C73, R25, R3, Y1, Y2

Commit message: simplify m88 logic further, reduce ICs, reorient the POST display, use an oscillator for 14.31818 MHz, update isa-i2c bridge BOM
Parts:
- removed C57, C71: 0.1uF 20% Ceramic, Capacitor_SMD:C_0805_2012Metric, symbol Device:C
- removed C73: 30 pF 1% 10V Ceramic, Capacitor_SMD:C_0805_2012Metric, symbol Device:C
- removed R1, R3: 510, Resistor_SMD:R_0805_2012Metric, symbol Device:R_US
- removed U1: 8284 CLOCK GENERATOR, Package_DIP:DIP-18_W7.62mm_Socket, symbol Timer:8284
- removed U37: 74HC74, Package_DIP:DIP-14_W7.62mm_Socket, symbol 74xx:74HC74
- removed Y2: 14.31818 MHz Crystal, Crystal:Crystal_HC49-4H_Vertical, symbol PCM_SL_Devices:Crystal_24MHz
- added C44, C46: 0.1uF 20% Ceramic, Capacitor_SMD:C_0805_2012Metric, symbol Device:C
- added C47: 30 pF 1% 10V Ceramic, Capacitor_SMD:C_0805_2012Metric, symbol Device:C
- added U3: 74LS92, Package_DIP:DIP-14_W7.62mm_Socket, symbol 74xx:74LS92
- added X1: 14.31818MHz Crystal Oscillator, Crystal:Crystal_SMD_5032-4Pin_5.0x3.2mm, symbol Oscillator:ASCO
- R26: LCSC Part # (none) -> C517536
Connections:
- net +5V: now also C44.1, C46.1, U3.5 (VCC), X1.4 (VDD)
- net CLK_1.19MHz: now also U3.8 (Q3)
- net GND: now also C44.2, C46.2, C47.2, U3.10 (GND), X1.2 (GND)
- net ISA_OSC: now also C47.1, U3.14 (CP0), X1.3 (OUT)
- net RESET: now also U3.6 (R0(1)), U3.7 (R0(2))
- new net: U3.1 (CP1..3), U3.12 (Q0)
- no-connect marks 7 -> 3
Other:
- note added: "14.318 MHz Clock (ISA OSC, PIT ticks)"
- note removed: "14.318 MHz Clock Generator (ISA OSC, PIT ticks) No READY logic."
- note removed: "PCLK = 1/6th of the input clock 1.19 MHz = 1/12th of the input clock"

Commit message: m88: use a dip-8 style oscillator footprint, not fully routed yet
Parts:
- removed X1: 14.31818MHz Crystal Oscillator, Crystal:Crystal_SMD_5032-4Pin_5.0x3.2mm, symbol Oscillator:ASCO
- added X1: CXO_DIP8, Package_DIP:DIP-8_W7.62mm, symbol Oscillator:CXO_DIP8
Connections:
- net +5V: now also X1.8 (Vcc)
- net GND: now also X1.4 (GND)
- net ISA_OSC: now also X1.5 (OUT)
- net CLK_7.159MHz: now reaches U3.1 (CP1..3), U3.12 (Q0)
- net CLK_2.386MHz_A: now reaches U3.11 (Q1)
- net CLK_2.386MHz_B: now reaches U3.9 (Q2)
- no-connect marks 3 -> 4
Other:
- note added: "B has a ~240 degree phase shift"
Changed lines of the file:
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@@
 	)
 	(no_connect
-		(at 62.23 163.83)
+		(at 86.36 161.29)
 	)
 	(no_connect
-		(at 21.59 109.22)
+		(at 24.13 109.22)
+	)
+	(no_connect
+		(at 86.36 163.83)
 	)
 	(no_connect
@@
 	(wire
 		(pts
+			(xy 62.23 161.29) (xy 86.36 161.29)
+		)
+		(stroke
+			(width 0)
+			(type default)
+		)
+	)
+	(wire
+		(pts
 			(xy 135.89 93.98) (xy 125.73 93.98)
 		)
@@
 	(wire
 		(pts
-			(xy 41.91 109.22) (xy 45.72 109.22)
+			(xy 31.75 92.71) (xy 38.1 92.71)
 		)
 		(stroke
@@
 	(wire
 		(pts
-			(xy 31.75 92.71) (xy 38.1 92.71)
+			(xy 71.12 43.18) (xy 81.28 43.18)
 		)
 		(stroke
@@
 	(wire
 		(pts
-			(xy 71.12 43.18) (xy 81.28 43.18)
+			(xy 49.53 147.32) (xy 49.53 151.13)
 		)
 		(stroke
@@
 	(wire
 		(pts
-			(xy 49.53 147.32) (xy 49.53 151.13)
+			(xy 125.73 125.73) (xy 146.05 125.73)
 		)
 		(stroke
@@
 	(wire
 		(pts
-			(xy 125.73 125.73) (xy 146.05 125.73)
+			(xy 72.39 184.15) (xy 72.39 158.75)
 		)
 		(stroke
@@
 	(wire
 		(pts
-			(xy 72.39 184.15) (xy 72.39 158.75)
+			(xy 81.28 43.18) (xy 81.28 41.91)
 		)
 		(stroke
@@
 	(wire
 		(pts
-			(xy 81.28 43.18) (xy 81.28 41.91)
+			(xy 62.23 163.83) (xy 86.36 163.83)
 		)
 		(stroke
@@
 	(wire
 		(pts
+			(xy 39.37 109.22) (xy 45.72 109.22)
+		)
+		(stroke
+			(width 0)
+			(type default)
+		)
+	)
+	(wire
+		(pts
 			(xy 114.3 91.44) (xy 114.3 99.06)
 		)
@@
 		)
 	)
+	(text "B has a ~240 degree phase shift"
+		(exclude_from_sim no)
+		(at 89.662 165.862 0)
+		(effects
+			(font
+				(size 1.27 1.27)
+			)
+			(justify left)
+		)
+	)
+	(label "CLK_7.159MHz"
+		(at 72.39 158.75 0)
+		(fields_autoplaced yes)
+		(effects
+			(font
+				(size 1.27 1.27)
+			)
+			(justify left bottom)
+		)
+	)
 	(label "RESET"
 		(at 163.83 96.52 0)
@@
 		)
 	)
+	(label "CLK_2.386MHz_B"
+		(at 76.2 163.83 0)
+		(fields_autoplaced yes)
+		(effects
+			(font
+				(size 1.27 1.27)
+			)
+			(justify left bottom)
+		)
+	)
+	(label "CLK_2.386MHz_A"
+		(at 76.2 161.29 0)
+		(fields_autoplaced yes)
+		(effects
+			(font
+				(size 1.27 1.27)
+			)
+			(justify left bottom)
+		)
+	)
 	(label "RESET"
 		(at 29.21 166.37 0)
@@
 	)
 	(symbol
+		(lib_id "Oscillator:CXO_DIP8")
+		(at 31.75 109.22 0)
+		(unit 1)
+		(exclude_from_sim no)
+		(in_bom yes)
+		(on_board yes)
+		(dnp no)
+		(fields_autoplaced yes)
+		(property "Reference" "X1"
+			(at 43.18 102.9014 0)
+			(effects
+				(font
+					(size 1.27 1.27)
+				)
+			)
+		)
+		(property "Value" "CXO_DIP8"
+			(at 43.18 105.4414 0)
+			(effects
+				(font
+					(size 1.27 1.27)
+				)
+			)
+		)
+		(property "Footprint" "Package_DIP:DIP-8_W7.62mm"
+			(at 43.18 118.11 0)
+			(effects
+				(font
+					(size 1.27 1.27)
+				)
+				(hide yes)
+			)
+		)
+		(property "Datasheet" "http://cdn-reichelt.de/documents/datenblatt/B400/OSZI.pdf"
+			(at 29.21 109.22 0)
+			(effects
+				(font
+					(size 1.27 1.27)
+				)
+				(hide yes)
+			)
+		)
+		(property "Description" "LCSC #C72124"
+			(at 31.75 109.22 0)
+			(effects
+				(font
+					(size 1.27 1.27)
+				)
+				(hide yes)
+			)
+		)
+		(property "LCSC Part #" "C72124"
+			(at 31.75 109.22 0)
+			(effects
+				(font
+					(size 1.27 1.27)
+				)
+				(hide yes)
+			)
+		)
+		(pin "1"
+		)
+		(pin "5"
+		)
+		(pin "8"
+		)
+		(pin "4"
+		)
+		(instances
+			(project ""
+				(path "/5e468d94-0319-44d1-a77f-2adc451eed13/fd224fc0-1ec7-490c-af34-c6b2523d21f4"
+					(reference "X1")
+					(unit 1)
+				)
+			)
+		)
+	)
+	(symbol
 		(lib_id "Device:C")
 		(at 45.72 114.3 0)
@@
 		(on_board yes)
 		(dnp no)
-		(fields_autoplaced yes)
 		(property "Reference" "C47"
 			(at 49.53 114.2999 0)
@@
 		)
 		(property "Value" "30 pF 1% 10V Ceramic"
-			(at 41.91 113.03 0)
+			(at 72.39 116.586 0)
 			(effects
 				(font
@@
 				)
 				(justify right)
-				(hide yes)
 			)
 		)
@@
 			)
 		)
-		(property "Description" "LCSC #C527184 "
+		(property "Description" "LCSC #C527184"
 			(at 45.72 114.3 0)
 			(effects
@@
 	)
 	(symbol
-		(lib_id "Oscillator:ASCO")
-		(at 31.75 109.22 0)
-		(unit 1)
-		(exclude_from_sim no)
-		(in_bom yes)
-		(on_board yes)
-		(dnp no)
-		(property "Reference" "X1"
-			(at 48.514 98.806 0)
-			(effects
-				(font
-					(size 1.27 1.27)
-				)
-			)
-		)
-		(property "Value" "14.31818MHz Crystal Oscillator"
-			(at 48.514 101.346 0)
-			(effects
-				(font
-					(size 1.27 1.27)
-				)
-			)
-		)
-		(property "Footprint" "Crystal:Crystal_SMD_5032-4Pin_5.0x3.2mm"
-			(at 34.29 118.11 0)
-			(effects
-				(font
-					(size 1.27 1.27)
-				)
-				(hide yes)
-			)
-		)
-		(property "Datasheet" "https://abracon.com/Oscillators/ASCO.pdf"
-			(at 26.035 106.045 0)
-			(effects
-				(font
-					(size 1.27 1.27)
-				)
-				(hide yes)
-			)
-		)
-		(property "Description" "Crystal Clock Oscillator, Abracon ASCO"
-			(at 31.75 109.22 0)
-			(effects
-				(font
-					(size 1.27 1.27)
-				)
-				(hide yes)
-			)
-		)
-		(pin "1"
-		)
-		(pin "4"
-		)
-		(pin "3"
-		)
-		(pin "2"
-		)
-		(instances
-			(project "sbc_8088"
-				(path "/5e468d94-0319-44d1-a77f-2adc451eed13/fd224fc0-1ec7-490c-af34-c6b2523d21f4"
-					(reference "X1")
-					(unit 1)
-				)
-			)
-		)
-	)
-	(symbol
 		(lib_id "power:+5V")
 		(at 114.3 86.36 0)
@@
 			)
 		)
-		(property "Description" "LCSC #C527184 "
+		(property "Description" "LCSC #C527184"
 			(at 181.61 106.68 0)
 			(effects
@@
 			)
 		)
-		(property "Description" "LCSC #C72116 "
+		(property "Description" "LCSC #C72116"
 			(at 146.05 101.6 0)
 			(effects

Commit message: motherboard tweaks for manufacturing run, i2c card tweaks for manufacturing run, de9 -> stemma adapter idea for the i2c card
Parts:
- added C56: 0.1uF 20% Ceramic, Capacitor_SMD:C_0805_2012Metric, symbol Device:C
- added C57: 30 pF 1% 10V Ceramic, Capacitor_SMD:C_0805_2012Metric, symbol Device:C
- added J21: Conn_01x03, Connector_PinHeader_2.54mm:PinHeader_1x03_P2.54mm_Vertical, symbol Connector_Generic:Conn_01x03
- added R10: 10k, Resistor_SMD:R_0805_2012Metric, symbol Device:R_US
- added X2: CXO_DIP8, Package_DIP:DIP-8_W7.62mm_Socket, symbol Oscillator:CXO_DIP8
- C16, R24, R25, Y1: now not fitted
- C44, C46, C55: LCSC Part # C1853649 -> C49678
- C47: LCSC Part # C527184 -> C107114
- R26: LCSC Part # C517536 -> C17513
- U3: LCSC Part # (none) -> C72114
- X1: footprint Package_DIP:DIP-8_W7.62mm -> Package_DIP:DIP-8_W7.62mm_Socket
Connections:
- net +5V: now also C56.1, J21.3 (Pin_3), R10.1, X2.8 (Vcc)
- net GND: now also C56.2, C57.2, J21.1 (Pin_1), X2.4 (GND); no longer U32.13 (F/~{C})
- net EFI: now reaches U32.14 (EFI)
- net EFI: now also C57.1, X2.5 (OUT)
- new net F/~{C}: J21.2 (Pin_2), R10.2, U32.13 (F/~{C})
Other:
- note added: "8284 Clock/Reset/Ready Generator For 8088 Jumper controls whether DIP oscillator or crystal is used"
- note added: "<=30 MHz Clock (CPU Clock, PCLK)"
- note removed: "8284 Clock/Reset/Ready Generator For 8088"
