File: bus_control.kicad_sch (KiCad schematic)
At the start: 12 parts, among them U12 74LS32, U13 74154, U14 74LS00, U15 74LS32, U34 74154, U8 74LS00

Commit message: bringing over learnings/improvements from prototype board
Parts:
- removed C12, C48: 0.1uF 20% Ceramic, Capacitor_SMD:C_0805_2012Metric, symbol Device:C
- removed U13, U34: 74154, Package_DIP:DIP-24_W7.62mm_Socket, symbol 74xx_IEEE:74154
- removed U14: 74LS00, Package_DIP:DIP-14_W7.62mm_Socket, symbol 74xx:74LS00
- added C49, C50, C51: 0.1uF 20% Ceramic, Capacitor_SMD:C_0805_2012Metric, symbol Device:C
- added U10, U38, U9: 74LS138, Package_DIP:DIP-16_W7.62mm_Socket, symbol 74xx:74LS138
- added U41: 74LS32, Package_DIP:DIP-14_W7.62mm_Socket, symbol 74xx:74LS32
Connections:
- net +5V: now also C49.1, C50.1, C51.1, U10.16 (VCC), U38.16 (VCC), U41.14 (VCC), U9.16 (VCC)
- net 7SEG_CS#: now also U9.7 (O7)
- net A16: now also U38.1 (A0)
- net A17: now also U38.2 (A1)
- net A18: now also U38.3 (A2)
- net A19: now also U38.6 (E3), U41.1
- net A4: now also U10.1 (A0), U9.1 (A0)
- net A5: now also U10.2 (A1), U9.2 (A1)
- net A6: now also U10.3 (A2), U9.3 (A2)
- net A7: now also U10.5 (E2), U9.6 (E3)
- net BIOS_ROM_CS#: now also U38.7 (O7)
- net DMA_CS#: now also U8.6; no longer U8.8
- net DMA_PAGE_CS#: now also U9.15 (O0)
- net GND: now also U8.10, U8.12, U8.13, U8.9, C49.2, C50.2, C51.2, U10.6 (E3), U10.8 (GND), U38.8 (GND), U41.12, U41.13, U41.4, U41.5, U41.7 (GND), U9.5 (E2), U9.8 (GND)
- net IO_0x00_CS#: now also U10.15 (O0)
- net IO_0x10_CS#: now also U8.2, U10.14 (O1); no longer U8.5
- net IO/M#: now also U41.2; no longer U8.12, U8.13
- net PIC_M_CS#: now also U10.13 (O2)
- net PIC_S_CS#: now also U9.13 (O2)
- net PIT_CS#: now also U10.11 (O4)
- net PS2_CS#: now also U10.9 (O6)
- net RAM_CS#: now also U41.3
- net ~{IS_IO}: now also U10.4 (E1), U9.4 (E1)
- net at U8.4: now also U8.3, U8.5; no longer U8.2
- net IO#/M: no longer names the net of U12.12
- net IO#/M: now also U41.8; no longer U8.11
- new net ~{IOR}: U41.9
- new net ~{IOW}: U41.10
- new net ~{MEMR}: U38.5 (E2)
- new net ~{MEMW}: U38.4 (E1)
- no-connect marks 25 -> 19
Other:
- note added: "DMA is 0x00 -> 0x1F AND the demux CS# to get a single CS# (if either/both is 0, CS# will be low, otherwise high)"
- note added: "HIMEM (A19=1) selects: A19 = 1 = BIOS (0x80000...0xFFFFF) 1111 = BIOS ROM (0xF0000...0xFFFFF)"
- note added: "I/O A7 = 0 = 0x00-0x7F"
- note added: "I/O A7 = 1 = 0x80-0xFF"
- note added: "LOMEM (A19=0) selects: A19 = 0 = RAM (0x00000...0x7FFFF)"
- note removed: "DMA is 0x00 -> 0x1F XOR the demux CS# to get a single CS#"
- note removed: "MEM selects: 0000 = RAM (0x00000...0x7FFFF) 1111 = BIOS ROM (0xF0000...0xFFFFF)"
- moved on the sheet: U12D, U8A, U8B, U8C, U8D

Commit message: more pcb routing, implementing learnings from the prototype board
Parts:
- removed C50, C9: 0.1uF 20% Ceramic, Capacitor_SMD:C_0805_2012Metric, symbol Device:C
- removed U10: 74LS138, Package_DIP:DIP-16_W7.62mm_Socket, symbol 74xx:74LS138
- removed U41: 74LS32, Package_DIP:DIP-14_W7.62mm_Socket, symbol 74xx:74LS32
Connections:
- net IO_0x10_CS# is gone; now on net ~{MEM_E000_CS}: U8.2
- net +5V: now also U38.6 (E3), U9.6 (E3)
- net A12+A13+A14+A15: now also U12.13; no longer U12.10
- net A16: now also U8.5; no longer U38.1 (A0)
- net A17: now also U38.1 (A0); no longer U38.2 (A1)
- net A18: now also U38.2 (A1); no longer U38.3 (A2)
- net A19: now also U38.3 (A2); no longer U38.6 (E3)
- net A4: no longer U9.1 (A0)
- net A5: now also U9.1 (A0); no longer U9.2 (A1)
- net A6: now also U9.2 (A1); no longer U9.3 (A2)
- net A7: now also U9.3 (A2); no longer U9.6 (E3)
- net A8+A19+A10+A11: now also U12.12; no longer U12.9
- net BIOS_ROM_CS#: now also U8.6; no longer U38.7 (O7)
- net DMA_CS#: now also U9.15 (O0); no longer U8.6
- net DMA_PAGE_CS#: now also U9.11 (O4); no longer U9.15 (O0)
- net GND: no longer U9.5 (E2)
- net PIC_M_CS#: now also U9.14 (O1)
- net PIC_S_CS#: now also U9.10 (O5); no longer U9.13 (O2)
- net PIT_CS#: now also U9.13 (O2)
- net PS2_CS#: now also U9.12 (O3)
- net ~{A8..15_ZERO}: now also U12.11, U9.5 (E2); no longer U12.13, U12.8
- net ~{IOR}: now also U12.9
- net ~{IOW}: now also U12.10
- net ~{IS_IO}: now also U12.8; no longer U12.11
- net at U8.3, U8.4: no longer U8.5
- net ~{MEM_A000_CS}: now reaches U38.10 (O5)
- net ~{MEM_8000_CS}: now reaches U38.11 (O4)
- net ~{MEM_6000_CS}: now reaches U38.12 (O3)
- net ~{MEM_4000_CS}: now reaches U38.13 (O2)
- net ~{MEM_2000_CS}: now reaches U38.14 (O1)
- net ~{MEM_0000_CS}: now reaches U38.15 (O0)
- net ~{MEM_C000_CS}: now reaches U38.9 (O6)
- net ~{IO_C0_CS}: now reaches U9.9 (O6)
- net IO_0x00_CS# renamed ~{MEM_E000_CS}
- net ~{MEM_E000_CS}: now also U38.7 (O7)
- no-connect marks 19 -> 3
Other:
- note added: "BIOS ROM: ~{E0000_CS} + A16=1 = ~{ROM_CS}"
- note added: "I/O For odd ~{CS}, additional downstream gates required."
- note removed: "DMA is 0x00 -> 0x1F AND the demux CS# to get a single CS# (if either/both is 0, CS# will be low, otherwise high)"
- note removed: "HIMEM (A19=1) selects: A19 = 1 = BIOS (0x80000...0xFFFFF) 1111 = BIOS ROM (0xF0000...0xFFFFF)"
- note removed: "I/O A7 = 0 = 0x00-0x7F"
- note removed: "I/O A7 = 1 = 0x80-0xFF"
- note removed: "LOMEM (A19=0) selects: A19 = 0 = RAM (0x00000...0x7FFFF)"
- moved on the sheet: U12C, U8A, U8B, U8C, U8D

Commit message: pcb is fully routed, working on power capacitor tweaks, some ROM testing
Parts:
- renumbered C51 to C37, C14 to C41, C15 to C42, C49 to C54, C8 to C55, U9 to U21, U12 to U26, U15 to U27, U38 to U35, U8 to U36
Changed lines of the file:
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@@
 		(dnp no)
 		(fields_autoplaced yes)
-		(property "Reference" "C51"
+		(property "Reference" "C37"
 			(at 124.46 52.07 90)
 			(effects
@@
 			(project "sbc_8088"
 				(path "/5e468d94-0319-44d1-a77f-2adc451eed13/8a7a4052-314b-4a01-9fd2-962ecfde1937"
-					(reference "C51")
+					(reference "C37")
 					(unit 1)
 				)
@@
 		(dnp no)
 		(fields_autoplaced yes)
-		(property "Reference" "U12"
+		(property "Reference" "U26"
 			(at 64.135 175.26 0)
 			(effects
@@
 			(project "sbc_8088"
 				(path "/5e468d94-0319-44d1-a77f-2adc451eed13/8a7a4052-314b-4a01-9fd2-962ecfde1937"
-					(reference "U12")
+					(reference "U26")
 					(unit 2)
 				)
@@
 		(on_board yes)
 		(dnp no)
-		(property "Reference" "U8"
+		(property "Reference" "U36"
 			(at 220.9717 98.425 0)
 			(effects
@@
 			(project "sbc_8088"
 				(path "/5e468d94-0319-44d1-a77f-2adc451eed13/8a7a4052-314b-4a01-9fd2-962ecfde1937"
-					(reference "U8")
+					(reference "U36")
 					(unit 1)
 				)
@@
 		(dnp no)
 		(fields_autoplaced yes)
-		(property "Reference" "U12"
+		(property "Reference" "U26"
 			(at 82.55 160.02 0)
 			(effects
@@
 			(project "sbc_8088"
 				(path "/5e468d94-0319-44d1-a77f-2adc451eed13/8a7a4052-314b-4a01-9fd2-962ecfde1937"
-					(reference "U12")
+					(reference "U26")
 					(unit 4)
 				)
@@
 		(dnp no)
 		(fields_autoplaced yes)
-		(property "Reference" "C15"
+		(property "Reference" "C42"
 			(at 165.1 147.32 90)
 			(effects
@@
 			(project "sbc_8088"
 				(path "/5e468d94-0319-44d1-a77f-2adc451eed13/8a7a4052-314b-4a01-9fd2-962ecfde1937"
-					(reference "C15")
+					(reference "C42")
 					(unit 1)
 				)
@@
 		(dnp no)
 		(fields_autoplaced yes)
-		(property "Reference" "U38"
+		(property "Reference" "U35"
 			(at 214.2841 50.8 0)
 			(effects
@@
 			(project "sbc_8088"
 				(path "/5e468d94-0319-44d1-a77f-2adc451eed13/8a7a4052-314b-4a01-9fd2-962ecfde1937"
-					(reference "U38")
+					(reference "U35")
 					(unit 1)
 				)
@@
 		(dnp no)
 		(fields_autoplaced yes)
-		(property "Reference" "U12"
+		(property "Reference" "U26"
 			(at 44.45 74.93 0)
 			(effects
@@
 			(project "sbc_8088"
 				(path "/5e468d94-0319-44d1-a77f-2adc451eed13/8a7a4052-314b-4a01-9fd2-962ecfde1937"
-					(reference "U12")
+					(reference "U26")
 					(unit 3)
 				)
@@
 		(dnp no)
 		(fields_autoplaced yes)
-		(property "Reference" "C14"
+		(property "Reference" "C41"
 			(at 139.7 146.685 90)
 			(effects
@@
 			(project "sbc_8088"
 				(path "/5e468d94-0319-44d1-a77f-2adc451eed13/8a7a4052-314b-4a01-9fd2-962ecfde1937"
-					(reference "C14")
+					(reference "C41")
 					(unit 1)
 				)
@@
 		(dnp no)
 		(fields_autoplaced yes)
-		(property "Reference" "U8"
+		(property "Reference" "U36"
 			(at 269.24 69.85 0)
 			(effects
@@
 			(project "sbc_8088"
 				(path "/5e468d94-0319-44d1-a77f-2adc451eed13/8a7a4052-314b-4a01-9fd2-962ecfde1937"
-					(reference "U8")
+					(reference "U36")
 					(unit 5)
 				)
@@
 		(dnp no)
 		(fields_autoplaced yes)
-		(property "Reference" "U15"
+		(property "Reference" "U27"
 			(at 166.37 167.64 0)
 			(effects
@@
 			(project "sbc_8088"
 				(path "/5e468d94-0319-44d1-a77f-2adc451eed13/8a7a4052-314b-4a01-9fd2-962ecfde1937"
-					(reference "U15")
+					(reference "U27")
 					(unit 5)
 				)
@@
 		(dnp no)
 		(fields_autoplaced yes)
-		(property "Reference" "U15"
+		(property "Reference" "U27"
 			(at 41.91 169.545 0)
 			(effects
@@
 			(project "sbc_8088"
 				(path "/5e468d94-0319-44d1-a77f-2adc451eed13/8a7a4052-314b-4a01-9fd2-962ecfde1937"
-					(reference "U15")
+					(reference "U27")
 					(unit 4)
 				)
@@
 		(dnp no)
 		(fields_autoplaced yes)
-		(property "Reference" "U9"
+		(property "Reference" "U21"
 			(at 121.5741 64.77 0)
 			(effects
@@
 			(project "sbc_8088"
 				(path "/5e468d94-0319-44d1-a77f-2adc451eed13/8a7a4052-314b-4a01-9fd2-962ecfde1937"
-					(reference "U9")
+					(reference "U21")
 					(unit 1)
 				)
@@
 		(dnp no)
 		(fields_autoplaced yes)
-		(property "Reference" "U12"
+		(property "Reference" "U26"
 			(at 64.135 147.955 0)
 			(effects
@@
 			(project "sbc_8088"
 				(path "/5e468d94-0319-44d1-a77f-2adc451eed13/8a7a4052-314b-4a01-9fd2-962ecfde1937"
-					(reference "U12")
+					(reference "U26")
 					(unit 1)
 				)
@@
 		(dnp no)
 		(fields_autoplaced yes)
-		(property "Reference" "U12"
+		(property "Reference" "U26"
 			(at 141.605 167.64 0)
 			(effects
@@
 			(project "sbc_8088"
 				(path "/5e468d94-0319-44d1-a77f-2adc451eed13/8a7a4052-314b-4a01-9fd2-962ecfde1937"
-					(reference "U12")
+					(reference "U26")
 					(unit 5)
 				)
@@
 		(dnp no)
 		(fields_autoplaced yes)
-		(property "Reference" "U8"
+		(property "Reference" "U36"
 			(at 265.4217 128.27 0)
 			(effects
@@
 			(project "sbc_8088"
 				(path "/5e468d94-0319-44d1-a77f-2adc451eed13/8a7a4052-314b-4a01-9fd2-962ecfde1937"
-					(reference "U8")
+					(reference "U36")
 					(unit 4)
 				)
@@
 		(dnp no)
 		(fields_autoplaced yes)
-		(property "Reference" "U15"
+		(property "Reference" "U27"
 			(at 41.91 141.605 0)
 			(effects
@@
 			(project "sbc_8088"
 				(path "/5e468d94-0319-44d1-a77f-2adc451eed13/8a7a4052-314b-4a01-9fd2-962ecfde1937"
-					(reference "U15")
+					(reference "U27")
 					(unit 1)
 				)
@@
 		(on_board yes)
 		(dnp no)
-		(property "Reference" "U8"
+		(property "Reference" "U36"
 			(at 245.1017 128.905 0)
 			(effects
@@
 			(project "sbc_8088"
 				(path "/5e468d94-0319-44d1-a77f-2adc451eed13/8a7a4052-314b-4a01-9fd2-962ecfde1937"
-					(reference "U8")
+					(reference "U36")
 					(unit 3)
 				)
@@
 		(dnp no)
 		(fields_autoplaced yes)
-		(property "Reference" "C8"
+		(property "Reference" "C55"
 			(at 267.97 49.53 90)
 			(effects
@@
 			(project "sbc_8088"
 				(path "/5e468d94-0319-44d1-a77f-2adc451eed13/8a7a4052-314b-4a01-9fd2-962ecfde1937"
-					(reference "C8")
+					(reference "C55")
 					(unit 1)
 				)
@@
 		(dnp no)
 		(fields_autoplaced yes)
-		(property "Reference" "C49"
+		(property "Reference" "C54"
 			(at 217.17 38.1 90)
 			(effects
@@
 			(project "sbc_8088"
 				(path "/5e468d94-0319-44d1-a77f-2adc451eed13/8a7a4052-314b-4a01-9fd2-962ecfde1937"
-					(reference "C49")
+					(reference "C54")
 					(unit 1)
 				)
@@
 		(dnp no)
 		(fields_autoplaced yes)
-		(property "Reference" "U15"
+		(property "Reference" "U27"
 			(at 41.91 182.88 0)
 			(effects
@@
 			(project "sbc_8088"
 				(path "/5e468d94-0319-44d1-a77f-2adc451eed13/8a7a4052-314b-4a01-9fd2-962ecfde1937"
-					(reference "U15")
+					(reference "U27")
 					(unit 3)
 				)
@@
 		(dnp no)
 		(fields_autoplaced yes)
-		(property "Reference" "U15"
+		(property "Reference" "U27"
 			(at 41.91 155.575 0)
 			(effects
@@
 			(project "sbc_8088"
 				(path "/5e468d94-0319-44d1-a77f-2adc451eed13/8a7a4052-314b-4a01-9fd2-962ecfde1937"
-					(reference "U15")
+					(reference "U27")
 					(unit 2)
 				)
@@
 		(dnp no)
 		(fields_autoplaced yes)
-		(property "Reference" "U8"
+		(property "Reference" "U36"
 			(at 248.9117 104.14 0)
 			(effects
@@
 			(project "sbc_8088"
 				(path "/5e468d94-0319-44d1-a77f-2adc451eed13/8a7a4052-314b-4a01-9fd2-962ecfde1937"
-					(reference "U8")
+					(reference "U36")
 					(unit 2)
 				)

Commit message: added ATtiny for SMC, added PC speaker
Parts:
- added J9: BIOS ROM Bypass, Connector_PinHeader_2.54mm:PinHeader_1x02_P2.54mm_Vertical, symbol Connector_Generic:Conn_01x02
- renumbered C37 to C42, C41 to C46, C42 to C47, C54 to C60, C55 to C61, U21 to U24, U26 to U30, U27 to U31, U35 to U40, U36 to U41
Connections:
- net BIOS_ROM_CS#: now also J9.1 (Pin_1); no longer U41.6
- net GND: no longer U41.10, U41.12, U41.13, U41.9
- net PS2_CS#: now also U41.10, U41.9
- net ~{PPI_CS}: now reaches U41.11
- net at U41.8: now also U41.12
- new net: J9.2 (Pin_2), U41.6
- new net A0: U41.13
- no-connect marks 3 -> 1
Other:
- note added: "PPI (0x61): ~{IO_60_CS} + A0=1 = ~{PPI_CS}"
- moved on the sheet: U41C, U41D

Commit message: tweaks and fixes from real hardware testing
Parts:
- added C69: 0.1uF 20% Ceramic, Capacitor_SMD:C_0805_2012Metric, symbol Device:C
- added U42: 74LS08, Package_DIP:DIP-14_W7.62mm_Socket, symbol 74xx:74LS08
Connections:
- net ~{MEMR} is gone; now on net GND: U40.5 (E2)
- net ~{MEMW} is gone; now on net GND: U40.4 (E1)
- net +5V: now also C69.1, U42.14 (VCC); no longer U40.6 (E3)
- net GND: now also U30.10, U30.9, C69.2, U42.10, U42.12, U42.13, U42.4, U42.5, U42.7 (GND), U42.9
- net ~{IOR}: now also U42.1; no longer U30.9
- net ~{IOW}: now also U42.2; no longer U30.10
- net ~{IS_IO}: now also U40.6 (E3), U42.3; no longer U30.8
- no-connect marks 1 -> 5
Other:
- note added: "TODO: fix this, it's meant to be ~{IOW} AND ~{IOR} = ~{IS_IO}"
- note added: "TODO: fix this, use ~{IS_IO} as the active-high E3, bridge E2/E1 to GND"
- moved on the sheet: U30C

Commit message: schematic fixes for DMA HRQ, DMA active cycle
Connections:
- net +5V: now also U40.6 (E3); no longer U24.6 (E3)
- net GND: no longer U40.4 (E1), U42.4, U42.5
- net ~{IS_IO}: no longer U40.6 (E3)
- net ~{IS_MEM}: now reaches U42.6
- net ~{IS_MEM}: now also U40.4 (E1)
- new net ~{DMA_AEN}: U24.6 (E3)
- new net ~{MEMR}: U42.4
- new net ~{MEMW}: U42.5
- no-connect marks 5 -> 4
Other:
- note added: "TODO: during DMA active cycle, ~{IOR} and ~{MEMW} will both be LO Need to NOT chip-select I/O devices during that phase. But need to chip-select MEM devices during that phase (so ~{IS_IO} can't be used active-high to enable the MEM select chip...)"
- note added: "When DMA AEN=HI, this will be LO and disable local I/O decode; DMA lowers ~{IOR} in active cycle."
- note removed: "TODO: fix this, it's meant to be ~{IOW} AND ~{IOR} = ~{IS_IO}"
- moved on the sheet: U42B
