File: bus_control.kicad_sch (KiCad schematic)
At the start: 13 parts, among them J9 BIOS ROM Bypass, U24 74LS138, U30 74LS32, U31 74LS32, U40 74LS138, U41 74LS00, U42 74LS08

Commit message: fix KBC/PPI CS# schematic bugs, add ISA expansion header for adding more cards
Parts:
- added C72: 0.1uF 20% Ceramic, Capacitor_SMD:C_0805_2012Metric, symbol Device:C
- added U45: 74LS138, Package_DIP:DIP-16_W7.62mm_Socket, symbol 74xx:74LS138
Connections:
- net DMA_PAGE_CS# is gone; now on net 7SEG_CS#: U24.11 (O4)
- net +5V: now also C72.1, U45.16 (VCC)
- net 7SEG_CS#: no longer U24.7 (O7)
- net A0: now also U45.1 (A0); no longer U41.13
- net A4: now also U41.10, U41.9
- net GND: now also U41.12, U41.13, C72.2, U45.8 (GND); no longer U42.10, U42.9
- net PS2_CS#: now also U42.8; no longer U24.12 (O3), U41.10, U41.9
- net ~{PPI_CS}: now also U45.14 (O1); no longer U41.11
- net at U41.8: now also U45.6 (E3); no longer U41.12
- new net A1: U45.2 (A1)
- new net A2: U45.3 (A2)
- new net A3: U45.5 (E2)
- new net ~{IO_60_CS}: U24.12 (O3), U45.4 (E1)
- new net ~{IO_DMUX_CS_60}: U42.9, U45.15 (O0)
- new net ~{IO_DMUX_CS_62}: U45.13 (O2)
- new net ~{IO_DMUX_CS_63}: U45.12 (O3)
- new net ~{IO_DMUX_CS_64}: U42.10, U45.11 (O4)
- new net ~{IO_DMUX_CS_65}: U45.10 (O5)
- new net ~{IO_DMUX_CS_66}: U45.9 (O6)
- new net ~{IO_DMUX_CS_67}: U45.7 (O7)
- new net ~{IO_E0_CS}: U24.7 (O7)
- no-connect marks 4 -> 10
Other:
- note added: "Demux for 0x60-0x6F range (A4=0) Ignores 0x69-0x6F (where A3=1)"
- note removed: "PPI (0x61): ~{IO_60_CS} + A0=1 = ~{PPI_CS}"
- note removed: "TODO: during DMA active cycle, ~{IOR} and ~{MEMW} will both be LO Need to NOT chip-select I/O devices during that phase. But need to chip-select MEM devices during that phase (so ~{IS_IO} can't be used active-high to enable the MEM select chip...)"
- note removed: "TODO: fix this, use ~{IS_IO} as the active-high E3, bridge E2/E1 to GND"
- moved on the sheet: U41C, U41D, U42C

Commit message: fixes, prep for final production run
Parts:
- removed J9: BIOS ROM Bypass, Connector_PinHeader_2.54mm:PinHeader_1x02_P2.54mm_Vertical, symbol Connector_Generic:Conn_01x02
- C42, C46, C47, C60, C61, C69, C72: LCSC Part # (none) -> C1853649
- U24, U40, U45: LCSC Part # (none) -> C72115
- U30, U31, U41, U42: LCSC Part # (none) -> C72114
Connections:
- net BIOS_ROM_CS#: now also U41.6

Commit message: routing tweaks, use identity comparator instead of OR gates for IO decode
Parts:
- removed C46, C47: 0.1uF 20% Ceramic, Capacitor_SMD:C_0805_2012Metric, symbol Device:C
- removed U30, U31: 74LS32, Package_DIP:DIP-14_W7.62mm_Socket, symbol 74xx:74LS32
- added C76: 0.1uF 20% Ceramic, Capacitor_SMD:C_0805_2012Metric, symbol Device:C
- added U3: 74LS688 OR 74F521, Package_DIP:DIP-20_W7.62mm_Socket, symbol 74xx:74LS688
Connections:
- net +5V: now also C76.1, U3.20 (VCC)
- net A10: now also U3.6 (P2)
- net A11: now also U3.8 (P3)
- net A12: now also U3.11 (P4)
- net A13: now also U3.13 (P5)
- net A14: now also U3.15 (P6)
- net A15: now also U3.17 (P7)
- net A8: now also U3.2 (P0)
- net A9: now also U3.4 (P1)
- net GND: now also C76.2, U3.1 (G), U3.10 (GND), U3.12 (R4), U3.14 (R5), U3.16 (R6), U3.18 (R7), U3.3 (R0), U3.5 (R1), U3.7 (R2), U3.9 (R3)
- net ~{A8..15_ZERO}: now also U3.19 (P=R)
- no-connect marks 10 -> 9
Other:
- note added: "We don't respond to I/O ports >= 0x100 (devices on the ISA bus can though) Comparator ensures A8..15 are all zero to enforce this."
- note removed: "We don't respond to I/O ports >= 0x100 (devices on the ISA bus can though) These OR gates ensure we never chip select those."

Commit message: add i2c bus with expansion card sockets
Connections:
- net ~{IO_E0_CS} renamed I2C_CS#
- no-connect marks 9 -> 8
Changed lines of the file:
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@@
-	)
-	(no_connect
-		(at 151.13 90.17)
 	)
 	(no_connect
@@
 		(fields_autoplaced yes)
 		(effects
+			(font
+				(size 1.27 1.27)
+			)
+			(justify left)
+		)
+	)
+	(hierarchical_label "I2C_CS#"
+		(shape output)
+		(at 151.13 90.17 0)
+		(fields_autoplaced yes)
+		(effects

Commit message: no more SMT for isa_i2c, tweak motherboard multiplex logic, handful of other tweaks
Parts:
- removed U41: 74LS00, Package_DIP:DIP-14_W7.62mm_Socket, symbol 74xx:74LS00
- added C24, C44: 0.1uF 20% Ceramic, Capacitor_SMD:C_0805_2012Metric, symbol Device:C
- added U11: 74LS138, Package_DIP:DIP-16_W7.62mm_Socket, symbol 74xx:74LS138
- added U18: 74AHC1GU04, Package_TO_SOT_SMD:SOT-23-5, symbol 74xGxx:74AHC1GU04
- added U25: 74AHC1G08, Package_TO_SOT_SMD:SOT-23-5, symbol 74xGxx:74AHC1G08
Connections:
- net +5V: now also C24.1, C44.1, U11.16 (VCC), U18.5 (VCC), U25.5 (VCC)
- net A16: now also U11.1 (A0)
- net A17: now also U11.2 (A1)
- net A18: now also U11.3 (A2)
- net A19: now also U11.6 (E3)
- net A4: now also U18.2
- net BIOS_ROM_CS#: now also U11.7 (O7)
- net GND: now also U42.10, U42.9, C24.2, C44.2, U11.5 (E2), U11.8 (GND), U18.3 (GND), U25.3 (GND)
- net PS2_CS#: now also U25.4; no longer U42.8
- net ~{IO_DMUX_CS_60}: now also U25.1; no longer U42.9
- net ~{IO_DMUX_CS_64}: now also U25.2; no longer U42.10
- net ~{IS_MEM}: now also U11.4 (E1)
- net ~{MEM_A000_CS}: now also U11.13 (O2); no longer U40.10 (O5)
- net ~{MEM_C000_CS}: now also U11.11 (O4); no longer U40.9 (O6)
- net ~{MEM_E000_CS}: now also U11.9 (O6); no longer U40.7 (O7)
- net !A4: now reaches U45.6 (E3)
- net !A4: now also U18.4
- new net ~{MEM_B000_CS}: U11.12 (O3)
- new net ~{MEM_D000_CS}: U11.10 (O5)
- no-connect marks 8 -> 13
Other:
- note added: "Conventional mem decode (0x00000 -> 0xA0000)"
- note added: "Upper memory decode (0x80000 -> 0x100000)"
- note removed: "BIOS ROM: ~{E0000_CS} + A16=1 = ~{ROM_CS}"
- moved on the sheet: C42, C60, C61, C69, C72, U42C, U42D, U42E

Commit message: simplify m88 logic further, reduce ICs, reorient the POST display, use an oscillator for 14.31818 MHz, update isa-i2c bridge BOM
Parts:
- removed C44, C61, C76: 0.1uF 20% Ceramic, Capacitor_SMD:C_0805_2012Metric, symbol Device:C
- removed U18: 74AHC1GU04, Package_TO_SOT_SMD:SOT-23-5, symbol 74xGxx:74AHC1GU04
- removed U25: 74AHC1G08, Package_TO_SOT_SMD:SOT-23-5, symbol 74xGxx:74AHC1G08
- removed U3: 74LS688 OR 74F521, Package_DIP:DIP-20_W7.62mm_Socket, symbol 74xx:74LS688
Connections:
- net !A4 is gone; now on net +5V: U45.6 (E3)
- net A3 is gone; now on net A4: U45.5 (E2)
- net ~{A8..15_ZERO} is gone; now on net A8: U24.5 (E2)
- net ~{IOR} is gone; now on net ~{IO_DMUX_CS_60}: U42.1
- net ~{IOW} is gone; now on net ~{IO_DMUX_CS_64}: U42.2
- net ~{MEMR} is gone; now on net GND: U42.4
- net ~{MEMW} is gone; now on net GND: U42.5
- net A9: now also U24.4 (E1)
- net GND: now also U11.4 (E1), U40.4 (E1)
- net PS2_CS#: now also U42.3
- net UMA_9000: now reaches U11.14 (O1)
- net UMA_8000: now reaches U11.15 (O0)
- removed net ~{IS_IO}: U24.4 (E1), U42.3
- removed net ~{IS_MEM}: U11.4 (E1), U40.4 (E1), U42.6
- no-connect marks 13 -> 14
Other:
- note added: "Conventional mem decode (0x00000 -> 0xA0000) in 128K blocks"
- note added: "Demux for 0x60-0x6F range (A4=0) Does not decode A3 to simplify the circuit, so the range is duplicated: e.g. 0x60 == 0x68, 0x64 == 0x6C"
- note added: "IO selects: 0x00-0x1F = DMA = A4..15 all zeroes 0x20-0x21 = PIC #1 = A5 one, rest zeroes 0x40-0x47 = PIT = A6 one, rest zeroes 0x60-0x64 = PS/2 controller = A6, A5 one, rest zeroes 0x80 = 7-Seg POST digit display = A7 one, rest zeroes 0x81-0x8F = DMA page registers = A7 one, rest zeroes 0xA0-0xA1 = PIC #2 = A7 one, A5 one, rest zeroes Check A9..A0 - 10 bits for I/O addr decode"
- note added: "Upper memory decode (0x80000 -> 0x100000) in 64K blocks"
- note removed: "Conventional mem decode (0x00000 -> 0xA0000)"
- note removed: "Demux for 0x60-0x6F range (A4=0) Ignores 0x69-0x6F (where A3=1)"
- note removed: "IO selects: 0x00-0x1F = DMA = A4..15 all zeroes 0x20-0x21 = PIC #1 = A5 one, rest zeroes 0x40-0x47 = PIT = A6 one, rest zeroes 0x60-0x64 = PS/2 controller = A6, A5 one, rest zeroes 0x80-0x8F = DMA page registers = A7 one, rest zeroes 0xA0-0xA1 = PIC #2 = A7 one, A5 one, rest zeroes 0xF0-0xF1 = POST 7-segment (4 bit BCD) check A15..A4 (12 bits), ignore lower 4 bits"
- note removed: "Upper memory decode (0x80000 -> 0x100000)"
- note removed: "We don't respond to I/O ports >= 0x100 (devices on the ISA bus can though) Comparator ensures A8..15 are all zero to enforce this."
- moved on the sheet: C24, C42, C60, U11, U24, U40, U42A, U42B, U42C, U42D
