File: bus_control.kicad_sch (KiCad schematic)
At the start: 10 parts, among them U11 74LS138, U24 74LS138, U40 74LS138, U42 74LS08, U45 74LS138

Commit message: motherboard tweaks for manufacturing run, i2c card tweaks for manufacturing run, de9 -> stemma adapter idea for the i2c card
Parts:
- C24, C42, C60, C69, C72: LCSC Part # C1853649 -> C49678
Changed lines of the file:
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@@
 			)
 		)
-		(property "Description" "LCSC #C1853649"
+		(property "Description" "LCSC #C49678"
 			(at 252.73 49.53 0)
 			(effects
@@
 			)
 		)
-		(property "LCSC Part #" "C1853649"
+		(property "LCSC Part #" "C49678"
 			(at 252.73 49.53 0)
 			(effects
@@
 			)
 		)
-		(property "Description" "LCSC #C1853649"
+		(property "Description" "LCSC #C49678"
 			(at 356.87 45.72 0)
 			(effects
@@
 			)
 		)
-		(property "LCSC Part #" "C1853649"
+		(property "LCSC Part #" "C49678"
 			(at 356.87 45.72 0)
 			(effects
@@
 			)
 		)
-		(property "Description" "LCSC #C1853649"
+		(property "Description" "LCSC #C49678"
 			(at 73.66 191.77 0)
 			(effects
@@
 			)
 		)
-		(property "LCSC Part #" "C1853649"
+		(property "LCSC Part #" "C49678"
 			(at 73.66 191.77 0)
 			(effects
@@
 			)
 		)
-		(property "Description" "LCSC #C1853649"
+		(property "Description" "LCSC #C49678"
 			(at 389.89 135.89 0)
 			(effects
@@
 			)
 		)
-		(property "LCSC Part #" "C1853649"
+		(property "LCSC Part #" "C49678"
 			(at 389.89 135.89 0)
 			(effects
@@
 			)
 		)
-		(property "Description" "LCSC #C1853649"
+		(property "Description" "LCSC #C49678"
 			(at 73.66 121.92 0)
 			(effects
@@
 			)
 		)
-		(property "LCSC Part #" "C1853649"
+		(property "LCSC Part #" "C49678"
 			(at 73.66 121.92 0)
 			(effects
