File: dma.kicad_sch (KiCad schematic)
At the start: 11 parts, among them U2 74LS670, U21 74LS04, U22 8237 DMA CONTROLLER, U23 74LS573, U29 74LS244

Commit message: bringing over learnings/improvements from prototype board
Parts:
- added NT1, NT2, NT3, NT4: NetTie_2, NetTie:NetTie-2_SMD_Pad0.5mm, symbol Device:NetTie_2
- added R1: 10k, Resistor_SMD:R_0805_2012Metric, symbol Device:R_US
Connections:
- net +5V: now also R1.2
- net A0: now also NT1.2; no longer U22.32 (A0), U29.2 (I0a)
- net A1: now also NT2.2; no longer U22.33 (A1), U29.4 (I1a)
- net A10: now also U23.14 (Q5); no longer U23.17 (Q2)
- net A11: now also U23.15 (Q4); no longer U23.19 (Q0)
- net A12: now also U23.16 (Q3); no longer U23.18 (Q1)
- net A13: now also U23.17 (Q2); no longer U23.16 (Q3)
- net A14: now also U23.18 (Q1); no longer U23.14 (Q5)
- net A15: now also U23.19 (Q0); no longer U23.12 (Q7)
- net A2: now also NT3.2; no longer U22.34 (A2), U29.6 (I2a)
- net A3: now also NT4.2; no longer U22.35 (A3), U29.8 (I3a)
- net A4: no longer U22.37 (A4), U29.11 (I0b)
- net A5: no longer U22.38 (A5), U29.13 (I1b)
- net A6: no longer U22.39 (A6), U29.15 (I2b)
- net A7: no longer U22.40 (A7), U29.17 (I3b)
- net A8: now also U23.12 (Q7); no longer U23.13 (Q6)
- net A9: now also U23.13 (Q6); no longer U23.15 (Q4)
- net D0: now also U23.9 (D7); no longer U23.8 (D6)
- net D1: now also U23.8 (D6); no longer U23.6 (D4)
- net D2: now also U23.7 (D5); no longer U23.4 (D2)
- net D3: now also U23.6 (D4); no longer U23.2 (D0)
- net D4: now also U23.5 (D3); no longer U23.3 (D1)
- net D5: now also U23.4 (D2); no longer U23.5 (D3)
- net D6: now also U23.3 (D1); no longer U23.7 (D5)
- net D7: now also U23.2 (D0); no longer U23.9 (D7)
- net HRQ: now also R1.1
- new net DMA_A0: NT1.1, U22.32 (A0), U29.2 (I0a)
- new net DMA_A1: NT2.1, U22.33 (A1), U29.4 (I1a)
- new net DMA_A2: NT3.1, U22.34 (A2), U29.6 (I2a)
- new net DMA_A3: NT4.1, U22.35 (A3), U29.8 (I3a)
- new net DMA_A4: U22.37 (A4), U29.11 (I0b)
- new net DMA_A5: U22.38 (A5), U29.13 (I1b)
- new net DMA_A6: U22.39 (A6), U29.15 (I2b)
- new net DMA_A7: U22.40 (A7), U29.17 (I3b)
Other:
- note removed: "Pin ordering optimized for PCB layout"

Commit message: more pcb routing, implementing learnings from the prototype board
Parts:
- removed R1: 10k, Resistor_SMD:R_0805_2012Metric, symbol Device:R_US
- added C9: 0.1uF 20% Ceramic, Capacitor_SMD:C_0805_2012Metric, symbol Device:C_Small
- added U10: 74LS74, Package_DIP:DIP-14_W7.62mm_Socket, symbol 74xx:74LS74
Connections:
- net +5V: now also C9.1, U10.10 (~{S}), U10.11 (C), U10.12 (D), U10.13 (~{R}), U10.14 (VCC)
- net CLK: now also U10.3 (C)
- net GND: now also C9.2, U10.4 (~{S}), U10.7 (GND)
- net HRQ: now also U10.5 (Q); no longer U22.10 (HRQ)
- net RESET: now also U10.1 (~{R})
- new net: U10.2 (D), U22.10 (HRQ)
- no-connect marks 0 -> 3
Other:
- note added: "8237 runs on an inverted CLK Pass HRQ through flip/flop to ensure it crosses the clock domain successfully"

Commit message: pcb is fully routed, working on power capacitor tweaks, some ROM testing
Parts:
- renumbered C22 to C15, C23 to C16, C24 to C31, C10 to C36, C9 to C4, C45 to C6, R32 to R5, U21 to U16, U29 to U2, U2 to U22, U10 to U3, U23 to U5, U22 to U7
Changed lines of the file:
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@@
 		(dnp no)
 		(fields_autoplaced yes)
-		(property "Reference" "U22"
+		(property "Reference" "U7"
 			(at 152.0541 137.16 0)
 			(effects
@@
 			(project "sbc_8088"
 				(path "/5e468d94-0319-44d1-a77f-2adc451eed13/b83b9fc0-04c9-48b0-9c67-1dac6abe53f7"
-					(reference "U22")
+					(reference "U7")
 					(unit 1)
 				)
@@
 		(dnp no)
 		(fields_autoplaced yes)
-		(property "Reference" "U21"
+		(property "Reference" "U16"
 			(at 267.97 141.605 0)
 			(effects
@@
 			(project "sbc_8088"
 				(path "/5e468d94-0319-44d1-a77f-2adc451eed13/b83b9fc0-04c9-48b0-9c67-1dac6abe53f7"
-					(reference "U21")
+					(reference "U16")
 					(unit 7)
 				)
@@
 		(dnp no)
 		(fields_autoplaced yes)
-		(property "Reference" "U21"
+		(property "Reference" "U16"
 			(at 111.76 73.66 0)
 			(effects
@@
 			(project "sbc_8088"
 				(path "/5e468d94-0319-44d1-a77f-2adc451eed13/b83b9fc0-04c9-48b0-9c67-1dac6abe53f7"
-					(reference "U21")
+					(reference "U16")
 					(unit 3)
 				)
@@
 		(dnp no)
 		(fields_autoplaced yes)
-		(property "Reference" "C22"
+		(property "Reference" "C15"
 			(at 156.2163 45.72 90)
 			(effects
@@
 			(project "sbc_8088"
 				(path "/5e468d94-0319-44d1-a77f-2adc451eed13/b83b9fc0-04c9-48b0-9c67-1dac6abe53f7"
-					(reference "C22")
+					(reference "C15")
 					(unit 1)
 				)
@@
 		(dnp no)
 		(fields_autoplaced yes)
-		(property "Reference" "U21"
+		(property "Reference" "U16"
 			(at 76.2 57.15 0)
 			(effects
@@
 			(project "sbc_8088"
 				(path "/5e468d94-0319-44d1-a77f-2adc451eed13/b83b9fc0-04c9-48b0-9c67-1dac6abe53f7"
-					(reference "U21")
+					(reference "U16")
 					(unit 1)
 				)
@@
 		(dnp no)
 		(fields_autoplaced yes)
-		(property "Reference" "C23"
+		(property "Reference" "C16"
 			(at 81.2863 107.95 90)
 			(effects
@@
 			(project "sbc_8088"
 				(path "/5e468d94-0319-44d1-a77f-2adc451eed13/b83b9fc0-04c9-48b0-9c67-1dac6abe53f7"
-					(reference "C23")
+					(reference "C16")
 					(unit 1)
 				)
@@
 		(dnp no)
 		(fields_autoplaced yes)
-		(property "Reference" "C24"
+		(property "Reference" "C31"
 			(at 266.0713 122.555 90)
 			(effects
@@
 			(project "sbc_8088"
 				(path "/5e468d94-0319-44d1-a77f-2adc451eed13/b83b9fc0-04c9-48b0-9c67-1dac6abe53f7"
-					(reference "C24")
+					(reference "C31")
 					(unit 1)
 				)
@@
 		(dnp no)
 		(fields_autoplaced yes)
-		(property "Reference" "U21"
+		(property "Reference" "U16"
 			(at 41.275 142.875 0)
 			(effects
@@
 			(project "sbc_8088"
 				(path "/5e468d94-0319-44d1-a77f-2adc451eed13/b83b9fc0-04c9-48b0-9c67-1dac6abe53f7"
-					(reference "U21")
+					(reference "U16")
 					(unit 2)
 				)
@@
 		(dnp no)
 		(fields_autoplaced yes)
-		(property "Reference" "R32"
+		(property "Reference" "R5"
 			(at 189.865 144.78 0)
 			(effects
@@
 			(project "sbc_8088"
 				(path "/5e468d94-0319-44d1-a77f-2adc451eed13/b83b9fc0-04c9-48b0-9c67-1dac6abe53f7"
-					(reference "R32")
+					(reference "R5")
 					(unit 1)
 				)
@@
 		(dnp no)
 		(fields_autoplaced yes)
-		(property "Reference" "U29"
+		(property "Reference" "U2"
 			(at 237.1441 93.98 0)
 			(effects
@@
 			(project "sbc_8088"
 				(path "/5e468d94-0319-44d1-a77f-2adc451eed13/b83b9fc0-04c9-48b0-9c67-1dac6abe53f7"
-					(reference "U29")
+					(reference "U2")
 					(unit 1)
 				)
@@
 		(dnp no)
 		(fields_autoplaced yes)
-		(property "Reference" "U10"
+		(property "Reference" "U3"
 			(at 111.4141 163.83 0)
 			(effects
@@
 			(project "sbc_8088"
 				(path "/5e468d94-0319-44d1-a77f-2adc451eed13/b83b9fc0-04c9-48b0-9c67-1dac6abe53f7"
-					(reference "U10")
+					(reference "U3")
 					(unit 2)
 				)
@@
 		(dnp no)
 		(fields_autoplaced yes)
-		(property "Reference" "C9"
+		(property "Reference" "C4"
 			(at 50.8063 161.925 90)
 			(effects
@@
 			(project "sbc_8088"
 				(path "/5e468d94-0319-44d1-a77f-2adc451eed13/b83b9fc0-04c9-48b0-9c67-1dac6abe53f7"
-					(reference "C9")
+					(reference "C4")
 					(unit 1)
 				)
@@
 		(dnp no)
 		(fields_autoplaced yes)
-		(property "Reference" "U23"
+		(property "Reference" "U5"
 			(at 77.1241 118.11 0)
 			(effects
@@
 			(project "sbc_8088"
 				(path "/5e468d94-0319-44d1-a77f-2adc451eed13/b83b9fc0-04c9-48b0-9c67-1dac6abe53f7"
-					(reference "U23")
+					(reference "U5")
 					(unit 1)
 				)
@@
 		(dnp no)
 		(fields_autoplaced yes)
-		(property "Reference" "U21"
+		(property "Reference" "U16"
 			(at 205.74 142.24 0)
 			(effects
@@
 			(project "sbc_8088"
 				(path "/5e468d94-0319-44d1-a77f-2adc451eed13/b83b9fc0-04c9-48b0-9c67-1dac6abe53f7"
-					(reference "U21")
+					(reference "U16")
 					(unit 6)
 				)
@@
 		(dnp no)
 		(fields_autoplaced yes)
-		(property "Reference" "U10"
+		(property "Reference" "U3"
 			(at 50.8 181.6099 0)
 			(effects
@@
 			(project "sbc_8088"
 				(path "/5e468d94-0319-44d1-a77f-2adc451eed13/b83b9fc0-04c9-48b0-9c67-1dac6abe53f7"
-					(reference "U10")
+					(reference "U3")
 					(unit 3)
 				)
@@
 		(dnp no)
 		(fields_autoplaced yes)
-		(property "Reference" "U10"
+		(property "Reference" "U3"
 			(at 200.3141 72.39 0)
 			(effects
@@
 			(project "sbc_8088"
 				(path "/5e468d94-0319-44d1-a77f-2adc451eed13/b83b9fc0-04c9-48b0-9c67-1dac6abe53f7"
-					(reference "U10")
+					(reference "U3")
 					(unit 1)
 				)
@@
 		(dnp no)
 		(fields_autoplaced yes)
-		(property "Reference" "U2"
+		(property "Reference" "U22"
 			(at 242.2241 30.48 0)
 			(effects
@@
 			(project "sbc_8088"
 				(path "/5e468d94-0319-44d1-a77f-2adc451eed13/b83b9fc0-04c9-48b0-9c67-1dac6abe53f7"
-					(reference "U2")
+					(reference "U22")
 					(unit 1)
 				)
@@
 		(dnp no)
 		(fields_autoplaced yes)
-		(property "Reference" "C45"
+		(property "Reference" "C6"
 			(at 240.0363 85.09 90)
 			(effects
@@
 			(project "sbc_8088"
 				(path "/5e468d94-0319-44d1-a77f-2adc451eed13/b83b9fc0-04c9-48b0-9c67-1dac6abe53f7"
-					(reference "C45")
+					(reference "C6")
 					(unit 1)
 				)
@@
 		(dnp no)
 		(fields_autoplaced yes)
-		(property "Reference" "C10"
+		(property "Reference" "C36"
 			(at 246.3863 19.685 90)
 			(effects
@@
 			(project "sbc_8088"
 				(path "/5e468d94-0319-44d1-a77f-2adc451eed13/b83b9fc0-04c9-48b0-9c67-1dac6abe53f7"
-					(reference "C10")
+					(reference "C36")
 					(unit 1)
 				)

Commit message: added ATtiny for SMC, added PC speaker
Parts:
- renumbered C4 to C2, C31 to C36, C36 to C41, R5 to R9, U3 to U1, U16 to U18, U22 to U25, U2 to U3, U7 to U8
Changed lines of the file:
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@@
 		(dnp no)
 		(fields_autoplaced yes)
-		(property "Reference" "U7"
+		(property "Reference" "U8"
 			(at 152.0541 137.16 0)
 			(effects
@@
 			(project "sbc_8088"
 				(path "/5e468d94-0319-44d1-a77f-2adc451eed13/b83b9fc0-04c9-48b0-9c67-1dac6abe53f7"
-					(reference "U7")
+					(reference "U8")
 					(unit 1)
 				)
@@
 		(dnp no)
 		(fields_autoplaced yes)
-		(property "Reference" "U16"
+		(property "Reference" "U18"
 			(at 267.97 141.605 0)
 			(effects
@@
 			(project "sbc_8088"
 				(path "/5e468d94-0319-44d1-a77f-2adc451eed13/b83b9fc0-04c9-48b0-9c67-1dac6abe53f7"
-					(reference "U16")
+					(reference "U18")
 					(unit 7)
 				)
@@
 		(dnp no)
 		(fields_autoplaced yes)
-		(property "Reference" "U16"
+		(property "Reference" "U18"
 			(at 111.76 73.66 0)
 			(effects
@@
 			(project "sbc_8088"
 				(path "/5e468d94-0319-44d1-a77f-2adc451eed13/b83b9fc0-04c9-48b0-9c67-1dac6abe53f7"
-					(reference "U16")
+					(reference "U18")
 					(unit 3)
 				)
@@
 		(dnp no)
 		(fields_autoplaced yes)
-		(property "Reference" "U16"
+		(property "Reference" "U18"
 			(at 76.2 57.15 0)
 			(effects
@@
 			(project "sbc_8088"
 				(path "/5e468d94-0319-44d1-a77f-2adc451eed13/b83b9fc0-04c9-48b0-9c67-1dac6abe53f7"
-					(reference "U16")
+					(reference "U18")
 					(unit 1)
 				)
@@
 		(dnp no)
 		(fields_autoplaced yes)
-		(property "Reference" "C31"
+		(property "Reference" "C36"
 			(at 266.0713 122.555 90)
 			(effects
@@
 			(project "sbc_8088"
 				(path "/5e468d94-0319-44d1-a77f-2adc451eed13/b83b9fc0-04c9-48b0-9c67-1dac6abe53f7"
-					(reference "C31")
+					(reference "C36")
 					(unit 1)
 				)
@@
 		(dnp no)
 		(fields_autoplaced yes)
-		(property "Reference" "U16"
+		(property "Reference" "U18"
 			(at 41.275 142.875 0)
 			(effects
@@
 			(project "sbc_8088"
 				(path "/5e468d94-0319-44d1-a77f-2adc451eed13/b83b9fc0-04c9-48b0-9c67-1dac6abe53f7"
-					(reference "U16")
+					(reference "U18")
 					(unit 2)
 				)
@@
 		(dnp no)
 		(fields_autoplaced yes)
-		(property "Reference" "R5"
+		(property "Reference" "R9"
 			(at 189.865 144.78 0)
 			(effects
@@
 			(project "sbc_8088"
 				(path "/5e468d94-0319-44d1-a77f-2adc451eed13/b83b9fc0-04c9-48b0-9c67-1dac6abe53f7"
-					(reference "R5")
+					(reference "R9")
 					(unit 1)
 				)
@@
 		(dnp no)
 		(fields_autoplaced yes)
-		(property "Reference" "U2"
+		(property "Reference" "U3"
 			(at 237.1441 93.98 0)
 			(effects
@@
 			(project "sbc_8088"
 				(path "/5e468d94-0319-44d1-a77f-2adc451eed13/b83b9fc0-04c9-48b0-9c67-1dac6abe53f7"
-					(reference "U2")
+					(reference "U3")
 					(unit 1)
 				)
@@
 		(dnp no)
 		(fields_autoplaced yes)
-		(property "Reference" "U3"
+		(property "Reference" "U1"
 			(at 111.4141 163.83 0)
 			(effects
@@
 			(project "sbc_8088"
 				(path "/5e468d94-0319-44d1-a77f-2adc451eed13/b83b9fc0-04c9-48b0-9c67-1dac6abe53f7"
-					(reference "U3")
+					(reference "U1")
 					(unit 2)
 				)
@@
 		(dnp no)
 		(fields_autoplaced yes)
-		(property "Reference" "C4"
+		(property "Reference" "C2"
 			(at 50.8063 161.925 90)
 			(effects
@@
 			(project "sbc_8088"
 				(path "/5e468d94-0319-44d1-a77f-2adc451eed13/b83b9fc0-04c9-48b0-9c67-1dac6abe53f7"
-					(reference "C4")
+					(reference "C2")
 					(unit 1)
 				)
@@
 		(dnp no)
 		(fields_autoplaced yes)
-		(property "Reference" "U16"
+		(property "Reference" "U18"
 			(at 205.74 142.24 0)
 			(effects
@@
 			(project "sbc_8088"
 				(path "/5e468d94-0319-44d1-a77f-2adc451eed13/b83b9fc0-04c9-48b0-9c67-1dac6abe53f7"
-					(reference "U16")
+					(reference "U18")
 					(unit 6)
 				)
@@
 		(dnp no)
 		(fields_autoplaced yes)
-		(property "Reference" "U3"
+		(property "Reference" "U1"
 			(at 50.8 181.6099 0)
 			(effects
@@
 			(project "sbc_8088"
 				(path "/5e468d94-0319-44d1-a77f-2adc451eed13/b83b9fc0-04c9-48b0-9c67-1dac6abe53f7"
-					(reference "U3")
+					(reference "U1")
 					(unit 3)
 				)
@@
 		(dnp no)
 		(fields_autoplaced yes)
-		(property "Reference" "U3"
+		(property "Reference" "U1"
 			(at 200.3141 72.39 0)
 			(effects
@@
 			(project "sbc_8088"
 				(path "/5e468d94-0319-44d1-a77f-2adc451eed13/b83b9fc0-04c9-48b0-9c67-1dac6abe53f7"
-					(reference "U3")
+					(reference "U1")
 					(unit 1)
 				)
@@
 		(dnp no)
 		(fields_autoplaced yes)
-		(property "Reference" "U22"
+		(property "Reference" "U25"
 			(at 242.2241 30.48 0)
 			(effects
@@
 			(project "sbc_8088"
 				(path "/5e468d94-0319-44d1-a77f-2adc451eed13/b83b9fc0-04c9-48b0-9c67-1dac6abe53f7"
-					(reference "U22")
+					(reference "U25")
 					(unit 1)
 				)
@@
 		(dnp no)
 		(fields_autoplaced yes)
-		(property "Reference" "C36"
+		(property "Reference" "C41"
 			(at 246.3863 19.685 90)
 			(effects
@@
 			(project "sbc_8088"
 				(path "/5e468d94-0319-44d1-a77f-2adc451eed13/b83b9fc0-04c9-48b0-9c67-1dac6abe53f7"
-					(reference "C36")
+					(reference "C41")
 					(unit 1)
 				)

Commit message: fix a few schematic bugs, missing pull-ups and pull-downs in particular
Parts:
- added R40: 10k, Resistor_SMD:R_0805_2012Metric, symbol Device:R_US
Connections:
- net AEN: now also R40.1
- net GND: now also R40.2
Changed lines of the file:
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@@
 	(wire
 		(pts
+			(xy 142.24 162.56) (xy 142.24 167.64)
+		)
+		(stroke
+			(width 0)
+			(type default)
+		)
+	)
+	(wire
+		(pts
 			(xy 242.57 91.44) (xy 247.65 91.44)
 		)
@@
 	(wire
 		(pts
+			(xy 142.24 175.26) (xy 142.24 179.07)
+		)
+		(stroke
+			(width 0)
+			(type default)
+		)
+	)
+	(wire
+		(pts
 			(xy 132.08 113.03) (xy 127 113.03)
 		)
@@
 		)
 	)
+	(label "AEN"
+		(at 142.24 162.56 270)
+		(fields_autoplaced yes)
+		(effects
+			(font
+				(size 1.27 1.27)
+			)
+			(justify right bottom)
+		)
+	)
 	(label "A19"
 		(at 262.89 45.72 180)
@@
 	)
 	(symbol
+		(lib_id "power:GND")
+		(at 142.24 179.07 0)
+		(unit 1)
+		(exclude_from_sim no)
+		(in_bom yes)
+		(on_board yes)
+		(dnp no)
+		(fields_autoplaced yes)
+		(property "Reference" "#PWR0328"
+			(at 142.24 185.42 0)
+			(effects
+				(font
+					(size 1.27 1.27)
+				)
+				(hide yes)
+			)
+		)
+		(property "Value" "GND"
+			(at 142.24 184.15 0)
+			(effects
+				(font
+					(size 1.27 1.27)
+				)
+			)
+		)
+		(property "Footprint" ""
+			(at 142.24 179.07 0)
+			(effects
+				(font
+					(size 1.27 1.27)
+				)
+				(hide yes)
+			)
+		)
+		(property "Datasheet" ""
+			(at 142.24 179.07 0)
+			(effects
+				(font
+					(size 1.27 1.27)
+				)
+				(hide yes)
+			)
+		)
+		(property "Description" ""
+			(at 142.24 179.07 0)
+			(effects
+				(font
+					(size 1.27 1.27)
+				)
+				(hide yes)
+			)
+		)
+		(pin "1"
+		)
+		(instances
+			(project "sbc_8088"
+				(path "/5e468d94-0319-44d1-a77f-2adc451eed13/b83b9fc0-04c9-48b0-9c67-1dac6abe53f7"
+					(reference "#PWR0328")
+					(unit 1)
+				)
+			)
+		)
+	)
+	(symbol
 		(lib_id "power:+5V")
 		(at 74.93 111.125 0)
@@
 				)
 			)
+		)
+	)
+	(symbol
+		(lib_id "Device:R_US")
+		(at 142.24 171.45 0)
+		(unit 1)
+		(exclude_from_sim no)
+		(in_bom yes)
+		(on_board yes)
+		(dnp no)
+		(fields_autoplaced yes)
+		(property "Reference" "R40"
+			(at 144.78 170.1799 0)
+			(effects
+				(font
+					(size 1.27 1.27)
+				)
+				(justify left)
+			)
+		)
+		(property "Value" "10k"
+			(at 144.78 172.7199 0)
+			(effects
+				(font
+					(size 1.27 1.27)
+				)
+				(justify left)
+			)
+		)
+		(property "Footprint" "Resistor_SMD:R_0805_2012Metric"
+			(at 143.256 171.704 90)
+			(effects
+				(font
+					(size 1.27 1.27)
+				)
+				(hide yes)
+			)
+		)
+		(property "Datasheet" "~"
+			(at 142.24 171.45 0)
+			(effects
+				(font
+					(size 1.27 1.27)
+				)
+				(hide yes)
+			)
+		)
+		(property "Description" ""
+			(at 142.24 171.45 0)
+			(effects
+				(font
+					(size 1.27 1.27)
+				)
+				(hide yes)
+			)
+		)
+		(pin "2"
+		)
+		(pin "1"
+		)
+		(instances
+			(project "sbc_8088"
+				(path "/5e468d94-0319-44d1-a77f-2adc451eed13/b83b9fc0-04c9-48b0-9c67-1dac6abe53f7"
+					(reference "R40")
+					(unit 1)
+				)
+			)

Commit message: schematic fixes for DMA HRQ, DMA active cycle
Connections:
- net +5V: now also U1.4 (~{S})
- net GND: no longer U1.4 (~{S})
- net RESET: no longer U1.1 (~{R})
- new net ~{RESET}: U1.1 (~{R})
Changed lines of the file:
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@@
 		)
 	)
-	(wire
-		(pts
-			(xy 187.96 69.85) (xy 198.12 69.85)
-		)
-		(stroke
-			(width 0)
-			(type default)
-		)
-	)
 	(bus
 		(pts
@@
 	(wire
 		(pts
-			(xy 198.12 69.85) (xy 198.12 74.93)
+			(xy 198.12 72.39) (xy 198.12 74.93)
 		)
 		(stroke
@@
 	(wire
 		(pts
-			(xy 187.96 69.85) (xy 187.96 71.12)
-		)
-		(stroke
-			(width 0)
-			(type default)
-		)
-	)
-	(wire
-		(pts
 			(xy 149.86 138.43) (xy 149.86 143.51)
 		)
@@
 		)
 	)
+	(wire
+		(pts
+			(xy 127 21.59) (xy 138.43 21.59)
+		)
+		(stroke
+			(width 0)
+			(type default)
+		)
+	)
 	(bus
 		(pts
@@
 		)
 	)
+	(label "~{DMA_AEN}"
+		(at 127 21.59 0)
+		(fields_autoplaced yes)
+		(effects
+			(font
+				(size 1.27 1.27)
+			)
+			(justify left bottom)
+		)
+	)
 	(label "DREQ1"
 		(at 123.825 97.79 0)
@@
 		)
 	)
+	(hierarchical_label "~{DMA_AEN}"
+		(shape input)
+		(at 138.43 21.59 0)
+		(fields_autoplaced yes)
+		(effects
+			(font
+				(size 1.27 1.27)
+			)
+			(justify left)
+		)
+	)
 	(hierarchical_label "DREQ[0..3]"
 		(shape input)
@@
 		)
 	)
-	(hierarchical_label "RESET"
+	(hierarchical_label "~{RESET}"
 		(shape input)
 		(at 194.31 92.71 180)
@@
 	)
 	(symbol
-		(lib_id "power:GND")
-		(at 187.96 71.12 0)
-		(unit 1)
-		(exclude_from_sim no)
-		(in_bom yes)
-		(on_board yes)
-		(dnp no)
-		(fields_autoplaced yes)
-		(property "Reference" "#PWR0215"
-			(at 187.96 77.47 0)
-			(effects
-				(font
-					(size 1.27 1.27)
-				)
-				(hide yes)
-			)
-		)
-		(property "Value" "GND"
-			(at 187.96 76.2 0)
-			(effects
-				(font
-					(size 1.27 1.27)
-				)
-			)
-		)
-		(property "Footprint" ""
-			(at 187.96 71.12 0)
-			(effects
-				(font
-					(size 1.27 1.27)
-				)
-				(hide yes)
-			)
-		)
-		(property "Datasheet" ""
-			(at 187.96 71.12 0)
-			(effects
-				(font
-					(size 1.27 1.27)
-				)
-				(hide yes)
-			)
-		)
-		(property "Description" ""
-			(at 187.96 71.12 0)
-			(effects
-				(font
-					(size 1.27 1.27)
-				)
-				(hide yes)
-			)
-		)
-		(pin "1"
-		)
-		(instances
-			(project "sbc_8088"
-				(path "/5e468d94-0319-44d1-a77f-2adc451eed13/b83b9fc0-04c9-48b0-9c67-1dac6abe53f7"
-					(reference "#PWR0215")
-					(unit 1)
-				)
-			)
-		)
-	)
-	(symbol
 		(lib_id "Device:C_Small")
 		(at 156.21 52.07 90)
@@
 				)
 			)
+		)
+	)
+	(symbol
+		(lib_id "power:+5V")
+		(at 198.12 72.39 0)
+		(unit 1)
+		(exclude_from_sim no)
+		(in_bom yes)
+		(on_board yes)
+		(dnp no)
+		(fields_autoplaced yes)
+		(property "Reference" "#PWR0215"
+			(at 198.12 76.2 0)
+			(effects
+				(font
+					(size 1.27 1.27)
+				)
+				(hide yes)
+			)
+		)
+		(property "Value" "+5V"
+			(at 198.12 67.31 0)
+			(effects
+				(font
+					(size 1.27 1.27)
+				)
+			)
+		)
+		(property "Footprint" ""
+			(at 198.12 72.39 0)
+			(effects
+				(font
+					(size 1.27 1.27)
+				)
+				(hide yes)
+			)
+		)
+		(property "Datasheet" ""
+			(at 198.12 72.39 0)
+			(effects
+				(font
+					(size 1.27 1.27)
+				)
+				(hide yes)
+			)
+		)
+		(property "Description" ""
+			(at 198.12 72.39 0)
+			(effects
+				(font
+					(size 1.27 1.27)
+				)
+				(hide yes)
+			)
+		)
+		(pin "1"
+		)
+		(instances
+			(project "sbc_8088"
+				(path "/5e468d94-0319-44d1-a77f-2adc451eed13/b83b9fc0-04c9-48b0-9c67-1dac6abe53f7"
+					(reference "#PWR0215")
+					(unit 1)
+				)
+			)
