File: sbc_8088.kicad_sch (KiCad schematic)
At the start: 5 parts, among them U1 8088

Commit message: bringing over learnings/improvements from prototype board
Parts:
- removed R2, R3, R4: 10k, Resistor_SMD:R_0805_2012Metric, symbol Device:R_US
Connections:
- net 8088_MN/~{MX} is gone; now on net +5V: U1.33 (MN/~{MX})
- net 8088_TEST# is gone; now on net GND: U1.23 (~{TEST})
Other:
- sheet Bus Controller ports: added ~{MEMR}, ~{MEMW}; removed none

Commit message: more pcb routing, implementing learnings from the prototype board
Connections:
- no-connect marks 3 -> 7
Other:
- sheet Bus Controller ports: added ~{IOR}, ~{IOW}, ~{MEM_0000_CS}, ~{MEM_2000_CS}, ~{MEM_4000_CS}, ~{MEM_6000_CS}, ~{MEM_8000_CS}, ~{MEM_A000_CS}, ~{MEM_C000_CS}, ~{MEM_E000_CS}; removed RAM_CS#, ~{BUSEN}
- sheet RAM ports: added ~{RAM_A_CS}, ~{RAM_B_CS}, ~{RAM_C_CS}, ~{RAM_D_CS}; removed ~{RAM_CS}

Commit message: more pcb routing
Changed lines of the file:
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@@
 		)
 	)
-	(label "IRQ[2..7]"
+	(label "IR[2..7]"
 		(at 74.93 124.46 180)
 		(fields_autoplaced yes)

Commit message: pcb is fully routed, working on power capacitor tweaks, some ROM testing
Parts:
- added R4: 10k, Resistor_SMD:R_0805_2012Metric, symbol Device:R_US
- renumbered C1 to C19, U1 to U6
Connections:
- net +5V: now also R4.1
- net 8088_INTA#: now also R4.2
Other:
- added sheet Real Time Clock (RTC.kicad_sch)
- added sheet Serial Port (serial_port.kicad_sch)
- sheet KB Controller ports: added KBC_CLK; removed 8MHz
- note added: "8088 Single-Board Computer"
- note added: "A1"
- note added: "Give KBC A2 instead of A0 I/O ports 0x60, 0x64"
- note added: "Make sure ~{INTA} can never float"
- note added: "TODO: Add DS1687-5+ for RTC TODO: Add something for RS323 and/or FTDI serial"

Commit message: added ATtiny for SMC, added PC speaker
Parts:
- renumbered C19 to C22, R4 to R8, U6 to U7
Connections:
- no-connect marks 7 -> 6
Other:
- removed sheet Real Time Clock
- removed sheet Serial Port
- added sheet Intel PPI (Emulation) (ppi.kicad_sch)
- added sheet System Management Controller (smc.kicad_sch)
- sheet Bus Controller ports: added ~{PPI_CS}; removed none
- sheet Buttons & Mounting ports: added FP_PWR_SWITCH; removed none
- sheet Power Management ports: added ~{PS_ON}; removed none
- note added: "2x 7-segment digits I/O 0xF0, two 4-bit BCD integers"
- note removed: "8088 Single-Board Computer"
- note removed: "A1"
- note removed: "TODO: Add DS1687-5+ for RTC TODO: Add something for RS323 and/or FTDI serial"
- moved on the sheet: R8

Commit message: fix a few schematic bugs, missing pull-ups and pull-downs in particular
Parts:
- added R39: 10k, Resistor_SMD:R_0805_2012Metric, symbol Device:R_US
Connections:
- net 8088_HLDA: now also R39.1
- net GND: now also R39.2
Changed lines of the file:
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@@
 	(wire
 		(pts
+			(xy 227.33 243.84) (xy 227.33 259.08)
+		)
+		(stroke
+			(width 0)
+			(type default)
+		)
+	)
+	(wire
+		(pts
 			(xy 53.34 87.63) (xy 57.15 87.63)
 		)
@@
 	(wire
 		(pts
+			(xy 227.33 266.7) (xy 227.33 274.32)
+		)
+		(stroke
+			(width 0)
+			(type default)
+		)
+	)
+	(wire
+		(pts
 			(xy 115.57 100.33) (xy 127 100.33)
 		)
@@
 		)
 	)
+	(label "8088_HLDA"
+		(at 227.33 243.84 270)
+		(fields_autoplaced yes)
+		(effects
+			(font
+				(size 1.27 1.27)
+			)
+			(justify right bottom)
+		)
+	)
 	(label "SPKR_GATE"
 		(at 116.84 215.9 0)
@@
 	)
 	(symbol
+		(lib_id "Device:R_US")
+		(at 227.33 262.89 0)
+		(unit 1)
+		(exclude_from_sim no)
+		(in_bom yes)
+		(on_board yes)
+		(dnp no)
+		(fields_autoplaced yes)
+		(property "Reference" "R39"
+			(at 229.87 261.6199 0)
+			(effects
+				(font
+					(size 1.27 1.27)
+				)
+				(justify left)
+			)
+		)
+		(property "Value" "10k"
+			(at 229.87 264.1599 0)
+			(effects
+				(font
+					(size 1.27 1.27)
+				)
+				(justify left)
+			)
+		)
+		(property "Footprint" "Resistor_SMD:R_0805_2012Metric"
+			(at 228.346 263.144 90)
+			(effects
+				(font
+					(size 1.27 1.27)
+				)
+				(hide yes)
+			)
+		)
+		(property "Datasheet" "~"
+			(at 227.33 262.89 0)
+			(effects
+				(font
+					(size 1.27 1.27)
+				)
+				(hide yes)
+			)
+		)
+		(property "Description" ""
+			(at 227.33 262.89 0)
+			(effects
+				(font
+					(size 1.27 1.27)
+				)
+				(hide yes)
+			)
+		)
+		(pin "2"
+		)
+		(pin "1"
+		)
+		(instances
+			(project "sbc_8088"
+				(path "/5e468d94-0319-44d1-a77f-2adc451eed13"
+					(reference "R39")
+					(unit 1)
+				)
+			)
+		)
+	)
+	(symbol
 		(lib_id "power:GND")
 		(at 387.35 107.95 0)
@@
 					(unit 1)
 				)
+			)
+		)
+	)
+	(symbol
+		(lib_id "power:GND")
+		(at 227.33 274.32 0)
+		(unit 1)
+		(exclude_from_sim no)
+		(in_bom yes)
+		(on_board yes)
+		(dnp no)
+		(fields_autoplaced yes)
+		(property "Reference" "#PWR0327"
+			(at 227.33 280.67 0)
+			(effects
+				(font
+					(size 1.27 1.27)
+				)
+				(hide yes)
+			)
+		)
+		(property "Value" "GND"
+			(at 227.33 279.4 0)
+			(effects
+				(font
+					(size 1.27 1.27)
+				)
+			)
+		)
+		(property "Footprint" ""
+			(at 227.33 274.32 0)
+			(effects
+				(font
+					(size 1.27 1.27)
+				)
+				(hide yes)
+			)
+		)
+		(property "Datasheet" ""
+			(at 227.33 274.32 0)
+			(effects
+				(font
+					(size 1.27 1.27)
+				)
+				(hide yes)
+			)
+		)
+		(property "Description" ""
+			(at 227.33 274.32 0)
+			(effects
+				(font
+					(size 1.27 1.27)
+				)
+				(hide yes)
+			)
+		)
+		(pin "1"
+		)
+		(instances
+			(project "sbc_8088"
+				(path "/5e468d94-0319-44d1-a77f-2adc451eed13"
+					(reference "#PWR0327")
+					(unit 1)
+				)

Commit message: schematic fixes for DMA HRQ, DMA active cycle
Other:
- sheet Bus Controller ports: added ~{DMA_AEN}; removed none
- sheet DMA Controller ports: added ~{DMA_AEN}, ~{RESET}; removed none
