File: sbc_8088.kicad_sch (KiCad schematic)
At the start: 4 parts, among them U7 8088

Commit message: fix KBC/PPI CS# schematic bugs, add ISA expansion header for adding more cards
Connections:
- no-connect marks 6 -> 5
Other:
- sheet RAM ports: added ~{RAM_E_CS}; removed none
Changed lines of the file:
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@@
 	)
 	(no_connect
-		(at 270.51 50.8)
-	)
-	(no_connect
 		(at 21.59 210.82)
 	)
@@
 	(wire
 		(pts
+			(xy 344.17 157.48) (xy 356.87 157.48)
+		)
+		(stroke
+			(width 0)
+			(type default)
+		)
+	)
+	(wire
+		(pts
 			(xy 34.29 166.37) (xy 34.29 167.64)
 		)
@@
 	(wire
 		(pts
+			(xy 283.21 50.8) (xy 270.51 50.8)
+		)
+		(stroke
+			(width 0)
+			(type default)
+		)
+	)
+	(wire
+		(pts
 			(xy 189.23 261.62) (xy 189.23 273.05)
 		)
@@
 		)
 	)
+	(label "~{RAM_E_CS}"
+		(at 344.17 157.48 0)
+		(fields_autoplaced yes)
+		(effects
+			(font
+				(size 1.27 1.27)
+			)
+			(justify left bottom)
+		)
+	)
 	(label "~{DMA_AEN}"
 		(at 278.13 129.54 180)
@@
 		)
 	)
+	(label "~{RAM_E_CS}"
+		(at 283.21 50.8 180)
+		(fields_autoplaced yes)
+		(effects
+			(font
+				(size 1.27 1.27)
+			)
+			(justify right bottom)
+		)
+	)
 	(label "8088_MN{slash}~{MX}"
 		(at 208.28 273.05 180)
@@
 	(sheet
 		(at 356.87 127)
-		(size 25.4 29.21)
+		(size 25.4 34.29)
 		(fields_autoplaced yes)
 		(stroke
@@
 		)
 		(property "Sheetfile" "ram.kicad_sch"
-			(at 356.87 156.7946 0)
+			(at 356.87 161.8746 0)
 			(effects
 				(font
@@
 			(effects
 				(font
+					(size 1.27 1.27)
+				)
+				(justify left)
+			)
+		)
+		(pin "~{RAM_E_CS}" input
+			(at 356.87 157.48 180)
+			(effects
+				(font

Commit message: add discharge resistors for all power rails
Changed lines of the file:
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@@
-	)
-	(junction
-		(at 25.4 264.16)
-		(diameter 0)
-		(color 0 0 0 0)
-	)
-	(junction
-		(at 25.4 260.35)
-		(diameter 0)
-		(color 0 0 0 0)
-	)
-	(junction
-		(at 25.4 261.62)
-		(diameter 0)
-		(color 0 0 0 0)
 	)
 	(junction
@@
 	)
 	(junction
-		(at 22.86 260.35)
-		(diameter 0)
-		(color 0 0 0 0)
-	)
-	(junction
 		(at 57.15 87.63)
 		(diameter 0)
@@
 	(wire
 		(pts
-			(xy 22.86 261.62) (xy 25.4 261.62)
-		)
-		(stroke
-			(width 0)
-			(type default)
-		)
-	)
-	(wire
-		(pts
 			(xy 144.78 40.64) (xy 144.78 43.18)
 		)
@@
 	(wire
 		(pts
-			(xy 25.4 261.62) (xy 29.21 261.62)
-		)
-		(stroke
-			(width 0)
-			(type default)
-		)
-	)
-	(wire
-		(pts
 			(xy 162.56 102.87) (xy 173.99 102.87)
 		)
@@
 	(wire
 		(pts
-			(xy 29.21 264.16) (xy 25.4 264.16)
-		)
-		(stroke
-			(width 0)
-			(type default)
-		)
-	)
-	(wire
-		(pts
 			(xy 281.94 227.33) (xy 285.75 227.33)
 		)
@@
 	(wire
 		(pts
-			(xy 22.86 260.35) (xy 22.86 261.62)
-		)
-		(stroke
-			(width 0)
-			(type default)
-		)
-	)
-	(wire
-		(pts
 			(xy 170.18 214.63) (xy 170.18 217.17)
 		)
@@
 		)
 		(stroke
-			(width 0)
-			(type default)
-		)
-	)
-	(wire
-		(pts
-			(xy 25.4 260.35) (xy 25.4 261.62)
-		)
-		(stroke

Commit message: working on removing DMA for now
Parts:
- added R40, R45, R46, R48, R9: 10k, Resistor_SMD:R_0805_2012Metric, symbol Device:R_US
Connections:
- net +5V: now also R48.1, R9.2; no longer U7.33 (MN/~{MX})
- net 8088_HOLD: now also R40.1
- net GND: now also R40.2, R45.2, R46.2; no longer U7.23 (~{TEST}), U7.34 (~{SSO})
- net ~{DMA_AEN}: now also R9.1
- new net 8088_MN/~{MX}: R48.2, U7.33 (MN/~{MX})
- new net 8088_SSO#: R45.1, U7.34 (~{SSO})
- new net 8088_TEST#: R46.1, U7.23 (~{TEST})
- no-connect marks 5 -> 7
Other:
- removed sheet DMA Controller
- sheet Intel PPI (Emulation) ports: added none; removed A0
- note added: "Removing DMA Controller for now. Pull all DMA signals accordingly."

Commit message: fixes, prep for final production run
Parts:
- C22: LCSC Part # (none) -> C1853649
- R39, R40, R45, R46, R48, R8, R9: LCSC Part # (none) -> C84376
- U7: LCSC Part # (none) -> C72123
Other:
- sheet Clock Generator ports: added ISA_OSC; removed none
- note added: "ISA CLK sits at CPU speed (8 MHz) ISA OSC runs at standard 14.318 MHz"

Commit message: add i2c bus with expansion card sockets
Other:
- added sheet I2C Bus (i2c.kicad_sch)
- sheet Bus Controller ports: added I2C_CS#; removed none

Commit message: no more SMT for isa_i2c, tweak motherboard multiplex logic, handful of other tweaks
Connections:
- no-connect marks 7 -> 9
Other:
- sheet Bus Controller ports: added ~{MEM_B000_CS}, ~{MEM_D000_CS}; removed none
- sheet Interrupt Controller ports: added none; removed S_CS#
- sheet POST 7-Segment ports: added ~{IOR}; removed none
- sheet RAM ports: added ~{RAM_UMA_CS}; removed none

Commit message: simplify m88 logic further, reduce ICs, reorient the POST display, use an oscillator for 14.31818 MHz, update isa-i2c bridge BOM
Parts:
- removed R45, R48: 10k, Resistor_SMD:R_0805_2012Metric, symbol Device:R_US
Connections:
- net 8088_MN/~{MX} is gone; now on net +5V: U7.33 (MN/~{MX})
- net 8088_SSO# is gone; now on net GND: U7.34 (~{SSO})
