File: sbc_8088.kicad_sch (KiCad schematic)
At the start: 7 parts, among them U7 8088

Commit message: motherboard tweaks for manufacturing run, i2c card tweaks for manufacturing run, de9 -> stemma adapter idea for the i2c card
Parts:
- C22: LCSC Part # C1853649 -> C49678
- R39, R40, R46, R8, R9: LCSC Part # C84376 -> C17414
Changed lines of the file:
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@@
 			)
 		)
-		(property "Description" "LCSC #C1853649"
+		(property "Description" "LCSC #C49678"
 			(at 154.94 43.18 0)
 			(effects
@@
 			)
 		)
-		(property "LCSC Part #" "C1853649"
+		(property "LCSC Part #" "C49678"
 			(at 154.94 43.18 0)
 			(effects
@@
 			)
 		)
-		(property "Description" "LCSC #C84376"
+		(property "Description" "LCSC #C17414"
 			(at 227.33 262.89 0)
 			(effects
@@
 			)
 		)
-		(property "LCSC Part #" "C84376 "
+		(property "LCSC Part #" "C17414"
 			(at 227.33 262.89 0)
 			(effects
@@
 			)
 		)
-		(property "Description" "LCSC #C84376"
+		(property "Description" "LCSC #C17414"
 			(at 138.43 264.16 0)
 			(effects
@@
 			)
 		)
-		(property "LCSC Part #" "C84376 "
+		(property "LCSC Part #" "C17414"
 			(at 138.43 264.16 0)
 			(effects
@@
 			)
 		)
-		(property "Description" "LCSC #C84376"
+		(property "Description" "LCSC #C17414"
 			(at 267.97 139.7 0)
 			(effects
@@
 			)
 		)
-		(property "LCSC Part #" "C84376 "
+		(property "LCSC Part #" "C17414"
 			(at 267.97 139.7 0)
 			(effects
@@
 			)
 		)
-		(property "Description" "LCSC #C84376"
+		(property "Description" "LCSC #C17414"
 			(at 163.83 260.35 0)
 			(effects
@@
 			)
 		)
-		(property "LCSC Part #" "C84376 "
+		(property "LCSC Part #" "C17414"
 			(at 163.83 260.35 0)
 			(effects
@@
 			)
 		)
-		(property "Description" "LCSC #C84376"
+		(property "Description" "LCSC #C17414"
 			(at 267.97 130.81 0)
 			(effects
@@
 			)
 		)
-		(property "LCSC Part #" "C84376 "
+		(property "LCSC Part #" "C17414"
 			(at 267.97 130.81 0)
 			(effects
