File: sbc_power.kicad_sch (KiCad schematic)
At the start: 15 parts, among them J3 ATX-24

Commit message: bringing over learnings/improvements from prototype board
Parts:
- removed C32: 100 uF 20% 35V Electrolytic, Capacitor_SMD:CP_Elec_6.3x7.7, symbol Device:C_Polarized_Small_US
- added C52, C53, C54: 100 uF 20% 35V Electrolytic, Capacitor_SMD:CP_Elec_5x5.8, symbol Device:C_Polarized_Small_US
- C30: value 10 uF 20% 10V Electrolytic -> 100 uF 20% 35V Electrolytic; footprint Capacitor_SMD:CP_Elec_6.3x7.7 -> Capacitor_SMD:CP_Elec_5x5.8
- C31, C39: footprint Capacitor_SMD:CP_Elec_6.3x7.7 -> Capacitor_SMD:CP_Elec_5x5.8
Connections:
- net +12V: now also C54.1; no longer C31.1
- net +5V: now also C52.1, C53.1
- net -12V: now also C31.2
- net GND: now also C31.1, C52.2, C53.2, C54.2; no longer C31.2

Commit message: more pcb routing, implementing learnings from the prototype board
Parts:
- removed C52, C53: 100 uF 20% 35V Electrolytic, Capacitor_SMD:CP_Elec_5x5.8, symbol Device:C_Polarized_Small_US
- added F2: Bourns MF-RHT200 2A hold, Fuse:Fuse_Bourns_MF-RHT200, symbol Device:Fuse
- added F3, F4: Bourns MF-RHT100 1A hold, Fuse:Fuse_Bourns_MF-RHT100, symbol Device:Fuse
Connections:
- net +12V: now also F4.2; no longer J3.10 (+12V), J3.11 (+12V)
- net +5V: now also F2.2; no longer J3.21 (+5V), J3.22 (+5V), J3.23 (+5V), J3.4 (+5V), J3.6 (+5V)
- net -12V: now also F3.2; no longer J3.14 (-12V)
- new net +12V_IN: F4.1, J3.10 (+12V), J3.11 (+12V)
- new net +5V_IN: F2.1, J3.21 (+5V), J3.22 (+5V), J3.23 (+5V), J3.4 (+5V), J3.6 (+5V)
- new net -12V_IN: F3.1, J3.14 (-12V)
Other:
- moved on the sheet: C31, C39, C54

Commit message: pcb is fully routed, working on power capacitor tweaks, some ROM testing
Parts:
- added C1, C12, C13, C17, C18, C20, C24, C26, C43, C44, C45: 4.7UF 16V 20%, Capacitor_SMD:CP_Elec_4x4.5, symbol Device:C_Polarized_Small_US
- C56: renamed from C31; value 100 uF 20% 35V Electrolytic -> 470 uF 20% 35V Electrolytic; footprint Capacitor_SMD:CP_Elec_5x5.8 -> Capacitor_SMD:CP_Elec_6.3x7.7
- C57: renamed from C39; value 100 uF 20% 35V Electrolytic -> 470 uF 20% 35V Electrolytic; footprint Capacitor_SMD:CP_Elec_5x5.8 -> Capacitor_SMD:CP_Elec_6.3x7.7
- C58: renamed from C54; value 100 uF 20% 35V Electrolytic -> 470 uF 20% 35V Electrolytic; footprint Capacitor_SMD:CP_Elec_5x5.8 -> Capacitor_SMD:CP_Elec_6.3x7.7
- C59: renamed from C30; footprint Capacitor_SMD:CP_Elec_5x5.8 -> Capacitor_SMD:CP_Elec_6.3x7.7
- renumbered F3 to F2, F2 to F3, J3 to J6, R65 to R11, TP2 to TP1, TP7 to TP2, TP6 to TP3, TP3 to TP4, TP8 to TP5, TP4 to TP6, TP5 to TP7, TP1 to TP8
Connections:
- net +5V: now also C1.1, C12.1, C13.1, C17.1, C18.1, C20.1, C24.1, C26.1, C43.1, C44.1, C45.1
- net GND: now also C1.2, C12.2, C13.2, C17.2, C18.2, C20.2, C24.2, C26.2, C43.2, C44.2, C45.2
Other:
- note added: "Distributed capacitance to be spread across the PCB Use smaller caps e.g. Nichicon UZT1E4R7MCL1GB"

Commit message: added ATtiny for SMC, added PC speaker
Parts:
- removed C56: 470 uF 20% 35V Electrolytic, Capacitor_SMD:CP_Elec_6.3x7.7, symbol Device:C_Polarized_Small_US
- removed S1: TL2230EEF140, SamacSys_Parts:TL2230OAF140, symbol SamacSys_Parts:TL2230EEF140
- added C63, C67: 470 uF 20% 35V Electrolytic, Capacitor_SMD:CP_Elec_6.3x7.7, symbol Device:C_Polarized_Small_US
- added TP8: TestPoint, Connector_PinHeader_2.54mm:PinHeader_1x01_P2.54mm_Vertical, symbol Connector:TestPoint
- renumbered C17 to C18, C26 to C19, C18 to C21, C20 to C23, C24 to C27, C43 to C48, C45 to C49, C44 to C50, C57 to C64, C58 to C65, C59 to C66, J6 to J10, R11 to R34, TP8 to TP1, TP3 to TP2, TP1 to TP3, TP2 to TP4, TP4 to TP5, TP5 to TP6, TP6 to TP7, TP7 to TP9
Connections:
- net +5V: now also C63.1, C67.1
- net +5V_IN: now also TP8.1
- net -12V: now also C65.2
- net GND: now also C63.2, C67.2; no longer C65.2
- net ~{PS_ON}: now reaches J10.16 (PS_ON#), R34.2, TP6.1
Other:
- note removed: "NB: Must be LATCHING"
- moved on the sheet: C65

Commit message: fix a few schematic bugs, missing pull-ups and pull-downs in particular
Parts:
- added C68: 470 uF 20% 35V Electrolytic, Capacitor_SMD:CP_Elec_6.3x7.7, symbol Device:C_Polarized_Small_US
Connections:
- net -12V: now also C68.2; no longer C65.2
- net GND: now also C65.2, C68.1
Other:
- moved on the sheet: C65
Changed lines of the file:
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@@
 	(wire
 		(pts
+			(xy 87.63 59.69) (xy 87.63 62.23)
+		)
+		(stroke
+			(width 0)
+			(type default)
+		)
+	)
+	(wire
+		(pts
 			(xy 83.82 160.02) (xy 92.71 160.02)
 		)
@@
 	(wire
 		(pts
-			(xy 77.47 50.8) (xy 80.01 50.8)
-		)
-		(stroke
-			(width 0)
-			(type default)
-		)
-	)
-	(wire
-		(pts
 			(xy 198.755 50.165) (xy 201.93 50.165)
 		)
@@
 	(wire
 		(pts
-			(xy 87.63 46.99) (xy 87.63 50.8)
+			(xy 87.63 46.99) (xy 87.63 54.61)
 		)
 		(stroke
@@
 	(wire
 		(pts
-			(xy 77.47 46.99) (xy 77.47 50.8)
+			(xy 77.47 46.99) (xy 77.47 54.61)
 		)
 		(stroke
@@
 	(wire
 		(pts
-			(xy 85.09 50.8) (xy 87.63 50.8)
+			(xy 77.47 59.69) (xy 77.47 62.23)
 		)
 		(stroke
@@
 	)
 	(symbol
+		(lib_id "power:GND")
+		(at 87.63 62.23 0)
+		(unit 1)
+		(exclude_from_sim no)
+		(in_bom yes)
+		(on_board yes)
+		(dnp no)
+		(fields_autoplaced yes)
+		(property "Reference" "#PWR0329"
+			(at 87.63 68.58 0)
+			(effects
+				(font
+					(size 1.27 1.27)
+				)
+				(hide yes)
+			)
+		)
+		(property "Value" "GND"
+			(at 87.63 67.31 0)
+			(effects
+				(font
+					(size 1.27 1.27)
+				)
+			)
+		)
+		(property "Footprint" ""
+			(at 87.63 62.23 0)
+			(effects
+				(font
+					(size 1.27 1.27)
+				)
+				(hide yes)
+			)
+		)
+		(property "Datasheet" ""
+			(at 87.63 62.23 0)
+			(effects
+				(font
+					(size 1.27 1.27)
+				)
+				(hide yes)
+			)
+		)
+		(property "Description" ""
+			(at 87.63 62.23 0)
+			(effects
+				(font
+					(size 1.27 1.27)
+				)
+				(hide yes)
+			)
+		)
+		(pin "1"
+		)
+		(instances
+			(project "sbc_8088"
+				(path "/5e468d94-0319-44d1-a77f-2adc451eed13/358c98de-0d7c-4d65-8641-e21576518f6e"
+					(reference "#PWR0329")
+					(unit 1)
+				)
+			)
+		)
+	)
+	(symbol
 		(lib_id "power:PWR_FLAG")
 		(at 154.94 38.1 0)
@@
 	(symbol
 		(lib_id "power:GND")
+		(at 77.47 62.23 0)
+		(unit 1)
+		(exclude_from_sim no)
+		(in_bom yes)
+		(on_board yes)
+		(dnp no)
+		(fields_autoplaced yes)
+		(property "Reference" "#PWR0330"
+			(at 77.47 68.58 0)
+			(effects
+				(font
+					(size 1.27 1.27)
+				)
+				(hide yes)
+			)
+		)
+		(property "Value" "GND"
+			(at 77.47 67.31 0)
+			(effects
+				(font
+					(size 1.27 1.27)
+				)
+			)
+		)
+		(property "Footprint" ""
+			(at 77.47 62.23 0)
+			(effects
+				(font
+					(size 1.27 1.27)
+				)
+				(hide yes)
+			)
+		)
+		(property "Datasheet" ""
+			(at 77.47 62.23 0)
+			(effects
+				(font
+					(size 1.27 1.27)
+				)
+				(hide yes)
+			)
+		)
+		(property "Description" ""
+			(at 77.47 62.23 0)
+			(effects
+				(font
+					(size 1.27 1.27)
+				)
+				(hide yes)
+			)
+		)
+		(pin "1"
+		)
+		(instances
+			(project "sbc_8088"
+				(path "/5e468d94-0319-44d1-a77f-2adc451eed13/358c98de-0d7c-4d65-8641-e21576518f6e"
+					(reference "#PWR0330")
+					(unit 1)
+				)
+			)
+		)
+	)
+	(symbol
+		(lib_id "power:GND")
 		(at 228.6 154.94 0)
 		(unit 1)
@@
 	(symbol
 		(lib_id "Device:C_Polarized_Small_US")
+		(at 87.63 57.15 180)
+		(unit 1)
+		(exclude_from_sim no)
+		(in_bom yes)
+		(on_board yes)
+		(dnp no)
+		(fields_autoplaced yes)
+		(property "Reference" "C68"
+			(at 90.17 57.5817 0)
+			(effects
+				(font
+					(size 1.27 1.27)
+				)
+				(justify right)
+			)
+		)
+		(property "Value" "470 uF 20% 35V Electrolytic"
+			(at 85.09 56.3118 0)
+			(effects
+				(font
+					(size 1.27 1.27)
+				)
+				(justify left)
+				(hide yes)
+			)
+		)
+		(property "Footprint" "Capacitor_SMD:CP_Elec_6.3x7.7"
+			(at 87.63 57.15 0)
+			(effects
+				(font
+					(size 1.27 1.27)
+				)
+				(hide yes)
+			)
+		)
+		(property "Datasheet" "~"
+			(at 87.63 57.15 0)
+			(effects
+				(font
+					(size 1.27 1.27)
+				)
+				(hide yes)
+			)
+		)
+		(property "Description" "UWT1E101MCL1GS -- Aluminum Electrolytic Capacitors - SMD 25volts 100uF AEC-Q200  "
+			(at 87.63 57.15 0)
+			(effects
+				(font
+					(size 1.27 1.27)
+				)
+				(hide yes)
+			)
+		)
+		(pin "1"
+		)
+		(pin "2"
+		)
+		(instances
+			(project "sbc_8088"
+				(path "/5e468d94-0319-44d1-a77f-2adc451eed13/358c98de-0d7c-4d65-8641-e21576518f6e"
+					(reference "C68")
+					(unit 1)
+				)
+			)
+		)
+	)
+	(symbol
+		(lib_id "Device:C_Polarized_Small_US")
 		(at 270.51 146.05 0)
 		(unit 1)
@@
 	(symbol
 		(lib_id "Device:C_Polarized_Small_US")
-		(at 82.55 50.8 90)
+		(at 77.47 57.15 0)
 		(unit 1)
 		(exclude_from_sim no)
@@
 		(fields_autoplaced yes)
 		(property "Reference" "C65"
-			(at 82.1182 46.99 90)
+			(at 80.01 56.7181 0)
 			(effects
 				(font
 					(size 1.27 1.27)
 				)
+				(justify left)
 			)
 		)
 		(property "Value" "470 uF 20% 35V Electrolytic"
-			(at 83.3882 48.26 0)
+			(at 80.01 57.9882 0)
 			(effects
 				(font
@@
 		)
 		(property "Footprint" "Capacitor_SMD:CP_Elec_6.3x7.7"
-			(at 82.55 50.8 0)
+			(at 77.47 57.15 0)
 			(effects
 				(font
@@
 		)
 		(property "Datasheet" "~"
-			(at 82.55 50.8 0)
+			(at 77.47 57.15 0)
 			(effects
 				(font
@@
 		)
 		(property "Description" "UWT1E101MCL1GS -- Aluminum Electrolytic Capacitors - SMD 25volts 100uF AEC-Q200  "
-			(at 82.55 50.8 0)
+			(at 77.47 57.15 0)
 			(effects
 				(font

Commit message: add discharge resistors for all power rails
Parts:
- added R41, R42, R43, R44: 100k 0.5W, Resistor_SMD:R_0805_2012Metric, symbol Device:R_US
Connections:
- net +12V: now also R41.1
- net +5V: now also R44.1
- net +5VSB: now also R43.1
- net -12V: now also R42.1
- net GND: now also R41.2, R42.2, R43.2, R44.2

Commit message: working on removing DMA for now
Changed lines of the file:
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@@
-	)
-	(junction
-		(at 154.94 38.1)
-		(diameter 0)
-		(color 0 0 0 0)
 	)
 	(junction
@@
 	(wire
 		(pts
-			(xy 142.875 38.1) (xy 154.94 38.1)
-		)
-		(stroke
-			(width 0)
-			(type default)
-		)
-	)
-	(wire
-		(pts
 			(xy 196.85 138.43) (xy 196.85 143.51)
 		)
@@
 	(wire
 		(pts
-			(xy 154.94 38.1) (xy 164.465 38.1)
+			(xy 142.875 38.1) (xy 164.465 38.1)
 		)
 		(stroke
@@
 					(unit 1)
 				)
-			)
-		)
-	)
-	(symbol
-		(lib_id "power:PWR_FLAG")
-		(at 154.94 38.1 0)
-		(unit 1)
-		(exclude_from_sim no)
-		(in_bom yes)
-		(on_board yes)
-		(dnp no)
-		(fields_autoplaced yes)
-		(property "Reference" "#FLG02"
-			(at 154.94 36.195 0)
-			(effects
-				(font
-					(size 1.27 1.27)
-				)
-				(hide yes)
-			)
-		)
-		(property "Value" "PWR_FLAG"
-			(at 154.94 33.02 0)
-			(effects
-				(font
-					(size 1.27 1.27)
-				)
-			)
-		)
-		(property "Footprint" ""
-			(at 154.94 38.1 0)
-			(effects
-				(font
-					(size 1.27 1.27)
-				)
-				(hide yes)
-			)
-		)
-		(property "Datasheet" "~"
-			(at 154.94 38.1 0)
-			(effects
-				(font
-					(size 1.27 1.27)
-				)
-				(hide yes)
-			)
-		)
-		(property "Description" "Special symbol for telling ERC where power comes from"
-			(at 154.94 38.1 0)
-			(effects
-				(font
-					(size 1.27 1.27)
-				)
-				(hide yes)
-			)
-		)
-		(pin "1"
-		)
-		(instances
-			(project "sbc_8088"
-				(path "/5e468d94-0319-44d1-a77f-2adc451eed13/358c98de-0d7c-4d65-8641-e21576518f6e"
-					(reference "#FLG02")
-					(unit 1)
-				)

Commit message: fixes, prep for final production run
Parts:
- added C15, C16, C6: 4.7UF 16V 20%, Capacitor_SMD:CP_Elec_4x4.5, symbol Device:C_Polarized_Small_US
- added J14, J15, J16: Conn_01x04, Connector:FanPinHeader_1x04_P2.54mm_Vertical, symbol Connector_Generic:Conn_01x04
- C1, C12, C13, C18, C19, C21, C23, C27, C48, C49, C50: LCSC Part # (none) -> C371122
- C63, C64, C65, C66, C67, C68: LCSC Part # (none) -> C72523
- F2, F4: LCSC Part # (none) -> C92887
- F3: LCSC Part # (none) -> C2687079
- J10: LCSC Part # (none) -> C7541562
- R34: LCSC Part # (none) -> C84376
- R41, R42, R43, R44: LCSC Part # (none) -> C723424
- TP1, TP2, TP3, TP4, TP5, TP6, TP7, TP8, TP9: LCSC Part # (none) -> C7501259
Connections:
- net +12V: now also C15.1, C16.1, C6.1, J14.2 (Pin_2), J15.2 (Pin_2), J16.2 (Pin_2)
- net GND: now also C15.2, C16.2, C6.2, J14.1 (Pin_1), J15.1 (Pin_1), J16.1 (Pin_1)
- no-connect marks 0 -> 6
Other:
- note added: "ATX Fan Headers"
