File: sbc_power.kicad_sch (KiCad schematic)
At the start: 41 parts, among them J10 ATX-24, J14 Conn_01x04, J15 Conn_01x04, J16 Conn_01x04

Commit message: bump cpu to 8mhz, add second clock gen for ISA bus and PIT
Parts:
- added C74, C75: 4.7UF 16V 20%, Capacitor_SMD:CP_Elec_4x4.5, symbol Device:C_Polarized_Small_US
- added F5: Bourns MF-RHT100 1A hold, Fuse:Fuse_Bourns_MF-RHT100, symbol Device:Fuse
Connections:
- net +12V: now also F5.1; no longer C15.1, C16.1, C6.1, J14.2 (Pin_2), J15.2 (Pin_2), J16.2 (Pin_2)
- net +5V: now also C74.1, C75.1
- net GND: now also C74.2, C75.2
- new net FAN_12V: C15.1, C16.1, C6.1, F5.2, J14.2 (Pin_2), J15.2 (Pin_2), J16.2 (Pin_2)

Commit message: part tweaks, BOM is pretty much finalized, use 0.5W resistors for bleeders
Parts:
- F2, F4, F5: LCSC Part # C92887 -> C3760254; Manufacturer_Name (none) -> Bourns; Manufacturer_Part_Number (none) -> MF-RHT100-0
- F3: LCSC Part # C2687079 -> C3761895; Manufacturer_Name (none) -> Bourns; Manufacturer_Part_Number (none) -> MF-RHT200-0
- J10: LCSC Part # C7541562 -> C587701; Manufacturer_Name (none) -> Molex; Manufacturer_Part_Number (none) -> 44206-0007
- R41, R42, R43, R44: footprint Resistor_SMD:R_0805_2012Metric -> Resistor_SMD:R_1210_3225Metric; LCSC Part # C723424 -> C620660
Changed lines of the file:
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@@
 			)
 		)
-		(property "Description" "LCSC #C92887"
+		(property "Description" "LCSC #C3760254"
 			(at 226.06 25.4 0)
 			(effects
@@
 			)
 		)
-		(property "Manufacturer_Name" ""
+		(property "Manufacturer_Name" "Bourns"
 			(at 226.06 25.4 0)
 			(effects
@@
 			)
 		)
-		(property "Manufacturer_Part_Number" ""
+		(property "Manufacturer_Part_Number" "MF-RHT100-0"
 			(at 226.06 25.4 0)
 			(effects
@@
 			)
 		)
-		(property "LCSC Part #" "C92887"
+		(property "LCSC Part #" "C3760254"
 			(at 226.06 25.4 0)
 			(effects
@@
 			)
 		)
-		(property "Footprint" "Resistor_SMD:R_0805_2012Metric"
+		(property "Footprint" "Resistor_SMD:R_1210_3225Metric"
 			(at 60.706 56.134 90)
 			(effects
@@
 			)
 		)
-		(property "Description" "LCSC #C723424 "
+		(property "Description" "LCSC #C620660"
 			(at 59.69 55.88 0)
 			(effects
@@
 			)
 		)
-		(property "LCSC Part #" "C723424 "
+		(property "LCSC Part #" "C620660"
 			(at 59.69 55.88 0)
 			(effects
@@
 			)
 		)
-		(property "Footprint" "Resistor_SMD:R_0805_2012Metric"
+		(property "Footprint" "Resistor_SMD:R_1210_3225Metric"
 			(at 112.776 165.354 90)
 			(effects
@@
 			)
 		)
-		(property "Description" "LCSC #C723424 "
+		(property "Description" "LCSC #C620660"
 			(at 111.76 165.1 0)
 			(effects
@@
 			)
 		)
-		(property "LCSC Part #" "C723424 "
+		(property "LCSC Part #" "C620660"
 			(at 111.76 165.1 0)
 			(effects
@@
 			)
 		)
-		(property "Footprint" "Resistor_SMD:R_0805_2012Metric"
+		(property "Footprint" "Resistor_SMD:R_1210_3225Metric"
 			(at 125.476 43.434 90)
 			(effects
@@
 			)
 		)
-		(property "Description" "LCSC #C723424 "
+		(property "Description" "LCSC #C620660"
 			(at 124.46 43.18 0)
 			(effects
@@
 			)
 		)
-		(property "LCSC Part #" "C723424 "
+		(property "LCSC Part #" "C620660"
 			(at 124.46 43.18 0)
 			(effects
@@
 			)
 		)
-		(property "Description" "LCSC #C7541562"
+		(property "Description" "LCSC #C587701"
 			(at 146.05 97.79 0)
 			(effects
@@
 			)
 		)
-		(property "Manufacturer_Name" ""
+		(property "Manufacturer_Name" "Molex"
 			(at 146.05 97.79 0)
 			(effects
@@
 			)
 		)
-		(property "Manufacturer_Part_Number" ""
+		(property "Manufacturer_Part_Number" "44206-0007"
 			(at 146.05 97.79 0)
 			(effects
@@
 			)
 		)
-		(property "LCSC Part #" "C7541562"
+		(property "LCSC Part #" "C587701"
 			(at 146.05 97.79 0)
 			(effects
@@
 			)
 		)
-		(property "Footprint" "Resistor_SMD:R_0805_2012Metric"
+		(property "Footprint" "Resistor_SMD:R_1210_3225Metric"
 			(at 98.806 56.134 90)
 			(effects
@@
 			)
 		)
-		(property "Description" "LCSC #C723424 "
+		(property "Description" "LCSC #C620660"
 			(at 97.79 55.88 0)
 			(effects
@@
 			)
 		)
-		(property "LCSC Part #" "C723424 "
+		(property "LCSC Part #" "C620660"
 			(at 97.79 55.88 0)
 			(effects
@@
 			)
 		)
-		(property "Description" "LCSC #C2687079"
+		(property "Description" "LCSC #C3761895"
 			(at 83.82 153.67 0)
 			(effects
@@
 			)
 		)
-		(property "Manufacturer_Name" ""
+		(property "Manufacturer_Name" "Bourns"
 			(at 83.82 153.67 0)
 			(effects
@@
 			)
 		)
-		(property "Manufacturer_Part_Number" ""
+		(property "Manufacturer_Part_Number" "MF-RHT200-0"
 			(at 83.82 153.67 0)
 			(effects
@@
 			)
 		)
-		(property "LCSC Part #" "C2687079"
+		(property "LCSC Part #" "C3761895"
 			(at 83.82 153.67 0)
 			(effects
@@
 			)
 		)
-		(property "Description" "LCSC #C92887"
+		(property "Description" "LCSC #C3760254"
 			(at 77.47 40.64 0)
 			(effects
@@
 			)
 		)
-		(property "Manufacturer_Name" ""
+		(property "Manufacturer_Name" "Bourns"
 			(at 77.47 40.64 0)
 			(effects
@@
 			)
 		)
-		(property "Manufacturer_Part_Number" ""
+		(property "Manufacturer_Part_Number" "MF-RHT100-0"
 			(at 77.47 40.64 0)
 			(effects
@@
 			)
 		)
-		(property "LCSC Part #" "C92887"
+		(property "LCSC Part #" "C3760254"
 			(at 77.47 40.64 0)
 			(effects
@@
 			)
 		)
-		(property "Description" "LCSC #C92887"
+		(property "Description" "LCSC #C3760254"
 			(at 87.63 40.64 0)
 			(effects
@@
 			)
 		)
-		(property "Manufacturer_Name" ""
+		(property "Manufacturer_Name" "Bourns"
 			(at 87.63 40.64 0)
 			(effects
@@
 			)
 		)
-		(property "Manufacturer_Part_Number" ""
+		(property "Manufacturer_Part_Number" "MF-RHT100-0"
 			(at 87.63 40.64 0)
 			(effects
@@
 			)
 		)
-		(property "LCSC Part #" "C92887"
+		(property "LCSC Part #" "C3760254"
 			(at 87.63 40.64 0)
 			(effects

Commit message: minor BOM tweaks due part availability. make some pcb routing a little nicer.
Parts:
- F2, F4, F5: LCSC Part # C3760254 -> C2687078
- F3: LCSC Part # C3761895 -> C2687079
Changed lines of the file:
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@@
 			)
 		)
-		(property "Description" "LCSC #C3760254"
+		(property "Description" "LCSC #C3760254 (Bourns) or LCSC #C2687078"
 			(at 226.06 25.4 0)
 			(effects
@@
 			)
 		)
-		(property "LCSC Part #" "C3760254"
+		(property "LCSC Part #" "C2687078"
 			(at 226.06 25.4 0)
 			(effects
@@
 			)
 		)
-		(property "Description" "LCSC #C3761895"
+		(property "Description" "LCSC #C3761895 (Bourns) or LCSC #C2687079"
 			(at 83.82 153.67 0)
 			(effects
@@
 			)
 		)
-		(property "LCSC Part #" "C3761895"
+		(property "LCSC Part #" "C2687079"
 			(at 83.82 153.67 0)
 			(effects
@@
 			)
 		)
-		(property "Description" "LCSC #C3760254"
+		(property "Description" "LCSC #C3760254 (Bourns) or LCSC #C2687078"
 			(at 77.47 40.64 0)
 			(effects
@@
 			)
 		)
-		(property "LCSC Part #" "C3760254"
+		(property "LCSC Part #" "C2687078"
 			(at 77.47 40.64 0)
 			(effects
@@
 			)
 		)
-		(property "Description" "LCSC #C3760254"
+		(property "Description" "LCSC #C3760254 (Bourns) or LCSC #C2687078"
 			(at 87.63 40.64 0)
 			(effects
@@
 			)
 		)
-		(property "LCSC Part #" "C3760254"
+		(property "LCSC Part #" "C2687078"
 			(at 87.63 40.64 0)
 			(effects

Commit message: routing tweaks, use identity comparator instead of OR gates for IO decode
Connections:
- net ATX3_SENSE: now reaches J16.3 (Pin_3)
- net ATX3_CTRL: now reaches J16.4 (Pin_4)
- net ATX2_SENSE: now reaches J15.3 (Pin_3)
- net ATX2_CTRL: now reaches J15.4 (Pin_4)
- net ATX1_SENSE: now reaches J14.3 (Pin_3)
- net ATX1_CTRL: now reaches J14.4 (Pin_4)
Other:
- moved on the sheet: C15, C16, C6

Commit message: add i2c bus with expansion card sockets
Parts:
- removed C15, C16, C6: 4.7UF 16V 20%, Capacitor_SMD:CP_Elec_4x4.5, symbol Device:C_Polarized_Small_US
- removed J14, J15, J16: Conn_01x04, Connector:FanPinHeader_1x04_P2.54mm_Vertical, symbol Connector_Generic:Conn_01x04
- removed R34: 10k, Resistor_SMD:R_0805_2012Metric, symbol Device:R_US
Connections:
- net FAN_12V is gone; now on net +5VSB: F5.2
- net +12V: no longer F5.1
- net +5VSB: no longer J10.9 (+5VSB)
- new net +5VSB_IN: F5.1, J10.9 (+5VSB)
- no-connect marks 6 -> 0
Other:
- note removed: "ATX Fan Headers"
- note removed: "Distributed capacitance to be spread across the PCB Use smaller caps e.g. Nichicon UZT1E4R7MCL1GB"
- moved on the sheet: C65, C66, F4, R41, R43, TP1, TP2, TP3, TP5, TP7, TP9

Commit message: no more SMT for isa_i2c, tweak motherboard multiplex logic, handful of other tweaks
Parts:
- added C39: 470 uF 20% 35V Electrolytic, Capacitor_SMD:CP_Elec_6.3x7.7, symbol Device:C_Polarized_Small_US
- added F6: Bourns MF-RHT100 1A hold, Fuse:Fuse_Bourns_MF-RHT100, symbol Device:Fuse
- added J18, J19: 47053-1000, 470531000, symbol SamacSys_Parts:47053-1000
Connections:
- net +12V: now also F6.1
- net GND: now also C39.2, J18.1, J19.1
- new net 12V_FANS: C39.1, F6.2, J18.2, J19.2
- no-connect marks 0 -> 4
Other:
- note added: "ATX Fan Power"

Commit message: simplify m88 logic further, reduce ICs, reorient the POST display, use an oscillator for 14.31818 MHz, update isa-i2c bridge BOM
Parts:
- J18, J19: LCSC Part # (none) -> C240840
Changed lines of the file:
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@@
+			)
+		)
+		(property "LCSC Part #" "C240840"
+			(at 44.45 118.11 0)
+			(effects
+				(font
+					(size 1.27 1.27)
+				)
+				(hide yes)
 			)
 		)
@@
 				(hide yes)
 			)
+		)
+		(property "LCSC Part #" "C240840"
+			(at 44.45 93.98 0)
+			(effects
+				(font
+					(size 1.27 1.27)
+				)
+				(hide yes)
+			)
