File: bus_flags.kicad_sch (KiCad schematic)
At the start: 11 parts, among them U11 74LS02, U21 74LS04, U24 74LS32, U25 74LS125

Commit message: bringing over learnings/improvements from prototype board
Parts:
- removed R1, R60, R63, R64: 10k, Resistor_SMD:R_0805_2012Metric, symbol Device:R_US
- added RN9: 10k, Resistor_THT:R_Array_SIP5, symbol Device:R_Network04
Connections:
- net +5V: now also RN9.1 (common)
- net ~{IOR}: now also RN9.4 (R3)
- net ~{IOW}: now also RN9.5 (R4)
- net ~{MEMR}: now also RN9.2 (R1)
- net ~{MEMW}: now also RN9.3 (R2)

Commit message: more pcb routing, implementing learnings from the prototype board
Connections:
- net ~{IO}/M: now reaches U21.8, U24.10, U24.13
Changed lines of the file:
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@@
+		)
+	)
+	(label "~{IO}{slash}M"
+		(at 96.52 123.19 0)
+		(fields_autoplaced yes)
+		(effects
+			(font
+				(size 1.27 1.27)
+			)
+			(justify left bottom)
 		)
 	)

Commit message: pcb is fully routed, working on power capacitor tweaks, some ROM testing
Parts:
- renumbered C25 to C21, C26 to C25, C2 to C39, RN9 to RN2, U24 to U11, U21 to U16, U11 to U23, U25 to U9
Changed lines of the file:
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@@
 		(dnp no)
 		(fields_autoplaced yes)
-		(property "Reference" "U21"
+		(property "Reference" "U16"
 			(at 82.55 107.95 0)
 			(effects
@@
 			(project "sbc_8088"
 				(path "/5e468d94-0319-44d1-a77f-2adc451eed13/93dfc828-b49f-4967-b4e5-8966b969d123"
-					(reference "U21")
+					(reference "U16")
 					(unit 4)
 				)
@@
 		(dnp no)
 		(fields_autoplaced yes)
-		(property "Reference" "C2"
+		(property "Reference" "C39"
 			(at 262.89 21.59 90)
 			(effects
@@
 			(project "sbc_8088"
 				(path "/5e468d94-0319-44d1-a77f-2adc451eed13/93dfc828-b49f-4967-b4e5-8966b969d123"
-					(reference "C2")
+					(reference "C39")
 					(unit 1)
 				)
@@
 		(dnp no)
 		(fields_autoplaced yes)
-		(property "Reference" "U24"
+		(property "Reference" "U11"
 			(at 262.89 113.665 0)
 			(effects
@@
 			(project "sbc_8088"
 				(path "/5e468d94-0319-44d1-a77f-2adc451eed13/93dfc828-b49f-4967-b4e5-8966b969d123"
-					(reference "U24")
+					(reference "U11")
 					(unit 5)
 				)
@@
 		(dnp no)
 		(fields_autoplaced yes)
-		(property "Reference" "U25"
+		(property "Reference" "U9"
 			(at 142.875 100.965 0)
 			(effects
@@
 			(project "sbc_8088"
 				(path "/5e468d94-0319-44d1-a77f-2adc451eed13/93dfc828-b49f-4967-b4e5-8966b969d123"
-					(reference "U25")
+					(reference "U9")
 					(unit 3)
 				)
@@
 		(dnp no)
 		(fields_autoplaced yes)
-		(property "Reference" "U11"
+		(property "Reference" "U23"
 			(at 162.56 149.86 0)
 			(effects
@@
 			(project "sbc_8088"
 				(path "/5e468d94-0319-44d1-a77f-2adc451eed13/93dfc828-b49f-4967-b4e5-8966b969d123"
-					(reference "U11")
+					(reference "U23")
 					(unit 3)
 				)
@@
 		(dnp no)
 		(fields_autoplaced yes)
-		(property "Reference" "U25"
+		(property "Reference" "U9"
 			(at 229.87 113.665 0)
 			(effects
@@
 			(project "sbc_8088"
 				(path "/5e468d94-0319-44d1-a77f-2adc451eed13/93dfc828-b49f-4967-b4e5-8966b969d123"
-					(reference "U25")
+					(reference "U9")
 					(unit 5)
 				)
@@
 		(dnp no)
 		(fields_autoplaced yes)
-		(property "Reference" "U24"
+		(property "Reference" "U11"
 			(at 121.285 67.31 0)
 			(effects
@@
 			(project "sbc_8088"
 				(path "/5e468d94-0319-44d1-a77f-2adc451eed13/93dfc828-b49f-4967-b4e5-8966b969d123"
-					(reference "U24")
+					(reference "U11")
 					(unit 1)
 				)
@@
 		(dnp no)
 		(fields_autoplaced yes)
-		(property "Reference" "U11"
+		(property "Reference" "U23"
 			(at 162.56 165.1 0)
 			(effects
@@
 			(project "sbc_8088"
 				(path "/5e468d94-0319-44d1-a77f-2adc451eed13/93dfc828-b49f-4967-b4e5-8966b969d123"
-					(reference "U11")
+					(reference "U23")
 					(unit 4)
 				)
@@
 		(dnp no)
 		(fields_autoplaced yes)
-		(property "Reference" "U25"
+		(property "Reference" "U9"
 			(at 143.51 117.475 0)
 			(effects
@@
 			(project "sbc_8088"
 				(path "/5e468d94-0319-44d1-a77f-2adc451eed13/93dfc828-b49f-4967-b4e5-8966b969d123"
-					(reference "U25")
+					(reference "U9")
 					(unit 4)
 				)
@@
 		(dnp no)
 		(fields_autoplaced yes)
-		(property "Reference" "U24"
+		(property "Reference" "U11"
 			(at 121.285 100.965 0)
 			(effects
@@
 			(project "sbc_8088"
 				(path "/5e468d94-0319-44d1-a77f-2adc451eed13/93dfc828-b49f-4967-b4e5-8966b969d123"
-					(reference "U24")
+					(reference "U11")
 					(unit 3)
 				)
@@
 		(dnp no)
 		(fields_autoplaced yes)
-		(property "Reference" "U25"
+		(property "Reference" "U9"
 			(at 142.875 83.82 0)
 			(effects
@@
 			(project "sbc_8088"
 				(path "/5e468d94-0319-44d1-a77f-2adc451eed13/93dfc828-b49f-4967-b4e5-8966b969d123"
-					(reference "U25")
+					(reference "U9")
 					(unit 2)
 				)
@@
 		(dnp no)
 		(fields_autoplaced yes)
-		(property "Reference" "U25"
+		(property "Reference" "U9"
 			(at 143.51 67.31 0)
 			(effects
@@
 			(project "sbc_8088"
 				(path "/5e468d94-0319-44d1-a77f-2adc451eed13/93dfc828-b49f-4967-b4e5-8966b969d123"
-					(reference "U25")
+					(reference "U9")
 					(unit 1)
 				)
@@
 		(dnp no)
 		(fields_autoplaced yes)
-		(property "Reference" "U24"
+		(property "Reference" "U11"
 			(at 120.65 116.84 0)
 			(effects
@@
 			(project "sbc_8088"
 				(path "/5e468d94-0319-44d1-a77f-2adc451eed13/93dfc828-b49f-4967-b4e5-8966b969d123"
-					(reference "U24")
+					(reference "U11")
 					(unit 4)
 				)
@@
 		(dnp no)
 		(fields_autoplaced yes)
-		(property "Reference" "U11"
+		(property "Reference" "U23"
 			(at 264.16 41.91 0)
 			(effects
@@
 			(project "sbc_8088"
 				(path "/5e468d94-0319-44d1-a77f-2adc451eed13/93dfc828-b49f-4967-b4e5-8966b969d123"
-					(reference "U11")
+					(reference "U23")
 					(unit 5)
 				)
@@
 		(dnp no)
 		(fields_autoplaced yes)
-		(property "Reference" "U24"
+		(property "Reference" "U11"
 			(at 121.285 84.455 0)
 			(effects
@@
 			(project "sbc_8088"
 				(path "/5e468d94-0319-44d1-a77f-2adc451eed13/93dfc828-b49f-4967-b4e5-8966b969d123"
-					(reference "U24")
+					(reference "U11")
 					(unit 2)
 				)
@@
 		(dnp no)
 		(fields_autoplaced yes)
-		(property "Reference" "RN9"
+		(property "Reference" "RN2"
 			(at 209.296 83.82 90)
 			(effects
@@
 			(project "sbc_8088"
 				(path "/5e468d94-0319-44d1-a77f-2adc451eed13/93dfc828-b49f-4967-b4e5-8966b969d123"
-					(reference "RN9")
+					(reference "RN2")
 					(unit 1)
 				)
@@
 		(dnp no)
 		(fields_autoplaced yes)
-		(property "Reference" "C25"
+		(property "Reference" "C21"
 			(at 228.6063 95.25 90)
 			(effects
@@
 			(project "sbc_8088"
 				(path "/5e468d94-0319-44d1-a77f-2adc451eed13/93dfc828-b49f-4967-b4e5-8966b969d123"
-					(reference "C25")
+					(reference "C21")
 					(unit 1)
 				)
@@
 		(dnp no)
 		(fields_autoplaced yes)
-		(property "Reference" "U11"
+		(property "Reference" "U23"
 			(at 177.165 26.67 0)
 			(effects
@@
 			(project "sbc_8088"
 				(path "/5e468d94-0319-44d1-a77f-2adc451eed13/93dfc828-b49f-4967-b4e5-8966b969d123"
-					(reference "U11")
+					(reference "U23")
 					(unit 2)
 				)
@@
 		(dnp no)
 		(fields_autoplaced yes)
-		(property "Reference" "U21"
+		(property "Reference" "U16"
 			(at 195.58 27.305 0)
 			(effects
@@
 			(project "sbc_8088"
 				(path "/5e468d94-0319-44d1-a77f-2adc451eed13/93dfc828-b49f-4967-b4e5-8966b969d123"
-					(reference "U21")
+					(reference "U16")
 					(unit 5)
 				)
@@
 		(dnp no)
 		(fields_autoplaced yes)
-		(property "Reference" "C26"
+		(property "Reference" "C25"
 			(at 261.6263 95.25 90)
 			(effects
@@
 			(project "sbc_8088"
 				(path "/5e468d94-0319-44d1-a77f-2adc451eed13/93dfc828-b49f-4967-b4e5-8966b969d123"
-					(reference "C26")
+					(reference "C25")
 					(unit 1)
 				)

Commit message: added ATtiny for SMC, added PC speaker
Parts:
- renumbered C21 to C24, C25 to C31, C39 to C44, U9 to U11, U11 to U14, U16 to U18, U23 to U27
Changed lines of the file:
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@@
 		(dnp no)
 		(fields_autoplaced yes)
-		(property "Reference" "U16"
+		(property "Reference" "U18"
 			(at 82.55 107.95 0)
 			(effects
@@
 			(project "sbc_8088"
 				(path "/5e468d94-0319-44d1-a77f-2adc451eed13/93dfc828-b49f-4967-b4e5-8966b969d123"
-					(reference "U16")
+					(reference "U18")
 					(unit 4)
 				)
@@
 		(dnp no)
 		(fields_autoplaced yes)
-		(property "Reference" "C39"
+		(property "Reference" "C44"
 			(at 262.89 21.59 90)
 			(effects
@@
 			(project "sbc_8088"
 				(path "/5e468d94-0319-44d1-a77f-2adc451eed13/93dfc828-b49f-4967-b4e5-8966b969d123"
-					(reference "C39")
+					(reference "C44")
 					(unit 1)
 				)
@@
 		(dnp no)
 		(fields_autoplaced yes)
-		(property "Reference" "U11"
+		(property "Reference" "U14"
 			(at 262.89 113.665 0)
 			(effects
@@
 			(project "sbc_8088"
 				(path "/5e468d94-0319-44d1-a77f-2adc451eed13/93dfc828-b49f-4967-b4e5-8966b969d123"
-					(reference "U11")
+					(reference "U14")
 					(unit 5)
 				)
@@
 		(dnp no)
 		(fields_autoplaced yes)
-		(property "Reference" "U9"
+		(property "Reference" "U11"
 			(at 142.875 100.965 0)
 			(effects
@@
 			(project "sbc_8088"
 				(path "/5e468d94-0319-44d1-a77f-2adc451eed13/93dfc828-b49f-4967-b4e5-8966b969d123"
-					(reference "U9")
+					(reference "U11")
 					(unit 3)
 				)
@@
 		(dnp no)
 		(fields_autoplaced yes)
-		(property "Reference" "U23"
+		(property "Reference" "U27"
 			(at 162.56 149.86 0)
 			(effects
@@
 			(project "sbc_8088"
 				(path "/5e468d94-0319-44d1-a77f-2adc451eed13/93dfc828-b49f-4967-b4e5-8966b969d123"
-					(reference "U23")
+					(reference "U27")
 					(unit 3)
 				)
@@
 		(dnp no)
 		(fields_autoplaced yes)
-		(property "Reference" "U9"
+		(property "Reference" "U11"
 			(at 229.87 113.665 0)
 			(effects
@@
 			(project "sbc_8088"
 				(path "/5e468d94-0319-44d1-a77f-2adc451eed13/93dfc828-b49f-4967-b4e5-8966b969d123"
-					(reference "U9")
+					(reference "U11")
 					(unit 5)
 				)
@@
 		(dnp no)
 		(fields_autoplaced yes)
-		(property "Reference" "U11"
+		(property "Reference" "U14"
 			(at 121.285 67.31 0)
 			(effects
@@
 			(project "sbc_8088"
 				(path "/5e468d94-0319-44d1-a77f-2adc451eed13/93dfc828-b49f-4967-b4e5-8966b969d123"
-					(reference "U11")
+					(reference "U14")
 					(unit 1)
 				)
@@
 		(dnp no)
 		(fields_autoplaced yes)
-		(property "Reference" "U23"
+		(property "Reference" "U27"
 			(at 162.56 165.1 0)
 			(effects
@@
 			(project "sbc_8088"
 				(path "/5e468d94-0319-44d1-a77f-2adc451eed13/93dfc828-b49f-4967-b4e5-8966b969d123"
-					(reference "U23")
+					(reference "U27")
 					(unit 4)
 				)
@@
 		(dnp no)
 		(fields_autoplaced yes)
-		(property "Reference" "U9"
+		(property "Reference" "U11"
 			(at 143.51 117.475 0)
 			(effects
@@
 			(project "sbc_8088"
 				(path "/5e468d94-0319-44d1-a77f-2adc451eed13/93dfc828-b49f-4967-b4e5-8966b969d123"
-					(reference "U9")
+					(reference "U11")
 					(unit 4)
 				)
@@
 		(dnp no)
 		(fields_autoplaced yes)
-		(property "Reference" "U11"
+		(property "Reference" "U14"
 			(at 121.285 100.965 0)
 			(effects
@@
 			(project "sbc_8088"
 				(path "/5e468d94-0319-44d1-a77f-2adc451eed13/93dfc828-b49f-4967-b4e5-8966b969d123"
-					(reference "U11")
+					(reference "U14")
 					(unit 3)
 				)
@@
 		(dnp no)
 		(fields_autoplaced yes)
-		(property "Reference" "U9"
+		(property "Reference" "U11"
 			(at 142.875 83.82 0)
 			(effects
@@
 			(project "sbc_8088"
 				(path "/5e468d94-0319-44d1-a77f-2adc451eed13/93dfc828-b49f-4967-b4e5-8966b969d123"
-					(reference "U9")
+					(reference "U11")
 					(unit 2)
 				)
@@
 		(dnp no)
 		(fields_autoplaced yes)
-		(property "Reference" "U9"
+		(property "Reference" "U11"
 			(at 143.51 67.31 0)
 			(effects
@@
 			(project "sbc_8088"
 				(path "/5e468d94-0319-44d1-a77f-2adc451eed13/93dfc828-b49f-4967-b4e5-8966b969d123"
-					(reference "U9")
+					(reference "U11")
 					(unit 1)
 				)
@@
 		(dnp no)
 		(fields_autoplaced yes)
-		(property "Reference" "U11"
+		(property "Reference" "U14"
 			(at 120.65 116.84 0)
 			(effects
@@
 			(project "sbc_8088"
 				(path "/5e468d94-0319-44d1-a77f-2adc451eed13/93dfc828-b49f-4967-b4e5-8966b969d123"
-					(reference "U11")
+					(reference "U14")
 					(unit 4)
 				)
@@
 		(dnp no)
 		(fields_autoplaced yes)
-		(property "Reference" "U23"
+		(property "Reference" "U27"
 			(at 264.16 41.91 0)
 			(effects
@@
 			(project "sbc_8088"
 				(path "/5e468d94-0319-44d1-a77f-2adc451eed13/93dfc828-b49f-4967-b4e5-8966b969d123"
-					(reference "U23")
+					(reference "U27")
 					(unit 5)
 				)
@@
 		(dnp no)
 		(fields_autoplaced yes)
-		(property "Reference" "U11"
+		(property "Reference" "U14"
 			(at 121.285 84.455 0)
 			(effects
@@
 			(project "sbc_8088"
 				(path "/5e468d94-0319-44d1-a77f-2adc451eed13/93dfc828-b49f-4967-b4e5-8966b969d123"
-					(reference "U11")
+					(reference "U14")
 					(unit 2)
 				)
@@
 		(dnp no)
 		(fields_autoplaced yes)
-		(property "Reference" "C21"
+		(property "Reference" "C24"
 			(at 228.6063 95.25 90)
 			(effects
@@
 			(project "sbc_8088"
 				(path "/5e468d94-0319-44d1-a77f-2adc451eed13/93dfc828-b49f-4967-b4e5-8966b969d123"
-					(reference "C21")
+					(reference "C24")
 					(unit 1)
 				)
@@
 		(dnp no)
 		(fields_autoplaced yes)
-		(property "Reference" "U23"
+		(property "Reference" "U27"
 			(at 177.165 26.67 0)
 			(effects
@@
 			(project "sbc_8088"
 				(path "/5e468d94-0319-44d1-a77f-2adc451eed13/93dfc828-b49f-4967-b4e5-8966b969d123"
-					(reference "U23")
+					(reference "U27")
 					(unit 2)
 				)
@@
 		(dnp no)
 		(fields_autoplaced yes)
-		(property "Reference" "U16"
+		(property "Reference" "U18"
 			(at 195.58 27.305 0)
 			(effects
@@
 			(project "sbc_8088"
 				(path "/5e468d94-0319-44d1-a77f-2adc451eed13/93dfc828-b49f-4967-b4e5-8966b969d123"
-					(reference "U16")
+					(reference "U18")
 					(unit 5)
 				)
@@
 		(dnp no)
 		(fields_autoplaced yes)
-		(property "Reference" "C25"
+		(property "Reference" "C31"
 			(at 261.6263 95.25 90)
 			(effects
@@
 			(project "sbc_8088"
 				(path "/5e468d94-0319-44d1-a77f-2adc451eed13/93dfc828-b49f-4967-b4e5-8966b969d123"
-					(reference "C25")
+					(reference "C31")
 					(unit 1)
 				)

Commit message: working on removing DMA for now
Parts:
- added C2: 0.1uF 20% Ceramic, Capacitor_SMD:C_0805_2012Metric, symbol Device:C
- added R47: 10k, Resistor_SMD:R_0805_2012Metric, symbol Device:R_US
- added unit 6 of U18
- added unit 2 of U18
- added unit 1 of U18
- added unit 7 of U18
- added unit 3 of U18
Connections:
- net DMA_AEN is gone; now on net GND: U27.6
- net HLDA is gone; now on net GND: U27.5
- net +5V: now also C2.1, U18.14 (VCC)
- net GND: now also U18.11, C2.2, R47.2, U18.1, U18.13, U18.3, U18.5, U18.7 (GND)
- net ~{BUSEN}: now also R47.1; no longer U18.10
- net at U27.4: no longer U18.11
- no-connect marks 2 -> 8
Other:
- moved on the sheet: U18E, U27B

Commit message: fixes, prep for final production run
Parts:
- C2, C24, C31, C44: LCSC Part # (none) -> C1853649
- R47: LCSC Part # (none) -> C84376
- RN2: LCSC Part # (none) -> C11394
- U11, U14, U18, U27: LCSC Part # (none) -> C72114

Commit message: no more SMT for isa_i2c, tweak motherboard multiplex logic, handful of other tweaks
Parts:
- removed C24, C31: 0.1uF 20% Ceramic, Capacitor_SMD:C_0805_2012Metric, symbol Device:C_Small
- removed C44: 0.1uF 20% Ceramic, Capacitor_SMD:C_0805_2012Metric, symbol Device:C
- removed U11: 74LS125, Package_DIP:DIP-14_W7.62mm_Socket, symbol 74xx:74LS125
- removed U14: 74LS32, Package_DIP:DIP-14_W7.62mm_Socket, symbol 74xx:74LS32
- removed U18: 74LS04, Package_DIP:DIP-14_W7.62mm_Socket, symbol 74xx:74LS04
- removed U27: 74LS02, Package_DIP:DIP-14_W7.62mm_Socket, symbol 74xx:74LS02
- added R34, R50, R51: 22, Resistor_SMD:R_0805_2012Metric, symbol Device:R_US
- added U8: 74LS138, Package_DIP:DIP-16_W7.62mm_Socket, symbol 74xx:74LS138
- R47: value 10k -> 22; LCSC Part # C84376 -> (none)
- RN2: value 10k -> 4.7k; LCSC Part # C11394 -> (none)
Connections:
- net +5V: now also U8.16 (VCC), U8.6 (E3)
- net GND: now also U8.4 (E1), U8.5 (E2), U8.8 (GND); no longer R47.2
- net IO/~{M}: now also U8.3 (A2)
- net ~{IOR}: now also R50.2
- net ~{IOW}: now also R51.2
- net ~{MEMR}: now also R34.2
- net ~{MEMW}: now also R47.2
- net ~{RD}: now also U8.2 (A1)
- net ~{WR}: now also U8.1 (A0)
- net ~{BUSEN}: no longer names the net of R47.1
- net ~{BUSEN}: now also U8.13 (O2)
- new net: R51.1, U8.9 (O6)
- new net: R34.1, U8.14 (O1)
- new net: R50.1, U8.10 (O5)
- no-connect marks 8 -> 4
Other:
- note added: "BUSEN can be used to float address bus when CPU is held and/or DMA is active Add pull-down when DMAC is added back to the design"
- note removed: "BUSEN can be used to float address bus when CPU is held and/or DMA is active"
