File: bus_flags.kicad_sch (KiCad schematic)
At the start: 7 parts, among them U8 74LS138

Commit message: simplify m88 logic further, reduce ICs, reorient the POST display, use an oscillator for 14.31818 MHz, update isa-i2c bridge BOM
Parts:
- R34, R47, R50, R51: LCSC Part # (none) -> C2933536
- RN2: LCSC Part # (none) -> C33175
Changed lines of the file:
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@@
 			)
 		)
-		(property "Description" ""
+		(property "Description" "LCSC #C2933536"
 			(at 140.97 102.87 0)
 			(effects
@@
 			)
 		)
-		(property "LCSC Part #" ""
+		(property "LCSC Part #" "C2933536"
 			(at 140.97 102.87 0)
 			(effects
@@
 			)
 		)
-		(property "Description" ""
+		(property "Description" "LCSC #C2933536"
 			(at 140.97 87.63 0)
 			(effects
@@
 			)
 		)
-		(property "LCSC Part #" ""
+		(property "LCSC Part #" "C2933536"
 			(at 140.97 87.63 0)
 			(effects
@@
 			)
 		)
-		(property "Description" ""
+		(property "Description" "LCSC #C2933536"
 			(at 140.97 78.74 0)
 			(effects
@@
 			)
 		)
-		(property "LCSC Part #" ""
+		(property "LCSC Part #" "C2933536"
 			(at 140.97 78.74 0)
 			(effects
@@
 			)
 		)
-		(property "Description" ""
+		(property "Description" "LCSC #C33175"
 			(at 189.23 97.79 0)
 			(effects
@@
 			)
 		)
-		(property "LCSC Part #" ""
+		(property "LCSC Part #" "C33175"
 			(at 189.23 97.79 0)
 			(effects
@@
 			)
 		)
-		(property "Description" ""
+		(property "Description" "LCSC #C2933536"
 			(at 140.97 100.33 0)
 			(effects
@@
 			)
 		)
-		(property "LCSC Part #" ""
+		(property "LCSC Part #" "C2933536"
 			(at 140.97 100.33 0)
 			(effects

Commit message: motherboard tweaks for manufacturing run, i2c card tweaks for manufacturing run, de9 -> stemma adapter idea for the i2c card
Parts:
- C2: LCSC Part # C1853649 -> C49678
- R34, R47, R50, R51: LCSC Part # C2933536 -> C17561
- RN2: footprint Resistor_THT:R_Array_SIP5 -> Resistor_THT:R_Array_SIP7; symbol Device:R_Network04 -> Device:R_Network06; LCSC Part # C33175 -> C39096
Connections:
- net ~{IOR}: now also RN2.5 (R4); no longer RN2.4 (R3)
- net ~{IOW}: now also RN2.6 (R5); no longer RN2.5 (R4)
- net ~{MEMR}: now also RN2.3 (R2); no longer RN2.2 (R1)
- net ~{MEMW}: now also RN2.4 (R3); no longer RN2.3 (R2)
- no-connect marks 4 -> 6
Changed lines of the file:
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@@
+	)
+	(no_connect
+		(at 184.15 92.71)
 	)
 	(no_connect
@@
 	)
 	(no_connect
+		(at 184.15 105.41)
+	)
+	(no_connect
 		(at 127 95.25)
 	)
@@
 	(wire
 		(pts
+			(xy 181.61 100.33) (xy 184.15 100.33)
+		)
+		(stroke
+			(width 0)
+			(type default)
+		)
+	)
+	(wire
+		(pts
 			(xy 114.3 74.93) (xy 114.3 80.01)
 		)
@@
 	(wire
 		(pts
+			(xy 82.55 100.33) (xy 101.6 100.33)
+		)
+		(stroke
+			(width 0)
+			(type default)
+		)
+	)
+	(wire
+		(pts
 			(xy 181.61 95.25) (xy 184.15 95.25)
 		)
@@
 	(wire
 		(pts
-			(xy 82.55 100.33) (xy 101.6 100.33)
-		)
-		(stroke
-			(width 0)
-			(type default)
-		)
-	)
-	(wire
-		(pts
 			(xy 144.78 78.74) (xy 146.05 78.74)
 		)
@@
 	(wire
 		(pts
+			(xy 181.61 97.79) (xy 184.15 97.79)
+		)
+		(stroke
+			(width 0)
+			(type default)
+		)
+	)
+	(wire
+		(pts
 			(xy 127 102.87) (xy 137.16 102.87)
 		)
@@
 	(wire
 		(pts
+			(xy 181.61 102.87) (xy 184.15 102.87)
+		)
+		(stroke
+			(width 0)
+			(type default)
+		)
+	)
+	(wire
+		(pts
 			(xy 96.52 87.63) (xy 101.6 87.63)
 		)
@@
 	(wire
 		(pts
-			(xy 181.61 92.71) (xy 184.15 92.71)
-		)
-		(stroke
-			(width 0)
-			(type default)
-		)
-	)
-	(wire
-		(pts
 			(xy 199.39 35.56) (xy 219.71 35.56)
 		)
@@
 	(wire
 		(pts
-			(xy 181.61 100.33) (xy 184.15 100.33)
-		)
-		(stroke
-			(width 0)
-			(type default)
-		)
-	)
-	(wire
-		(pts
 			(xy 114.3 71.12) (xy 114.3 74.93)
 		)
@@
 		(pts
 			(xy 120.65 31.75) (xy 120.65 30.48)
-		)
-		(stroke
-			(width 0)
-			(type default)
-		)
-	)
-	(wire
-		(pts
-			(xy 181.61 97.79) (xy 184.15 97.79)
 		)
 		(stroke
@@
 	(hierarchical_label "~{MEMW}"
 		(shape tri_state)
-		(at 181.61 95.25 180)
+		(at 181.61 97.79 180)
 		(fields_autoplaced yes)
 		(effects
@@
 	(hierarchical_label "~{IOR}"
 		(shape tri_state)
-		(at 181.61 97.79 180)
+		(at 181.61 100.33 180)
 		(fields_autoplaced yes)
 		(effects
@@
 		)
 	)
+	(hierarchical_label "~{IOW}"
+		(shape tri_state)
+		(at 181.61 102.87 180)
+		(fields_autoplaced yes)
+		(effects
+			(font
+				(size 1.27 1.27)
+			)
+			(justify right)
+		)
+	)
 	(hierarchical_label "~{IOR}"
 		(shape tri_state)
@@
 	(hierarchical_label "~{MEMR}"
 		(shape tri_state)
-		(at 181.61 92.71 180)
+		(at 146.05 78.74 0)
 		(fields_autoplaced yes)
 		(effects
@@
 				(size 1.27 1.27)
 			)
-			(justify right)
-		)
-	)
-	(hierarchical_label "~{MEMR}"
+			(justify left)
+		)
+	)
+	(hierarchical_label "~{MEMW}"
 		(shape tri_state)
-		(at 146.05 78.74 0)
+		(at 147.32 87.63 0)
 		(fields_autoplaced yes)
 		(effects
@@
 		)
 	)
-	(hierarchical_label "~{IOW}"
+	(hierarchical_label "~{MEMR}"
 		(shape tri_state)
-		(at 181.61 100.33 180)
+		(at 181.61 95.25 180)
 		(fields_autoplaced yes)
 		(effects
@@
 			)
 			(justify right)
-		)
-	)
-	(hierarchical_label "~{MEMW}"
-		(shape tri_state)
-		(at 147.32 87.63 0)
-		(fields_autoplaced yes)
-		(effects
-			(font
-				(size 1.27 1.27)
-			)
-			(justify left)
 		)
 	)
@@
 			)
 		)
-		(property "Description" "LCSC #C2933536"
+		(property "Description" "LCSC #C17561"
 			(at 140.97 102.87 0)
 			(effects
@@
 			)
 		)
-		(property "LCSC Part #" "C2933536"
+		(property "LCSC Part #" "C17561"
 			(at 140.97 102.87 0)
 			(effects
@@
 			)
 		)
-		(property "Description" "LCSC #C2933536"
+		(property "Description" "LCSC #C17561"
 			(at 140.97 87.63 0)
 			(effects
@@
 			)
 		)
-		(property "LCSC Part #" "C2933536"
+		(property "LCSC Part #" "C17561"
 			(at 140.97 87.63 0)
 			(effects
@@
 			)
 		)
-		(property "Description" "LCSC #C2933536"
+		(property "Description" "LCSC #C17561"
 			(at 140.97 78.74 0)
 			(effects
@@
 			)
 		)
-		(property "LCSC Part #" "C2933536"
+		(property "LCSC Part #" "C17561"
 			(at 140.97 78.74 0)
 			(effects
@@
 	)
 	(symbol
-		(lib_id "Device:R_Network04")
-		(at 189.23 97.79 270)
+		(lib_id "Device:R_Network06")
+		(at 189.23 100.33 270)
 		(unit 1)
 		(exclude_from_sim no)
@@
 			)
 		)
-		(property "Footprint" "Resistor_THT:R_Array_SIP5"
-			(at 189.23 104.775 90)
+		(property "Footprint" "Resistor_THT:R_Array_SIP7"
+			(at 189.23 109.855 90)
 			(effects
 				(font
@@
 		)
 		(property "Datasheet" "http://www.vishay.com/docs/31509/csc.pdf"
-			(at 189.23 97.79 0)
-			(effects
-				(font
-					(size 1.27 1.27)
-				)
-				(hide yes)
-			)
-		)
-		(property "Description" "LCSC #C33175"
-			(at 189.23 97.79 0)
+			(at 189.23 100.33 0)
+			(effects
+				(font
+					(size 1.27 1.27)
+				)
+				(hide yes)
+			)
+		)
+		(property "Description" "LCSC #C39096"
+			(at 189.23 100.33 0)
 			(effects
 				(font
@@
 		)
 		(property "Height" ""
-			(at 189.23 97.79 0)
+			(at 189.23 100.33 0)
 			(effects
 				(font
@@
 		)
 		(property "Manufacturer_Name" ""
-			(at 189.23 97.79 0)
+			(at 189.23 100.33 0)
 			(effects
 				(font
@@
 		)
 		(property "Manufacturer_Part_Number" ""
-			(at 189.23 97.79 0)
+			(at 189.23 100.33 0)
 			(effects
 				(font
@@
 		)
 		(property "Mouser Part Number" ""
-			(at 189.23 97.79 0)
+			(at 189.23 100.33 0)
 			(effects
 				(font
@@
 		)
 		(property "Mouser Price/Stock" ""
-			(at 189.23 97.79 0)
-			(effects
-				(font
-					(size 1.27 1.27)
-				)
-				(hide yes)
-			)
-		)
-		(property "LCSC Part #" "C33175"
-			(at 189.23 97.79 0)
+			(at 189.23 100.33 0)
+			(effects
+				(font
+					(size 1.27 1.27)
+				)
+				(hide yes)
+			)
+		)
+		(property "LCSC Part #" "C39096"
+			(at 189.23 100.33 0)
 			(effects
 				(font
@@
 		)
 		(pin "4"
+		)
+		(pin "6"
+		)
+		(pin "7"
 		)
 		(instances
@@
 			)
 		)
-		(property "Description" "LCSC #C1853649"
+		(property "Description" "LCSC #C49678"
 			(at 123.19 74.93 0)
 			(effects
@@
 			)
 		)
-		(property "LCSC Part #" "C1853649"
+		(property "LCSC Part #" "C49678"
 			(at 123.19 74.93 0)
 			(effects
@@
 			)
 		)
-		(property "Description" "LCSC #C2933536"
+		(property "Description" "LCSC #C17561"
 			(at 140.97 100.33 0)
 			(effects
@@
 			)
 		)
-		(property "LCSC Part #" "C2933536"
+		(property "LCSC Part #" "C17561"
 			(at 140.97 100.33 0)
 			(effects
