File: RTC.kicad_sch (KiCad schematic)
At the start: 2 parts, among them IC1 DS12887+

Commit message: rev A3 pcb, added a fun logo to the BIOS startup
Parts:
- renumbered C60 to C100, IC1 to U55
Connections:
- net ~{RESET} is gone; now on net +5V: U55.18 (~{RESET})
- net AD6: now reaches U55.10 (AD6)
- net AD7: now reaches U55.11 (AD7)
- net AEN: now reaches U55.14 (AS)
- net AD0: now reaches U55.4 (AD0)
- net AD1: now reaches U55.5 (AD1)
- net AD2: now reaches U55.6 (AD2)
- net AD3: now reaches U55.7 (AD3)
- net AD4: now reaches U55.8 (AD4)
- net AD5: now reaches U55.9 (AD5)
