File: 8088_addrbus.kicad_sch (KiCad schematic)
At the start: 26 parts, among them U3 74LS573, U4 74LS573, U5 74LS573

Commit message: bringing over learnings/improvements from prototype board
Parts:
- removed R36, R37, R38, R39, R40, R41, R42, R43, R44, R45, R46, R47, R48, R49, R50, R51, R52, R53, R54, R55: 10k, Resistor_SMD:R_0805_2012Metric, symbol Device:R_US
- added RN4, RN5, RN6: 10k, Resistor_THT:R_Array_SIP9, symbol Device:R_Network08
Connections:
- net +5V: now also RN4.1 (common), RN5.1 (common), RN6.1 (common)
- net 8088_A16: now also U5.2 (D0); no longer U5.5 (D3)
- net 8088_A17: now also U5.3 (D1); no longer U5.4 (D2)
- net 8088_A18: now also U5.4 (D2); no longer U5.3 (D1)
- net 8088_A19: now also U5.5 (D3); no longer U5.2 (D0)
- net A0: now also RN4.2 (R1)
- net A1: now also RN4.3 (R2)
- net A10: now also RN5.4 (R3)
- net A11: now also RN5.5 (R4)
- net A12: now also RN5.6 (R5)
- net A13: now also RN5.7 (R6)
- net A14: now also RN5.8 (R7)
- net A15: now also RN5.9 (R8)
- net A16: now also U5.19 (Q0), RN6.2 (R1); no longer U5.16 (Q3)
- net A17: now also U5.18 (Q1), RN6.3 (R2); no longer U5.17 (Q2)
- net A18: now also U5.17 (Q2), RN6.4 (R3); no longer U5.18 (Q1)
- net A19: now also U5.16 (Q3), RN6.5 (R4); no longer U5.19 (Q0)
- net A2: now also RN4.4 (R3)
- net A3: now also RN4.5 (R4)
- net A4: now also RN4.6 (R5)
- net A5: now also RN4.7 (R6)
- net A6: now also RN4.8 (R7)
- net A7: now also RN4.9 (R8)
- net A8: now also RN5.2 (R1)
- net A9: now also RN5.3 (R2)
- no-connect marks 4 -> 8

Commit message: more pcb routing, implementing learnings from the prototype board
Parts:
- removed RN6: 10k, Resistor_THT:R_Array_SIP9, symbol Device:R_Network08
- added RN12: R_Network04, Resistor_THT:R_Array_SIP5, symbol Device:R_Network04
Connections:
- net +5V: now also RN12.1 (common)
- net A16: now also RN12.2 (R1)
- net A17: now also RN12.3 (R2)
- net A18: now also RN12.4 (R3)
- net A19: now also RN12.5 (R4)
- no-connect marks 8 -> 4
Changed lines of the file:
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@@
 	)
 	(no_connect
-		(at 265.43 115.57)
-	)
-	(no_connect
-		(at 270.51 115.57)
-	)
-	(no_connect
-		(at 262.89 115.57)
-	)
-	(no_connect
-		(at 267.97 115.57)
-	)
-	(no_connect
 		(at 143.51 163.83)
 	)
@@
 	)
 	(symbol
+		(lib_id "Device:R_Network04")
+		(at 257.81 110.49 0)
+		(unit 1)
+		(exclude_from_sim no)
+		(in_bom yes)
+		(on_board yes)
+		(dnp no)
+		(fields_autoplaced yes)
+		(property "Reference" "RN12"
+			(at 262.89 109.4739 0)
+			(effects
+				(font
+					(size 1.27 1.27)
+				)
+				(justify left)
+			)
+		)
+		(property "Value" "R_Network04"
+			(at 262.89 112.0139 0)
+			(effects
+				(font
+					(size 1.27 1.27)
+				)
+				(justify left)
+			)
+		)
+		(property "Footprint" "Resistor_THT:R_Array_SIP5"
+			(at 264.795 110.49 90)
+			(effects
+				(font
+					(size 1.27 1.27)
+				)
+				(hide yes)
+			)
+		)
+		(property "Datasheet" "http://www.vishay.com/docs/31509/csc.pdf"
+			(at 257.81 110.49 0)
+			(effects
+				(font
+					(size 1.27 1.27)
+				)
+				(hide yes)
+			)
+		)
+		(property "Description" "4 resistor network, star topology, bussed resistors, small symbol"
+			(at 257.81 110.49 0)
+			(effects
+				(font
+					(size 1.27 1.27)
+				)
+				(hide yes)
+			)
+		)
+		(pin "1"
+		)
+		(pin "4"
+		)
+		(pin "2"
+		)
+		(pin "5"
+		)
+		(pin "3"
+		)
+		(instances
+			(project "sbc_8088"
+				(path "/5e468d94-0319-44d1-a77f-2adc451eed13/3d1f10e8-a4e0-41e6-95d9-dab1bfbc76fe"
+					(reference "RN12")
+					(unit 1)
+				)
+			)
+		)
+	)
+	(symbol
 		(lib_id "power:GND")
 		(at 130.81 67.31 0)
@@
 					(unit 1)
 				)
-			)
-		)
-	)
-	(symbol
-		(lib_id "Device:R_Network08")
-		(at 262.89 110.49 0)
-		(unit 1)
-		(exclude_from_sim no)
-		(in_bom yes)
-		(on_board yes)
-		(dnp no)
-		(fields_autoplaced yes)
-		(property "Reference" "RN6"
-			(at 273.05 109.4739 0)
-			(effects
-				(font
-					(size 1.27 1.27)
-				)
-				(justify left)
-			)
-		)
-		(property "Value" "10k"
-			(at 273.05 112.0139 0)
-			(effects
-				(font
-					(size 1.27 1.27)
-				)
-				(justify left)
-			)
-		)
-		(property "Footprint" "Resistor_THT:R_Array_SIP9"
-			(at 274.955 110.49 90)
-			(effects
-				(font
-					(size 1.27 1.27)
-				)
-				(hide yes)
-			)
-		)
-		(property "Datasheet" "http://www.vishay.com/docs/31509/csc.pdf"
-			(at 262.89 110.49 0)
-			(effects
-				(font
-					(size 1.27 1.27)
-				)
-				(hide yes)
-			)
-		)
-		(property "Description" "8 resistor network, star topology, bussed resistors, small symbol"
-			(at 262.89 110.49 0)
-			(effects
-				(font
-					(size 1.27 1.27)
-				)
-				(hide yes)
-			)
-		)
-		(pin "4"
-		)
-		(pin "8"
-		)
-		(pin "2"
-		)
-		(pin "9"
-		)
-		(pin "1"
-		)
-		(pin "7"
-		)
-		(pin "3"
-		)
-		(pin "6"
-		)
-		(pin "5"
-		)
-		(instances
-			(project "sbc_8088"
-				(path "/5e468d94-0319-44d1-a77f-2adc451eed13/3d1f10e8-a4e0-41e6-95d9-dab1bfbc76fe"
-					(reference "RN6")
-					(unit 1)
-				)

Commit message: pcb is fully routed, working on power capacitor tweaks, some ROM testing
Parts:
- renumbered C4 to C23, C3 to C30, RN12 to RN1, RN5 to RN3, RN4 to RN5, U5 to U1, U4 to U10, U3 to U14
Changed lines of the file:
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@@
 		(dnp no)
 		(fields_autoplaced yes)
-		(property "Reference" "C4"
+		(property "Reference" "C23"
 			(at 187.96 60.325 0)
 			(effects
@@
 			(project "sbc_8088"
 				(path "/5e468d94-0319-44d1-a77f-2adc451eed13/3d1f10e8-a4e0-41e6-95d9-dab1bfbc76fe"
-					(reference "C4")
+					(reference "C23")
 					(unit 1)
 				)
@@
 		(dnp no)
 		(fields_autoplaced yes)
-		(property "Reference" "RN5"
+		(property "Reference" "RN3"
 			(at 245.11 109.4739 0)
 			(effects
@@
 			(project "sbc_8088"
 				(path "/5e468d94-0319-44d1-a77f-2adc451eed13/3d1f10e8-a4e0-41e6-95d9-dab1bfbc76fe"
-					(reference "RN5")
+					(reference "RN3")
 					(unit 1)
 				)
@@
 		(dnp no)
 		(fields_autoplaced yes)
-		(property "Reference" "C3"
+		(property "Reference" "C30"
 			(at 175.26 60.325 0)
 			(effects
@@
 			(project "sbc_8088"
 				(path "/5e468d94-0319-44d1-a77f-2adc451eed13/3d1f10e8-a4e0-41e6-95d9-dab1bfbc76fe"
-					(reference "C3")
+					(reference "C30")
 					(unit 1)
 				)
@@
 		(dnp no)
 		(fields_autoplaced yes)
-		(property "Reference" "RN4"
+		(property "Reference" "RN5"
 			(at 217.17 109.4739 0)
 			(effects
@@
 			(project "sbc_8088"
 				(path "/5e468d94-0319-44d1-a77f-2adc451eed13/3d1f10e8-a4e0-41e6-95d9-dab1bfbc76fe"
-					(reference "RN4")
+					(reference "RN5")
 					(unit 1)
 				)
@@
 		(dnp no)
 		(fields_autoplaced yes)
-		(property "Reference" "U4"
+		(property "Reference" "U10"
 			(at 133.0041 83.82 0)
 			(effects
@@
 			(project "sbc_8088"
 				(path "/5e468d94-0319-44d1-a77f-2adc451eed13/3d1f10e8-a4e0-41e6-95d9-dab1bfbc76fe"
-					(reference "U4")
+					(reference "U10")
 					(unit 1)
 				)
@@
 		(dnp no)
 		(fields_autoplaced yes)
-		(property "Reference" "RN12"
+		(property "Reference" "RN1"
 			(at 262.89 109.4739 0)
 			(effects
@@
 			(project "sbc_8088"
 				(path "/5e468d94-0319-44d1-a77f-2adc451eed13/3d1f10e8-a4e0-41e6-95d9-dab1bfbc76fe"
-					(reference "RN12")
+					(reference "RN1")
 					(unit 1)
 				)
@@
 		(dnp no)
 		(fields_autoplaced yes)
-		(property "Reference" "U3"
+		(property "Reference" "U14"
 			(at 133.0041 24.13 0)
 			(effects
@@
 			(project "sbc_8088"
 				(path "/5e468d94-0319-44d1-a77f-2adc451eed13/3d1f10e8-a4e0-41e6-95d9-dab1bfbc76fe"
-					(reference "U3")
+					(reference "U14")
 					(unit 1)
 				)
@@
 		(dnp no)
 		(fields_autoplaced yes)
-		(property "Reference" "U5"
+		(property "Reference" "U1"
 			(at 133.0041 140.97 0)
 			(effects
@@
 			(project "sbc_8088"
 				(path "/5e468d94-0319-44d1-a77f-2adc451eed13/3d1f10e8-a4e0-41e6-95d9-dab1bfbc76fe"
-					(reference "U5")
-					(unit 1)
-				)
+					(reference "U1")
+					(unit 1)
+				)

Commit message: added ATtiny for SMC, added PC speaker
Parts:
- renumbered C23 to C28, C30 to C35, U10 to U12, U14 to U15, U1 to U2
Changed lines of the file:
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@@
 		(dnp no)
 		(fields_autoplaced yes)
-		(property "Reference" "C23"
+		(property "Reference" "C28"
 			(at 187.96 60.325 0)
 			(effects
@@
 			(project "sbc_8088"
 				(path "/5e468d94-0319-44d1-a77f-2adc451eed13/3d1f10e8-a4e0-41e6-95d9-dab1bfbc76fe"
-					(reference "C23")
+					(reference "C28")
 					(unit 1)
 				)
@@
 		(dnp no)
 		(fields_autoplaced yes)
-		(property "Reference" "C30"
+		(property "Reference" "C35"
 			(at 175.26 60.325 0)
 			(effects
@@
 			(project "sbc_8088"
 				(path "/5e468d94-0319-44d1-a77f-2adc451eed13/3d1f10e8-a4e0-41e6-95d9-dab1bfbc76fe"
-					(reference "C30")
+					(reference "C35")
 					(unit 1)
 				)
@@
 		(dnp no)
 		(fields_autoplaced yes)
-		(property "Reference" "U10"
+		(property "Reference" "U12"
 			(at 133.0041 83.82 0)
 			(effects
@@
 			(project "sbc_8088"
 				(path "/5e468d94-0319-44d1-a77f-2adc451eed13/3d1f10e8-a4e0-41e6-95d9-dab1bfbc76fe"
-					(reference "U10")
+					(reference "U12")
 					(unit 1)
 				)
@@
 		(dnp no)
 		(fields_autoplaced yes)
-		(property "Reference" "U14"
+		(property "Reference" "U15"
 			(at 133.0041 24.13 0)
 			(effects
@@
 			(project "sbc_8088"
 				(path "/5e468d94-0319-44d1-a77f-2adc451eed13/3d1f10e8-a4e0-41e6-95d9-dab1bfbc76fe"
-					(reference "U14")
+					(reference "U15")
 					(unit 1)
 				)
@@
 		(dnp no)
 		(fields_autoplaced yes)
-		(property "Reference" "U1"
+		(property "Reference" "U2"
 			(at 133.0041 140.97 0)
 			(effects
@@
 			(project "sbc_8088"
 				(path "/5e468d94-0319-44d1-a77f-2adc451eed13/3d1f10e8-a4e0-41e6-95d9-dab1bfbc76fe"
-					(reference "U1")
-					(unit 1)
-				)
+					(reference "U2")
+					(unit 1)
+				)

Commit message: fixes, prep for final production run
Parts:
- C28, C35, C5: LCSC Part # (none) -> C1853649
- RN1: LCSC Part # (none) -> C11394
- RN3, RN5: LCSC Part # (none) -> C8692
- U12, U15, U2: LCSC Part # (none) -> C72118

Commit message: bump cpu to 8mhz, add second clock gen for ISA bus and PIT
Connections:
- net 8088_A16: now also U2.6 (D4); no longer U2.2 (D0)
- net 8088_A17: now also U2.7 (D5); no longer U2.3 (D1)
- net 8088_A18: now also U2.8 (D6); no longer U2.4 (D2)
- net 8088_A19: now also U2.9 (D7); no longer U2.5 (D3)
- net A16: now also U2.15 (Q4); no longer U2.19 (Q0)
- net A17: now also U2.14 (Q5); no longer U2.18 (Q1)
- net A18: now also U2.13 (Q6); no longer U2.17 (Q2)
- net A19: now also U2.12 (Q7); no longer U2.16 (Q3)
- net GND: now also U2.2 (D0), U2.3 (D1), U2.4 (D2), U2.5 (D3); no longer U2.6 (D4), U2.7 (D5), U2.8 (D6), U2.9 (D7)

Commit message: no more SMT for isa_i2c, tweak motherboard multiplex logic, handful of other tweaks
Other:
- moved on the sheet: C28, C35, C5
Changed lines of the file:
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@@
 	)
 	(junction
+		(at 191.77 70.485)
+		(diameter 0)
+		(color 0 0 0 0)
+	)
+	(junction
 		(at 236.22 105.41)
 		(diameter 0)
@@
 	)
 	(junction
+		(at 191.77 53.975)
+		(diameter 0)
+		(color 0 0 0 0)
+	)
+	(junction
 		(at 85.09 101.6)
 		(diameter 0)
@@
 	(wire
 		(pts
-			(xy 184.15 70.485) (xy 198.12 70.485)
+			(xy 184.15 70.485) (xy 191.77 70.485)
 		)
 		(stroke
@@
 	(wire
 		(pts
-			(xy 184.15 65.405) (xy 184.15 70.485)
+			(xy 191.77 64.77) (xy 191.77 70.485)
 		)
 		(stroke
@@
 	(wire
 		(pts
-			(xy 184.15 53.975) (xy 171.45 53.975)
+			(xy 184.15 53.975) (xy 165.1 53.975)
 		)
 		(stroke
@@
 	(wire
 		(pts
-			(xy 198.12 53.975) (xy 198.12 57.785)
+			(xy 217.17 53.975) (xy 217.17 57.15)
 		)
 		(stroke
@@
 	(wire
 		(pts
-			(xy 171.45 53.975) (xy 171.45 57.785)
+			(xy 165.1 53.975) (xy 165.1 57.15)
 		)
 		(stroke
@@
 	(wire
 		(pts
-			(xy 171.45 70.485) (xy 184.15 70.485)
+			(xy 165.1 70.485) (xy 184.15 70.485)
 		)
 		(stroke
@@
 	(wire
 		(pts
-			(xy 198.12 70.485) (xy 198.12 65.405)
+			(xy 217.17 70.485) (xy 217.17 64.77)
 		)
 		(stroke
@@
 	(wire
 		(pts
-			(xy 184.15 53.975) (xy 184.15 57.785)
+			(xy 191.77 53.975) (xy 191.77 57.15)
 		)
 		(stroke
@@
 	(wire
 		(pts
-			(xy 184.15 53.975) (xy 198.12 53.975)
+			(xy 184.15 53.975) (xy 191.77 53.975)
 		)
 		(stroke
@@
 	(wire
 		(pts
-			(xy 171.45 65.405) (xy 171.45 70.485)
+			(xy 165.1 64.77) (xy 165.1 70.485)
+		)
+		(stroke
+			(width 0)
+			(type default)
+		)
+	)
+	(wire
+		(pts
+			(xy 191.77 53.975) (xy 217.17 53.975)
 		)
 		(stroke
@@
 	(wire
 		(pts
+			(xy 191.77 70.485) (xy 217.17 70.485)
+		)
+		(stroke
+			(width 0)
+			(type default)
+		)
+	)
+	(wire
+		(pts
 			(xy 236.22 95.25) (xy 236.22 105.41)
 		)
@@
 	(symbol
 		(lib_id "Device:C")
-		(at 184.15 61.595 0)
+		(at 191.77 60.96 0)
 		(unit 1)
 		(exclude_from_sim no)
@@
 		(fields_autoplaced yes)
 		(property "Reference" "C28"
-			(at 187.96 60.325 0)
+			(at 195.58 59.69 0)
 			(effects
 				(font
@@
 		)
 		(property "Value" "0.1uF 20% Ceramic"
-			(at 187.96 62.865 0)
+			(at 195.58 62.23 0)
 			(effects
 				(font
@@
 		)
 		(property "Footprint" "Capacitor_SMD:C_0805_2012Metric"
-			(at 185.1152 65.405 0)
+			(at 192.7352 64.77 0)
 			(effects
 				(font
@@
 		)
 		(property "Datasheet" "~"
-			(at 184.15 61.595 0)
+			(at 191.77 60.96 0)
 			(effects
 				(font
@@
 		)
 		(property "Description" "LCSC #C1853649"
-			(at 184.15 61.595 0)
+			(at 191.77 60.96 0)
 			(effects
 				(font
@@
 		)
 		(property "Height" ""
-			(at 184.15 61.595 0)
+			(at 191.77 60.96 0)
 			(effects
 				(font
@@
 		)
 		(property "Manufacturer_Name" ""
-			(at 184.15 61.595 0)
+			(at 191.77 60.96 0)
 			(effects
 				(font
@@
 		)
 		(property "Manufacturer_Part_Number" ""
-			(at 184.15 61.595 0)
+			(at 191.77 60.96 0)
 			(effects
 				(font
@@
 		)
 		(property "Mouser Part Number" ""
-			(at 184.15 61.595 0)
+			(at 191.77 60.96 0)
 			(effects
 				(font
@@
 		)
 		(property "Mouser Price/Stock" ""
-			(at 184.15 61.595 0)
+			(at 191.77 60.96 0)
 			(effects
 				(font
@@
 		)
 		(property "LCSC Part #" "C1853649"
-			(at 184.15 61.595 0)
+			(at 191.77 60.96 0)
 			(effects
 				(font
@@
 	(symbol
 		(lib_id "Device:C")
-		(at 198.12 61.595 0)
+		(at 217.17 60.96 0)
 		(unit 1)
 		(exclude_from_sim no)
@@
 		(fields_autoplaced yes)
 		(property "Reference" "C5"
-			(at 201.93 60.325 0)
+			(at 220.98 59.69 0)
 			(effects
 				(font
@@
 		)
 		(property "Value" "0.1uF 20% Ceramic"
-			(at 201.93 62.865 0)
+			(at 220.98 62.23 0)
 			(effects
 				(font
@@
 		)
 		(property "Footprint" "Capacitor_SMD:C_0805_2012Metric"
-			(at 199.0852 65.405 0)
+			(at 218.1352 64.77 0)
 			(effects
 				(font
@@
 		)
 		(property "Datasheet" "~"
-			(at 198.12 61.595 0)
+			(at 217.17 60.96 0)
 			(effects
 				(font
@@
 		)
 		(property "Description" "LCSC #C1853649"
-			(at 198.12 61.595 0)
+			(at 217.17 60.96 0)
 			(effects
 				(font
@@
 		)
 		(property "Height" ""
-			(at 198.12 61.595 0)
+			(at 217.17 60.96 0)
 			(effects
 				(font
@@
 		)
 		(property "Manufacturer_Name" ""
-			(at 198.12 61.595 0)
+			(at 217.17 60.96 0)
 			(effects
 				(font
@@
 		)
 		(property "Manufacturer_Part_Number" ""
-			(at 198.12 61.595 0)
+			(at 217.17 60.96 0)
 			(effects
 				(font
@@
 		)
 		(property "Mouser Part Number" ""
-			(at 198.12 61.595 0)
+			(at 217.17 60.96 0)
 			(effects
 				(font
@@
 		)
 		(property "Mouser Price/Stock" ""
-			(at 198.12 61.595 0)
+			(at 217.17 60.96 0)
 			(effects
 				(font
@@
 		)
 		(property "LCSC Part #" "C1853649"
-			(at 198.12 61.595 0)
+			(at 217.17 60.96 0)
 			(effects
 				(font
@@
 	(symbol
 		(lib_id "Device:C")
-		(at 171.45 61.595 0)
+		(at 165.1 60.96 0)
 		(unit 1)
 		(exclude_from_sim no)
@@
 		(fields_autoplaced yes)
 		(property "Reference" "C35"
-			(at 175.26 60.325 0)
+			(at 168.91 59.69 0)
 			(effects
 				(font
@@
 		)
 		(property "Value" "0.1uF 20% Ceramic"
-			(at 175.26 62.865 0)
+			(at 168.91 62.23 0)
 			(effects
 				(font
@@
 		)
 		(property "Footprint" "Capacitor_SMD:C_0805_2012Metric"
-			(at 172.4152 65.405 0)
+			(at 166.0652 64.77 0)
 			(effects
 				(font
@@
 		)
 		(property "Datasheet" "~"
-			(at 171.45 61.595 0)
+			(at 165.1 60.96 0)
 			(effects
 				(font
@@
 		)
 		(property "Description" "LCSC #C1853649"
-			(at 171.45 61.595 0)
+			(at 165.1 60.96 0)
 			(effects
 				(font
@@
 		)
 		(property "Height" ""
-			(at 171.45 61.595 0)
+			(at 165.1 60.96 0)
 			(effects
 				(font
@@
 		)
 		(property "Manufacturer_Name" ""
-			(at 171.45 61.595 0)
+			(at 165.1 60.96 0)
 			(effects
 				(font
@@
 		)
 		(property "Manufacturer_Part_Number" ""
-			(at 171.45 61.595 0)
+			(at 165.1 60.96 0)
 			(effects
 				(font
@@
 		)
 		(property "Mouser Part Number" ""
-			(at 171.45 61.595 0)
+			(at 165.1 60.96 0)
 			(effects
 				(font
@@
 		)
 		(property "Mouser Price/Stock" ""
-			(at 171.45 61.595 0)
+			(at 165.1 60.96 0)
 			(effects
 				(font
@@
 		)
 		(property "LCSC Part #" "C1853649"
-			(at 171.45 61.595 0)
+			(at 165.1 60.96 0)
 			(effects
 				(font
