File: 8088_addrbus.kicad_sch (KiCad schematic)
At the start: 9 parts, among them U12 74LS573, U15 74LS573, U2 74LS573

Commit message: motherboard tweaks for manufacturing run, i2c card tweaks for manufacturing run, de9 -> stemma adapter idea for the i2c card
Parts:
- C28, C35, C5: LCSC Part # C1853649 -> C49678
- RN1: value R_Network04 -> 10k (bussed)
- RN3, RN5: value 10k -> 10k (bussed)
Changed lines of the file:
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@@
 			)
 		)
-		(property "Description" "LCSC #C1853649"
+		(property "Description" "LCSC #C49678"
 			(at 191.77 60.96 0)
 			(effects
@@
 			)
 		)
-		(property "LCSC Part #" "C1853649"
+		(property "LCSC Part #" "C49678"
 			(at 191.77 60.96 0)
 			(effects
@@
 			)
 		)
-		(property "Value" "10k"
+		(property "Value" "10k (bussed)"
 			(at 245.11 112.0139 0)
 			(effects
@@
 			)
 		)
-		(property "Description" "LCSC #C1853649"
+		(property "Description" "LCSC #C49678"
 			(at 217.17 60.96 0)
 			(effects
@@
 			)
 		)
-		(property "LCSC Part #" "C1853649"
+		(property "LCSC Part #" "C49678"
 			(at 217.17 60.96 0)
 			(effects
@@
 			)
 		)
-		(property "Description" "LCSC #C1853649"
+		(property "Description" "LCSC #C49678"
 			(at 165.1 60.96 0)
 			(effects
@@
 			)
 		)
-		(property "LCSC Part #" "C1853649"
+		(property "LCSC Part #" "C49678"
 			(at 165.1 60.96 0)
 			(effects
@@
 			)
 		)
-		(property "Value" "10k"
+		(property "Value" "10k (bussed)"
 			(at 217.17 112.0139 0)
 			(effects
@@
 			)
 		)
-		(property "Value" "R_Network04"
+		(property "Value" "10k (bussed)"
 			(at 262.89 112.0139 0)
 			(effects
