File: i2c.kicad_sch (KiCad schematic)
At the start: 12 parts, among them J14 Conn_02x04_Counter_Clockwise, J15 Conn_02x04_Counter_Clockwise, J16 Conn_02x04_Counter_Clockwise, J17 Conn_02x04_Counter_Clockwise, J18 Conn_02x04_Counter_Clockwise, J19 Conn_02x04_Counter_Clockwise, J3 Conn_02x04_Counter_Clockwise, J9 Conn_02x04_Counter_Clockwise, U5 PCF8584

Commit message: no more SMT for isa_i2c, tweak motherboard multiplex logic, handful of other tweaks
Parts:
- removed J14, J17, J3, J9: Conn_02x04_Counter_Clockwise, Connector_PinSocket_2.54mm:PinSocket_2x05_P2.54mm_Vertical, symbol Connector_Generic:Conn_02x05_Counter_Clockwise
- removed J15, J16, J18, J19: Conn_02x04_Counter_Clockwise, Connector_PinSocket_2.54mm:PinSocket_2x05_P2.54mm_Horizontal, symbol Connector_Generic:Conn_02x05_Counter_Clockwise
- added J14, J15, J3, J9: Conn_01x04, Connector_JST:JST_SH_BM04B-SRSS-TB_1x04-1MP_P1.00mm_Vertical, symbol Connector_Generic:Conn_01x04
- added J16, J17: Conn_01x04, Connector_JST:JST_SH_SM04B-SRSS-TB_1x04-1MP_P1.00mm_Horizontal, symbol Connector_Generic:Conn_01x04
Connections:
- net +5V: now also J14.3 (Pin_3), J15.3 (Pin_3), J16.3 (Pin_3), J17.3 (Pin_3), J3.3 (Pin_3), J9.3 (Pin_3)
- net GND: now also J14.4 (Pin_4), J15.4 (Pin_4), J16.4 (Pin_4), J17.4 (Pin_4), J3.4 (Pin_4), J9.4 (Pin_4)
- net SCL: now also J14.1 (Pin_1), J15.1 (Pin_1), J16.1 (Pin_1), J17.1 (Pin_1), J3.1 (Pin_1), J9.1 (Pin_1)
- net SDA: now also J14.2 (Pin_2), J15.2 (Pin_2), J16.2 (Pin_2), J17.2 (Pin_2), J3.2 (Pin_2), J9.2 (Pin_2)
- no-connect marks 17 -> 1
Other:
- note added: "STEMMA QT I2C SOCKETS @ +5V"
- note added: "The PCF8584 is a little hard to get in 2024, but the newer PCA9564 is dificult to get in a DIP form factor. The ISA-to-I2C card will use the PCA9564 - the M88 motherboard can use the legacy chip."
- note removed: "M88 I2C CARD BUS MAIN BOARD BLOCK"
- note removed: "M88 I2C CARD BUS REAR I/O PANEL BLOCK"

Commit message: simplify m88 logic further, reduce ICs, reorient the POST display, use an oscillator for 14.31818 MHz, update isa-i2c bridge BOM
Parts:
- J14, J15, J3, J9: footprint Connector_JST:JST_SH_BM04B-SRSS-TB_1x04-1MP_P1.00mm_Vertical -> Connector_JST:JST_PH_S4B-PH-K_1x04_P2.00mm_Horizontal; LCSC Part # (none) -> C157926; Manufacturer_Name (none) -> JST; Manufacturer_Part_Number (none) -> S4B-PH-K-S(LF)(SN)
- J16, J17: footprint Connector_JST:JST_SH_SM04B-SRSS-TB_1x04-1MP_P1.00mm_Horizontal -> Connector_JST:JST_PH_S4B-PH-K_1x04_P2.00mm_Horizontal; LCSC Part # (none) -> C157926; Manufacturer_Name (none) -> JST; Manufacturer_Part_Number (none) -> S4B-PH-K-S(LF)(SN)
- R59, R60: footprint Resistor_SMD:R_0805_2012Metric -> Resistor_SMD:R_0603_1608Metric; LCSC Part # (none) -> C4190
- U5: LCSC Part # C7442 -> C72118
Other:
- note added: "STEMMA I2C SOCKETS @ +5V"
- note removed: "STEMMA QT I2C SOCKETS @ +5V"
Changed lines of the file:
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@@
 		)
 	)
-	(text "STEMMA QT I2C SOCKETS @ +5V"
+	(text "STEMMA I2C SOCKETS @ +5V"
 		(exclude_from_sim no)
 		(at 128.016 26.162 0)
@@
 			)
 		)
-		(property "Footprint" "Connector_JST:JST_SH_SM04B-SRSS-TB_1x04-1MP_P1.00mm_Horizontal"
+		(property "Footprint" "Connector_JST:JST_PH_S4B-PH-K_1x04_P2.00mm_Horizontal"
 			(at 105.41 91.44 0)
 			(effects
@@
 			)
 		)
-		(property "Description" "Generic connector, single row, 01x04, script generated (kicad-library-utils/schlib/autogen/connector/)"
+		(property "Description" "LCSC #C157926"
+			(at 105.41 91.44 0)
+			(effects
+				(font
+					(size 1.27 1.27)
+				)
+				(hide yes)
+			)
+		)
+		(property "LCSC Part #" "C157926"
+			(at 105.41 91.44 0)
+			(effects
+				(font
+					(size 1.27 1.27)
+				)
+				(hide yes)
+			)
+		)
+		(property "Manufacturer_Name" "JST"
+			(at 105.41 91.44 0)
+			(effects
+				(font
+					(size 1.27 1.27)
+				)
+				(hide yes)
+			)
+		)
+		(property "Manufacturer_Part_Number" " S4B-PH-K-S(LF)(SN)"
 			(at 105.41 91.44 0)
 			(effects
@@
 			)
 		)
-		(property "Footprint" "Connector_JST:JST_SH_BM04B-SRSS-TB_1x04-1MP_P1.00mm_Vertical"
+		(property "Footprint" "Connector_JST:JST_PH_S4B-PH-K_1x04_P2.00mm_Horizontal"
 			(at 151.13 67.31 0)
 			(effects
@@
 			)
 		)
-		(property "Description" "Generic connector, single row, 01x04, script generated (kicad-library-utils/schlib/autogen/connector/)"
+		(property "Description" "LCSC #C157926"
+			(at 151.13 67.31 0)
+			(effects
+				(font
+					(size 1.27 1.27)
+				)
+				(hide yes)
+			)
+		)
+		(property "LCSC Part #" "C157926"
+			(at 151.13 67.31 0)
+			(effects
+				(font
+					(size 1.27 1.27)
+				)
+				(hide yes)
+			)
+		)
+		(property "Manufacturer_Name" "JST"
+			(at 151.13 67.31 0)
+			(effects
+				(font
+					(size 1.27 1.27)
+				)
+				(hide yes)
+			)
+		)
+		(property "Manufacturer_Part_Number" " S4B-PH-K-S(LF)(SN)"
 			(at 151.13 67.31 0)
 			(effects
@@
 			)
 		)
-		(property "Footprint" "Connector_JST:JST_SH_BM04B-SRSS-TB_1x04-1MP_P1.00mm_Vertical"
+		(property "Footprint" "Connector_JST:JST_PH_S4B-PH-K_1x04_P2.00mm_Horizontal"
 			(at 105.41 43.18 0)
 			(effects
@@
 			)
 		)
-		(property "Description" "Generic connector, single row, 01x04, script generated (kicad-library-utils/schlib/autogen/connector/)"
+		(property "Description" "LCSC #C157926"
+			(at 105.41 43.18 0)
+			(effects
+				(font
+					(size 1.27 1.27)
+				)
+				(hide yes)
+			)
+		)
+		(property "LCSC Part #" "C157926"
+			(at 105.41 43.18 0)
+			(effects
+				(font
+					(size 1.27 1.27)
+				)
+				(hide yes)
+			)
+		)
+		(property "Manufacturer_Name" "JST"
+			(at 105.41 43.18 0)
+			(effects
+				(font
+					(size 1.27 1.27)
+				)
+				(hide yes)
+			)
+		)
+		(property "Manufacturer_Part_Number" " S4B-PH-K-S(LF)(SN)"
 			(at 105.41 43.18 0)
 			(effects
@@
 			)
 		)
-		(property "Footprint" "Resistor_SMD:R_0805_2012Metric"
+		(property "Footprint" "Resistor_SMD:R_0603_1608Metric"
 			(at 40.64 66.04 0)
 			(effects
@@
 			)
 		)
-		(property "Description" "Resistor, small US symbol"
+		(property "Description" "LCSC #C4190"
 			(at 40.64 66.04 0)
 			(effects
@@
 			)
 		)
-		(property "LCSC Part #" ""
+		(property "LCSC Part #" "C4190"
 			(at 40.64 66.04 0)
 			(effects
@@
 			)
 		)
-		(property "Footprint" "Resistor_SMD:R_0805_2012Metric"
+		(property "Footprint" "Resistor_SMD:R_0603_1608Metric"
 			(at 34.29 57.15 0)
 			(effects
@@
 			)
 		)
-		(property "Description" "Resistor, small US symbol"
+		(property "Description" "LCSC #C4190"
 			(at 34.29 57.15 0)
 			(effects
@@
 			)
 		)
-		(property "LCSC Part #" ""
+		(property "LCSC Part #" "C4190"
 			(at 34.29 57.15 0)
 			(effects
@@
 			)
 		)
-		(property "Footprint" "Connector_JST:JST_SH_SM04B-SRSS-TB_1x04-1MP_P1.00mm_Horizontal"
+		(property "Footprint" "Connector_JST:JST_PH_S4B-PH-K_1x04_P2.00mm_Horizontal"
 			(at 151.13 91.44 0)
 			(effects
@@
 			)
 		)
-		(property "Description" "Generic connector, single row, 01x04, script generated (kicad-library-utils/schlib/autogen/connector/)"
+		(property "Description" "LCSC #C157926"
+			(at 151.13 91.44 0)
+			(effects
+				(font
+					(size 1.27 1.27)
+				)
+				(hide yes)
+			)
+		)
+		(property "LCSC Part #" "C157926"
+			(at 151.13 91.44 0)
+			(effects
+				(font
+					(size 1.27 1.27)
+				)
+				(hide yes)
+			)
+		)
+		(property "Manufacturer_Name" "JST"
+			(at 151.13 91.44 0)
+			(effects
+				(font
+					(size 1.27 1.27)
+				)
+				(hide yes)
+			)
+		)
+		(property "Manufacturer_Part_Number" " S4B-PH-K-S(LF)(SN)"
 			(at 151.13 91.44 0)
 			(effects
@@
 			)
 		)
-		(property "Footprint" "Connector_JST:JST_SH_BM04B-SRSS-TB_1x04-1MP_P1.00mm_Vertical"
+		(property "Footprint" "Connector_JST:JST_PH_S4B-PH-K_1x04_P2.00mm_Horizontal"
 			(at 151.13 43.18 0)
 			(effects
@@
 			)
 		)
-		(property "Description" "Generic connector, single row, 01x04, script generated (kicad-library-utils/schlib/autogen/connector/)"
+		(property "Description" "LCSC #C157926"
+			(at 151.13 43.18 0)
+			(effects
+				(font
+					(size 1.27 1.27)
+				)
+				(hide yes)
+			)
+		)
+		(property "LCSC Part #" "C157926"
+			(at 151.13 43.18 0)
+			(effects
+				(font
+					(size 1.27 1.27)
+				)
+				(hide yes)
+			)
+		)
+		(property "Manufacturer_Name" "JST"
+			(at 151.13 43.18 0)
+			(effects
+				(font
+					(size 1.27 1.27)
+				)
+				(hide yes)
+			)
+		)
+		(property "Manufacturer_Part_Number" " S4B-PH-K-S(LF)(SN)"
 			(at 151.13 43.18 0)
 			(effects
@@
 			)
 		)
-		(property "Footprint" "Connector_JST:JST_SH_BM04B-SRSS-TB_1x04-1MP_P1.00mm_Vertical"
+		(property "Footprint" "Connector_JST:JST_PH_S4B-PH-K_1x04_P2.00mm_Horizontal"
 			(at 105.41 67.31 0)
 			(effects
@@
 			)
 		)
-		(property "Description" "Generic connector, single row, 01x04, script generated (kicad-library-utils/schlib/autogen/connector/)"
+		(property "Description" "LCSC #C157926"
+			(at 105.41 67.31 0)
+			(effects
+				(font
+					(size 1.27 1.27)
+				)
+				(hide yes)
+			)
+		)
+		(property "LCSC Part #" "C157926"
+			(at 105.41 67.31 0)
+			(effects
+				(font
+					(size 1.27 1.27)
+				)
+				(hide yes)
+			)
+		)
+		(property "Manufacturer_Name" "JST"
+			(at 105.41 67.31 0)
+			(effects
+				(font
+					(size 1.27 1.27)
+				)
+				(hide yes)
+			)
+		)
+		(property "Manufacturer_Part_Number" " S4B-PH-K-S(LF)(SN)"
 			(at 105.41 67.31 0)
 			(effects
@@
 			)
 		)
-		(property "Description" "I2C Bus Controller, DIP/SOIC-20"
+		(property "Description" "LCSC #C72118 "
 			(at 245.11 68.58 0)
 			(effects
@@
 			)
 		)
-		(property "LCSC Part #" "C7442"
+		(property "LCSC Part #" "C72118 "
 			(at 245.11 68.58 0)
 			(effects

Commit message: motherboard tweaks for manufacturing run, i2c card tweaks for manufacturing run, de9 -> stemma adapter idea for the i2c card
Parts:
- C6: LCSC Part # C1853649 -> C49678
- R59, R60: LCSC Part # C4190 -> C17520
Changed lines of the file:
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@@
 			)
 		)
-		(property "Description" "LCSC #C1853649"
+		(property "Description" "LCSC #C49678"
 			(at 261.62 36.83 0)
 			(effects
@@
 			)
 		)
-		(property "LCSC Part #" "C1853649"
+		(property "LCSC Part #" "C49678"
 			(at 261.62 36.83 0)
 			(effects
@@
 			)
 		)
-		(property "Description" "LCSC #C4190"
-			(at 40.64 66.04 0)
-			(effects
-				(font
-					(size 1.27 1.27)
-				)
-				(hide yes)
-			)
-		)
-		(property "LCSC Part #" "C4190"
+		(property "Description" "LCSC #C17520"
+			(at 40.64 66.04 0)
+			(effects
+				(font
+					(size 1.27 1.27)
+				)
+				(hide yes)
+			)
+		)
+		(property "LCSC Part #" "C17520"
 			(at 40.64 66.04 0)
 			(effects
@@
 			)
 		)
-		(property "Description" "LCSC #C4190"
+		(property "Description" "LCSC #C17520"
 			(at 34.29 57.15 0)
 			(effects
@@
 			)
 		)
-		(property "LCSC Part #" "C4190"
+		(property "LCSC Part #" "C17520"
 			(at 34.29 57.15 0)
 			(effects
