File: ppi.kicad_sch (KiCad schematic)
At the start: 14 parts, among them J7 PC Speaker, U10 74LS125, U13 74LS244, U17 74LS175

Commit message: more work on test BIOS, porting stuff to C
Parts:
- U6: value ~ -> 75477
Changed lines of the file:
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@@
 		(shape output)
 		(at 256.54 120.65 0)
+		(fields_autoplaced yes)
 		(effects
 			(font
@@
 			)
 		)
-		(property "Value" "~"
+		(property "Value" "75477"
 			(at 192.6941 39.37 0)
 			(effects

Commit message: working on removing DMA for now
Changed lines of the file:
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@@
 	(wire
 		(pts
-			(xy 224.79 151.13) (xy 224.79 153.67)
+			(xy 224.79 151.13) (xy 224.79 154.94)
 		)
 		(stroke
@@
 	)
 	(symbol
-		(lib_id "power:GND")
-		(at 143.51 191.77 0)
-		(unit 1)
-		(exclude_from_sim no)
-		(in_bom yes)
-		(on_board yes)
-		(dnp no)
-		(fields_autoplaced yes)
-		(property "Reference" "#PWR0311"
-			(at 143.51 198.12 0)
-			(effects
-				(font
-					(size 1.27 1.27)
-				)
-				(hide yes)
-			)
-		)
-		(property "Value" "GND"
-			(at 143.51 196.85 0)
-			(effects
-				(font
-					(size 1.27 1.27)
-				)
-			)
-		)
-		(property "Footprint" ""
-			(at 143.51 191.77 0)
-			(effects
-				(font
-					(size 1.27 1.27)
-				)
-				(hide yes)
-			)
-		)
-		(property "Datasheet" ""
-			(at 143.51 191.77 0)
-			(effects
-				(font
-					(size 1.27 1.27)
-				)
-				(hide yes)
-			)
-		)
-		(property "Description" ""
-			(at 143.51 191.77 0)
-			(effects
-				(font
-					(size 1.27 1.27)
-				)
-				(hide yes)
-			)
-		)
-		(pin "1"
-		)
-		(instances
-			(project "sbc_8088"
-				(path "/5e468d94-0319-44d1-a77f-2adc451eed13/0e663061-fd9f-4de5-946e-4939a5fe656c"
-					(reference "#PWR0311")
-					(unit 1)
-				)
-			)
-		)
-	)
-	(symbol
 		(lib_id "power:+5V")
 		(at 163.83 52.07 0)
@@
 	)
 	(symbol
-		(lib_id "power:GND")
-		(at 87.63 191.77 0)
-		(unit 1)
-		(exclude_from_sim no)
-		(in_bom yes)
-		(on_board yes)
-		(dnp no)
-		(fields_autoplaced yes)
-		(property "Reference" "#PWR0312"
-			(at 87.63 198.12 0)
-			(effects
-				(font
-					(size 1.27 1.27)
-				)
-				(hide yes)
-			)
-		)
-		(property "Value" "GND"
-			(at 87.63 196.85 0)
-			(effects
-				(font
-					(size 1.27 1.27)
-				)
-			)
-		)
-		(property "Footprint" ""
-			(at 87.63 191.77 0)
-			(effects
-				(font
-					(size 1.27 1.27)
-				)
-				(hide yes)
-			)
-		)
-		(property "Datasheet" ""
-			(at 87.63 191.77 0)
-			(effects
-				(font
-					(size 1.27 1.27)
-				)
-				(hide yes)
-			)
-		)
-		(property "Description" ""
-			(at 87.63 191.77 0)
-			(effects
-				(font
-					(size 1.27 1.27)
-				)
-				(hide yes)
-			)
-		)
-		(pin "1"
-		)
-		(instances
-			(project "sbc_8088"
-				(path "/5e468d94-0319-44d1-a77f-2adc451eed13/0e663061-fd9f-4de5-946e-4939a5fe656c"
-					(reference "#PWR0312")
-					(unit 1)
-				)
-			)
-		)
-	)
-	(symbol
 		(lib_id "74xx:74LS175")
 		(at 224.79 130.81 0)
@@
 	(symbol
 		(lib_id "power:GND")
-		(at 224.79 153.67 0)
+		(at 224.79 154.94 0)
 		(unit 1)
 		(exclude_from_sim no)
@@
 		(fields_autoplaced yes)
 		(property "Reference" "#PWR0301"
+			(at 224.79 161.29 0)
+			(effects
+				(font
+					(size 1.27 1.27)
+				)
+				(hide yes)
+			)
+		)
+		(property "Value" "GND"
 			(at 224.79 160.02 0)
 			(effects
@@
 					(size 1.27 1.27)
 				)
-				(hide yes)
-			)
-		)
-		(property "Value" "GND"
-			(at 224.79 158.75 0)
-			(effects
-				(font
-					(size 1.27 1.27)
-				)
 			)
 		)
 		(property "Footprint" ""
-			(at 224.79 153.67 0)
+			(at 224.79 154.94 0)
 			(effects
 				(font
@@
 		)
 		(property "Datasheet" ""
-			(at 224.79 153.67 0)
+			(at 224.79 154.94 0)
 			(effects
 				(font
@@
 		)
 		(property "Description" ""
-			(at 224.79 153.67 0)
-			(effects
-				(font
+			(at 224.79 154.94 0)
+			(effects
+				(font

Commit message: fixes, prep for final production run
Parts:
- C17, C25, C29, C30: LCSC Part # (none) -> C1853649
- C20: LCSC Part # (none) -> C2180714
- J7: LCSC Part # (none) -> C6332197
- R4: LCSC Part # (none) -> C706316
- R5, R6, R7: LCSC Part # (none) -> C84376
- U10: LCSC Part # (none) -> C72114
- U13: LCSC Part # (none) -> C72118
- U17: LCSC Part # (none) -> C72115
- U6: LCSC Part # (none) -> C72124

Commit message: part tweaks, BOM is pretty much finalized, use 0.5W resistors for bleeders
Parts:
- R4: LCSC Part # C706316 -> C706383
Changed lines of the file:
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@@
 			)
 		)
-		(property "Description" "LCSC #C706316 "
+		(property "Description" "LCSC #C706383"
 			(at 251.46 55.88 0)
 			(effects
@@
 			)
 		)
-		(property "LCSC Part #" "C706316 "
+		(property "LCSC Part #" "C706383"
 			(at 251.46 55.88 0)
 			(effects

Commit message: no more SMT for isa_i2c, tweak motherboard multiplex logic, handful of other tweaks
Connections:
- net +5V: now also U10.13
- net GND: no longer U10.13
Other:
- moved on the sheet: C25, C30, R7, U10C, U17

Commit message: motherboard tweaks for manufacturing run, i2c card tweaks for manufacturing run, de9 -> stemma adapter idea for the i2c card
Parts:
- C17, C25, C29, C30: LCSC Part # C1853649 -> C49678
- C20: LCSC Part # C2180714 -> C1710
- R4: value 30 -> 33; LCSC Part # C706383 -> C17634
- R5, R6, R7: LCSC Part # C84376 -> C17414
Changed lines of the file:
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@@
 			)
 		)
-		(property "Description" "LCSC #C1853649"
+		(property "Description" "LCSC #C49678"
 			(at 201.93 29.845 0)
 			(effects
@@
 			)
 		)
-		(property "LCSC Part #" "C1853649"
+		(property "LCSC Part #" "C49678"
 			(at 201.93 29.845 0)
 			(effects
@@
 			)
 		)
-		(property "Description" "LCSC #C84376"
+		(property "Description" "LCSC #C17414"
 			(at 158.75 59.69 0)
 			(effects
@@
 			)
 		)
-		(property "LCSC Part #" "C84376 "
+		(property "LCSC Part #" "C17414"
 			(at 158.75 59.69 0)
 			(effects
@@
 			)
 		)
-		(property "Description" "LCSC #C1853649"
+		(property "Description" "LCSC #C49678"
 			(at 66.04 157.48 0)
 			(effects
@@
 			)
 		)
-		(property "LCSC Part #" "C1853649"
+		(property "LCSC Part #" "C49678"
 			(at 66.04 157.48 0)
 			(effects
@@
 			)
 		)
-		(property "Description" "LCSC #C1853649"
+		(property "Description" "LCSC #C49678"
 			(at 144.78 81.915 0)
 			(effects
@@
 			)
 		)
-		(property "LCSC Part #" "C1853649"
+		(property "LCSC Part #" "C49678"
 			(at 144.78 81.915 0)
 			(effects
@@
 			)
 		)
-		(property "Description" "LCSC #C2180714"
+		(property "Description" "LCSC #C1710"
 			(at 214.63 49.53 0)
 			(effects
@@
 			)
 		)
-		(property "LCSC Part #" "C2180714 "
+		(property "LCSC Part #" "C1710"
 			(at 214.63 49.53 0)
 			(effects
@@
 			)
 		)
-		(property "Description" "LCSC #C84376"
+		(property "Description" "LCSC #C17414"
 			(at 201.93 135.89 0)
 			(effects
@@
 			)
 		)
-		(property "LCSC Part #" "C84376 "
+		(property "LCSC Part #" "C17414"
 			(at 201.93 135.89 0)
 			(effects
@@
 			)
 		)
-		(property "Value" "30"
+		(property "Value" "33"
 			(at 254 57.1499 0)
 			(effects
@@
 			)
 		)
-		(property "Description" "LCSC #C706383"
+		(property "Description" "LCSC #C17634"
 			(at 251.46 55.88 0)
 			(effects
@@
 			)
 		)
-		(property "LCSC Part #" "C706383"
+		(property "LCSC Part #" "C17634"
 			(at 251.46 55.88 0)
 			(effects
@@
 			)
 		)
-		(property "Description" "LCSC #C84376"
+		(property "Description" "LCSC #C17414"
 			(at 101.6 116.84 0)
 			(effects
@@
 			)
 		)
-		(property "LCSC Part #" "C84376 "
+		(property "LCSC Part #" "C17414"
 			(at 101.6 116.84 0)
 			(effects
@@
 			)
 		)
-		(property "Description" "LCSC #C1853649"
+		(property "Description" "LCSC #C49678"
 			(at 241.3 105.41 0)
 			(effects
@@
 			)
 		)
-		(property "LCSC Part #" "C1853649"
+		(property "LCSC Part #" "C49678"
 			(at 241.3 105.41 0)
 			(effects
