File: smc.kicad_sch (KiCad schematic)
At the start: 8 parts, among them SW2 SMD_4.6x2.8mm_h2.5mm, U39 ATtiny13A-PU

Commit message: fixes, prep for final production run
Parts:
- added J13: FP Reset Switch, Connector_PinHeader_2.54mm:PinHeader_1x02_P2.54mm_Vertical, symbol Connector_Generic:Conn_01x02
- C59: LCSC Part # (none) -> C1853649
- C62: LCSC Part # (none) -> C1952580
- R27, R28, R29, R30: LCSC Part # (none) -> C84376
- SW2: value SMD_4.6x2.8mm_h2.5mm -> ~; LCSC Part # (none) -> C7470126
- U39: LCSC Part # (none) -> C72124
Connections:
- net GND: now also J13.2 (Pin_2)
- net ~{RESET_BTN}: now also J13.1 (Pin_1)

Commit message: no more SMT for isa_i2c, tweak motherboard multiplex logic, handful of other tweaks
Other:
- moved on the sheet: C59, J13
Changed lines of the file:
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@@
 	(wire
 		(pts
-			(xy 55.88 93.98) (xy 86.36 93.98)
+			(xy 55.88 93.98) (xy 71.12 93.98)
 		)
 		(stroke
@@
 	(wire
 		(pts
-			(xy 55.88 81.28) (xy 86.36 81.28)
+			(xy 55.88 81.28) (xy 71.12 81.28)
 		)
 		(stroke
@@
 	(wire
 		(pts
-			(xy 138.43 67.31) (xy 142.24 67.31)
-		)
-		(stroke
-			(width 0)
-			(type default)
-		)
-	)
-	(wire
-		(pts
-			(xy 86.36 81.28) (xy 86.36 87.63)
+			(xy 138.43 67.31) (xy 147.32 67.31)
+		)
+		(stroke
+			(width 0)
+			(type default)
+		)
+	)
+	(wire
+		(pts
+			(xy 71.12 81.28) (xy 71.12 86.36)
 		)
 		(stroke
@@
 	(wire
 		(pts
-			(xy 153.035 67.31) (xy 153.035 68.58)
+			(xy 158.75 67.31) (xy 158.75 72.39)
 		)
 		(stroke
@@
 	(wire
 		(pts
-			(xy 86.36 93.98) (xy 86.36 90.17)
+			(xy 71.12 93.98) (xy 71.12 88.9)
 		)
 		(stroke
@@
 	(wire
 		(pts
-			(xy 147.32 67.31) (xy 153.035 67.31)
+			(xy 152.4 67.31) (xy 158.75 67.31)
 		)
 		(stroke
@@
 	(symbol
 		(lib_id "power:GND")
-		(at 153.035 68.58 0)
+		(at 158.75 72.39 0)
 		(unit 1)
 		(exclude_from_sim no)
@@
 		(fields_autoplaced yes)
 		(property "Reference" "#PWR0279"
-			(at 153.035 74.93 0)
+			(at 158.75 78.74 0)
 			(effects
 				(font
@@
 		)
 		(property "Value" "GND"
-			(at 153.035 73.66 0)
+			(at 158.75 77.47 0)
 			(effects
 				(font
@@
 		)
 		(property "Footprint" ""
-			(at 153.035 68.58 0)
+			(at 158.75 72.39 0)
 			(effects
 				(font
@@
 		)
 		(property "Datasheet" ""
-			(at 153.035 68.58 0)
+			(at 158.75 72.39 0)
 			(effects
 				(font
@@
 		)
 		(property "Description" ""
-			(at 153.035 68.58 0)
+			(at 158.75 72.39 0)
 			(effects
 				(font
@@
 	(symbol
 		(lib_id "Device:C_Small")
-		(at 144.78 67.31 90)
+		(at 149.86 67.31 90)
 		(unit 1)
 		(exclude_from_sim no)
@@
 		(fields_autoplaced yes)
 		(property "Reference" "C59"
-			(at 144.7863 60.96 90)
+			(at 149.8663 60.96 90)
 			(effects
 				(font
@@
 		)
 		(property "Value" "0.1uF 20% Ceramic"
-			(at 144.7863 63.5 90)
+			(at 149.8663 63.5 90)
 			(effects
 				(font
@@
 		)
 		(property "Footprint" "Capacitor_SMD:C_0805_2012Metric"
-			(at 144.78 67.31 0)
+			(at 149.86 67.31 0)
 			(effects
 				(font
@@
 		)
 		(property "Datasheet" "~"
-			(at 144.78 67.31 0)
+			(at 149.86 67.31 0)
 			(effects
 				(font
@@
 		)
 		(property "Description" "LCSC #C1853649"
-			(at 144.78 67.31 0)
+			(at 149.86 67.31 0)
 			(effects
 				(font
@@
 		)
 		(property "Height" ""
-			(at 144.78 67.31 0)
+			(at 149.86 67.31 0)
 			(effects
 				(font
@@
 		)
 		(property "Manufacturer_Name" ""
-			(at 144.78 67.31 0)
+			(at 149.86 67.31 0)
 			(effects
 				(font
@@
 		)
 		(property "Manufacturer_Part_Number" ""
-			(at 144.78 67.31 0)
+			(at 149.86 67.31 0)
 			(effects
 				(font
@@
 		)
 		(property "Mouser Part Number" ""
-			(at 144.78 67.31 0)
+			(at 149.86 67.31 0)
 			(effects
 				(font
@@
 		)
 		(property "Mouser Price/Stock" ""
-			(at 144.78 67.31 0)
+			(at 149.86 67.31 0)
 			(effects
 				(font
@@
 		)
 		(property "LCSC Part #" "C1853649"
-			(at 144.78 67.31 0)
+			(at 149.86 67.31 0)
 			(effects
 				(font
@@
 	(symbol
 		(lib_id "Connector_Generic:Conn_01x02")
-		(at 91.44 87.63 0)
+		(at 76.2 86.36 0)
 		(unit 1)
 		(exclude_from_sim no)
@@
 		(fields_autoplaced yes)
 		(property "Reference" "J13"
-			(at 93.98 87.6299 0)
+			(at 78.74 86.3599 0)
 			(effects
 				(font
@@
 		)
 		(property "Value" "FP Reset Switch"
-			(at 93.98 90.1699 0)
+			(at 78.74 88.8999 0)
 			(effects
 				(font
@@
 		)
 		(property "Footprint" "Connector_PinHeader_2.54mm:PinHeader_1x02_P2.54mm_Vertical"
-			(at 91.44 87.63 0)
+			(at 76.2 86.36 0)
 			(effects
 				(font
@@
 		)
 		(property "Datasheet" "~"
-			(at 91.44 87.63 0)
+			(at 76.2 86.36 0)
 			(effects
 				(font
@@
 		)
 		(property "Description" "LCSC #C124375"
-			(at 91.44 87.63 0)
+			(at 76.2 86.36 0)
 			(effects
 				(font
@@
 		)
 		(property "Height" ""
-			(at 91.44 87.63 0)
+			(at 76.2 86.36 0)
 			(effects
 				(font
@@
 		)
 		(property "Manufacturer_Name" ""
-			(at 91.44 87.63 0)
+			(at 76.2 86.36 0)
 			(effects
 				(font
@@
 		)
 		(property "Manufacturer_Part_Number" ""
-			(at 91.44 87.63 0)
+			(at 76.2 86.36 0)
 			(effects
 				(font
@@
 		)
 		(property "Mouser Part Number" ""
-			(at 91.44 87.63 0)
+			(at 76.2 86.36 0)
 			(effects
 				(font
@@
 		)
 		(property "Mouser Price/Stock" ""
-			(at 91.44 87.63 0)
+			(at 76.2 86.36 0)
 			(effects
 				(font
@@
 		)
 		(property "LCSC Part #" "C124375"
-			(at 91.44 87.63 0)
-			(effects
-				(font
+			(at 76.2 86.36 0)
+			(effects
+				(font

Commit message: motherboard tweaks for manufacturing run, i2c card tweaks for manufacturing run, de9 -> stemma adapter idea for the i2c card
Parts:
- C59: LCSC Part # C1853649 -> C49678
- C62: LCSC Part # C1952580 -> C15850
- R27, R28, R29, R30: LCSC Part # C84376 -> C17414
Changed lines of the file:
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@@
 			)
 		)
-		(property "Description" "LCSC #C1853649"
+		(property "Description" "LCSC #C49678"
 			(at 149.86 67.31 0)
 			(effects
@@
 			)
 		)
-		(property "LCSC Part #" "C1853649"
+		(property "LCSC Part #" "C49678"
 			(at 149.86 67.31 0)
 			(effects
@@
 			)
 		)
-		(property "Description" "LCSC #C84376"
+		(property "Description" "LCSC #C17414"
 			(at 176.53 137.16 0)
 			(effects
@@
 			)
 		)
-		(property "LCSC Part #" "C84376 "
+		(property "LCSC Part #" "C17414"
 			(at 176.53 137.16 0)
 			(effects
@@
 			)
 		)
-		(property "Description" "LCSC #C84376"
+		(property "Description" "LCSC #C17414"
 			(at 154.94 135.89 0)
 			(effects
@@
 			)
 		)
-		(property "LCSC Part #" "C84376 "
+		(property "LCSC Part #" "C17414"
 			(at 154.94 135.89 0)
 			(effects
@@
 			)
 		)
-		(property "Description" "LCSC #C84376"
+		(property "Description" "LCSC #C17414"
 			(at 205.74 130.81 0)
 			(effects
@@
 			)
 		)
-		(property "LCSC Part #" "C84376 "
+		(property "LCSC Part #" "C17414"
 			(at 205.74 130.81 0)
 			(effects
@@
 			)
 		)
-		(property "Description" "LCSC #C84376"
+		(property "Description" "LCSC #C17414"
 			(at 55.88 71.12 0)
 			(effects
@@
 			)
 		)
-		(property "LCSC Part #" "C84376 "
+		(property "LCSC Part #" "C17414"
 			(at 55.88 71.12 0)
 			(effects
@@
 			)
 		)
-		(property "Description" "LCSC #C1952580"
+		(property "Description" "LCSC #C15850"
 			(at 43.18 87.63 0)
 			(effects
@@
 			)
 		)
-		(property "LCSC Part #" "C1952580"
+		(property "LCSC Part #" "C15850"
 			(at 43.18 87.63 0)
 			(effects
