File: isa_i2c/isa_i2c.kicad_pcb (KiCad board)
At the start: 4 copper layers, 99.9 x 87.1 mm, 24 parts, among them J1 Conn_01x02, J2 Conn_01x03, J3 Conn_01x03, J4 Conn_01x03, J5 Conn_01x03, J6 Conn_01x03, J7 Conn_01x03, J8 Bus_ISA_8bit, SW1 SW_DIP_x08, U1 PCF8584, U2 74HC245, U6 74AHC1GU04, U7 74HCT688

Commit message: no more SMT for isa_i2c, tweak motherboard multiplex logic, handful of other tweaks
Parts:
- removed J1: Conn_01x02, Connector_PinHeader_2.54mm:PinHeader_1x02_P2.54mm_Vertical
- removed J2, J3, J4, J5, J6, J7: Conn_01x03, Connector_PinHeader_2.54mm:PinHeader_1x03_P2.54mm_Vertical
- removed U6: 74AHC1GU04, Package_TO_SOT_SMD:SOT-23-5
- added C3: 10 uF, Capacitor_THT:C_Disc_D3.0mm_W1.6mm_P2.50mm, F.Cu at (150.5, 75.6)
- added C4: 0.1 uF, Capacitor_THT:C_Disc_D3.0mm_W1.6mm_P2.50mm, F.Cu at (150.5, 73.0)
- added G***: LOGO, LOGO, F.Cu at (137.2, 51.4)
- added J10: Conn_01x04, Connector_JST:JST_PH_S4B-PH-K_1x04_P2.00mm_Horizontal, F.Cu at (101.0, 59.7)
- added J12: Conn_01x04, Connector_JST:JST_PH_S4B-PH-K_1x04_P2.00mm_Horizontal, F.Cu at (187.3, 99.7)
- added J13: Conn_01x04, Connector_JST:JST_PH_S4B-PH-K_1x04_P2.00mm_Horizontal, F.Cu at (187.3, 88.3)
- added J14: Conn_01x04, Connector_JST:JST_PH_S4B-PH-K_1x04_P2.00mm_Horizontal, F.Cu at (101.0, 71.1)
- added J15: Conn_01x04, Connector_JST:JST_PH_S4B-PH-K_1x04_P2.00mm_Horizontal, F.Cu at (187.3, 65.4)
- added J16: Conn_01x04, Connector_JST:JST_PH_S4B-PH-K_1x04_P2.00mm_Horizontal, F.Cu at (187.3, 76.8)
- added Q1: BS170, Package_TO_SOT_THT:TO-92_Inline, F.Cu at (189.2, 115.6)
- added Q2: BS250, Package_TO_SOT_THT:TO-92_Inline, F.Cu at (184.2, 118.1)
- added U4: LD1117V33, Package_TO_SOT_THT:TO-220-3_Horizontal_TabDown, F.Cu at (147.3, 78.1)
- C1, C2, C6, C7: footprint Capacitor_SMD:C_0603_1608Metric -> Capacitor_THT:C_Disc_D3.0mm_W1.6mm_P2.50mm
- R1, R2: value 2.2k -> 2.2k 1/8W; footprint Resistor_SMD:R_0603_1608Metric -> Resistor_THT:R_Axial_DIN0204_L3.6mm_D1.6mm_P5.08mm_Horizontal
- U1: value PCF8584 -> PCA9564N; footprint Package_SO:SO-20_12.8x7.5mm_P1.27mm -> Package_DIP:DIP-20_W7.62mm_Socket
- moved R1 30.1 mm to (181.0, 85.1), turned to -90 degrees
- moved R2 26.5 mm to (181.0, 81.9), turned to 90 degrees
- moved C1 23.6 mm to (153.0, 94.0), turned to 180 degrees
- moved U1 15.7 mm to (156.2, 101.6), turned to 90 degrees
- moved C6 7.03 mm to (179.7, 116.2), turned to 180 degrees
- moved RN2 2.54 mm to (153.7, 105.4)
- moved C2 0.14 mm to (148.0, 108.6)
Connections:
- C1 pad 1: +5V -> +3.3V
- U1 pad 1: /CLK -> /D0
- U1 pad 11: /D3 -> /~{IOW}
- U1 pad 12: /D4 -> /~{IOR}
- U1 pad 13: /D5 -> /~{CS}
- U1 pad 14: /D6 -> /BA00
- U1 pad 15: /D7 -> /BA01
- U1 pad 16: /~{IOR} -> unconnected-(U1-~{INT}-Pad16)
- U1 pad 17: /~{CS} -> /~{RESET}
- U1 pad 18: /~{IOW} -> /SCL
- U1 pad 19: /~{RESET} -> /SDA
- U1 pad 2: /SDA -> /D1
- U1 pad 20: +5V -> +3.3V
- U1 pad 3: /SCL -> /D2
- U1 pad 4: +5V -> /D3
- U1 pad 5: unconnected-(U1-~{INT}-Pad5) -> /D4
- U1 pad 6: /BA00 -> /D5
- U1 pad 7: /D0 -> /D6
- U1 pad 8: /D1 -> /D7
- U1 pad 9: /D2 -> unconnected-(U1-DNU-Pad9)
Routing:
- net /SCL: track 53.8 -> 178.8 mm
- net /SDA: track 56.4 -> 180.1 mm
- net /BA01: track 0.00 -> 116.5 mm
- net /CLK: track 79.0 -> 0.00 mm, vias 1 -> 0
- net +3.3V: track 0.00 -> 26.9 mm
- net /D5: track 24.0 -> 6.98 mm
- net /D6: track 24.0 -> 6.98 mm
- net /D3: track 24.0 -> 6.98 mm
- net /D4: track 24.0 -> 6.98 mm
- net /D7: track 24.0 -> 6.98 mm
- net +5V: track 26.9 -> 11.8 mm, vias 7 -> 2
- net /D0: track 21.8 -> 6.98 mm
- net /D1: track 19.5 -> 6.98 mm
- net /~{IOR}: track 91.5 -> 79.2 mm, vias 1 -> 0
- net /~{IOW}: track 88.2 -> 75.9 mm, vias 1 -> 0
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Other:
- board text added: "PCA9564"
- board text added: "REV A2"
- board text added: "at +5V"
- board text removed: "+5V"
- board text removed: "GND"
- board text removed: "I2C CONNECTIONS"
- board text removed: "PCF8584"
- board text removed: "REV A1"
- board text removed: "SCL"
- board text removed: "SDA"

Commit message: i2c card tweaks, manual tweaks
Parts:
- removed C3: 10 uF, Capacitor_THT:C_Disc_D3.0mm_W1.6mm_P2.50mm
- removed C4: 0.1 uF, Capacitor_THT:C_Disc_D3.0mm_W1.6mm_P2.50mm
- removed U1: PCA9564N, Package_DIP:DIP-20_W7.62mm_Socket
- removed U4: LD1117V33, Package_TO_SOT_THT:TO-220-3_Horizontal_TabDown
- added U3: PCF8584, Package_DIP:DIP-20_W7.62mm_Socket, F.Cu at (156.2, 68.6)
- moved C1 29.0 mm to (167.0, 68.6), turned to 0 degrees
- moved R1 19.9 mm to (177.8, 65.4)
- moved R2 18.7 mm to (177.8, 63.5)
- turned C7 to 90 degrees
Connections:
- C1 pad 1: +3.3V -> +5V
Routing:
- net /BA01: track 116.5 -> 0.00 mm
- net /CLK: track 0.00 -> 90.0 mm
- net /~{CS}: track 85.5 -> 124.7 mm, vias 0 -> 2
- net /~{IOW}: track 75.9 -> 111.6 mm
- net /D7: track 6.98 -> 37.0 mm
- net /~{IOR}: track 79.2 -> 107.3 mm
- net +3.3V: track 26.9 -> 0.00 mm
- net /D0: track 6.98 -> 32.2 mm
- net /D6: track 6.98 -> 31.4 mm
- net /SDA: track 180.1 -> 156.1 mm
- net /D1: track 6.98 -> 30.9 mm
- net /D2: track 6.98 -> 29.7 mm
- net /SCL: track 178.8 -> 157.5 mm, vias 0 -> 1
- net /D5: track 6.98 -> 26.8 mm
- net /~{RESET}: track 55.1 -> 71.7 mm
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Other:
- board text added: "PCF8584"
- board text removed: "PCA9564"

Commit message: simplify m88 logic further, reduce ICs, reorient the POST display, use an oscillator for 14.31818 MHz, update isa-i2c bridge BOM
Parts:
- added C3: 10-100uF 16V Electrolytic, Capacitor_THT:CP_Radial_D5.0mm_P2.00mm, F.Cu at (100.3, 121.3)
Routing:
- net +5V: track 11.8 -> 16.2 mm, vias 2 -> 1
- net /BA00: track 110.2 -> 107.5 mm
- net /~{CS}: track 124.7 -> 124.2 mm
- net GND: vias 58 -> 65
Other:
- board text added: "2.2k"

Commit message: isa_i2c: current-limit the reset line inverter
Parts:
- added R3: 680 1/8W, Resistor_THT:R_Axial_DIN0204_L3.6mm_D1.6mm_P5.08mm_Horizontal, F.Cu at (184.2, 109.9)
Connections:
- Q2 pad 3: +5V -> Net-(Q2-S)
Routing:
- net Net-(Q2-S): track 0.00 -> 5.71 mm
Other:
- board text added: "680"

Commit message: motherboard tweaks for manufacturing run, i2c card tweaks for manufacturing run, de9 -> stemma adapter idea for the i2c card
Parts:
- removed C6: 0.1 uF, Capacitor_THT:C_Disc_D3.0mm_W1.6mm_P2.50mm
- removed H1: MountingHole, MountingHole:MountingHole_3.2mm_M3
- removed H2: MountingHole_Pad, MountingHole:MountingHole_3.2mm_M3_Pad_Via
- removed J12, J13, J14, J15, J16: Conn_01x04, Connector_JST:JST_PH_S4B-PH-K_1x04_P2.00mm_Horizontal
- removed Q1: BS170, Package_TO_SOT_THT:TO-92_Inline
- removed Q2: BS250, Package_TO_SOT_THT:TO-92_Inline
- removed R3: 680 1/8W, Resistor_THT:R_Axial_DIN0204_L3.6mm_D1.6mm_P5.08mm_Horizontal
- added C4: 0.1 uF, Capacitor_SMD:C_0603_1608Metric, F.Cu at (182.1, 111.1)
- added J1: DE9_Receptacle, SamacSys_Parts:L77SDE09SA4CH4F, F.Cu at (188.0, 77.6)
- added R4: 47 1/8W, Resistor_THT:R_Axial_DIN0204_L3.6mm_D1.6mm_P5.08mm_Horizontal, F.Cu at (153.0, 70.5)
- added R5: 47 1/8W, Resistor_THT:R_Axial_DIN0204_L3.6mm_D1.6mm_P5.08mm_Horizontal, F.Cu at (156.8, 67.9)
- added U1: 74AHC1G04, Package_TO_SOT_SMD:SOT-23-5, F.Cu at (186.1, 112.4)
- U3: footprint Package_DIP:DIP-20_W7.62mm_Socket -> Package_SO:SOIC-20W_7.5x12.8mm_P1.27mm
- moved G*** 45.3 mm to (99.7, 76.8)
- moved R1 29.3 mm to (149.9, 74.3), turned to 180 degrees
- moved R2 28.8 mm to (149.9, 70.5), turned to 180 degrees
- moved U3 15.7 mm to (160.0, 83.8)
- moved C1 8.28 mm to (167.6, 76.8), turned to 90 degrees
- moved G*** 8.13 mm to (104.8, 59.7)
- moved J10 6.48 mm to (102.2, 66.0)
- moved RN2 1.27 mm to (153.7, 104.1)
Connections:
- R1 pad 1: /SCL -> /PCF_SCL
- R2 pad 1: /SDA -> /PCF_SDA
- U3 pad 2: /SDA -> /PCF_SDA
- U3 pad 3: /SCL -> /PCF_SCL
Routing:
- net +5V: track 16.2 -> 352.1 mm, vias 1 -> 6
- net /SDA: track 156.1 -> 108.4 mm
- net /SCL: track 157.5 -> 114.1 mm, vias 1 -> 0
- net /PCF_SCL: track 0.00 -> 24.2 mm
- net /~{CS}: track 124.0 -> 100.3 mm, vias 2 -> 0
- net /~{RESET}: track 72.2 -> 53.0 mm
- net /~{IOW}: track 111.6 -> 96.2 mm, vias 0 -> 1
- net /PCF_SDA: track 0.00 -> 13.6 mm
- net /CLK: track 90.0 -> 79.6 mm, vias 0 -> 1
- net /~{IOR}: track 107.3 -> 98.2 mm, vias 0 -> 1
- net /D3: track 17.1 -> 24.4 mm
- net Net-(Q2-S): track 5.71 -> 0.00 mm
- net /BA00: track 107.1 -> 102.0 mm
- net /D7: track 37.0 -> 33.0 mm
- net /D4: track 21.7 -> 24.4 mm
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- removed copper zone on In1.Cu, net +5V
- removed copper zone on In2.Cu, net GND
Other:
- board size 99.9 x 87.1 mm -> 99.7 x 78.3 mm
- copper layers 4 -> 2
- board text added: "1,2,3,4 5,9 6 7 8"
- board text added: "47"
- board text added: "DB9 PINOUT"
- board text added: "GND NC SDA +5V SCL"
- board text added: "TOP OF BRACKET"
- board text removed: "680"
