File: isa_i2c/isa_i2c.kicad_sch (KiCad schematic)
At the start: 23 parts, among them J1 Conn_01x02, J2 Conn_01x03, J3 Conn_01x03, J4 Conn_01x03, J5 Conn_01x03, J6 Conn_01x03, J7 Conn_01x03, J8 Bus_ISA_8bit, SW1 SW_DIP_x08, U1 PCF8584, U2 74HC245, U6 74AHC1GU04, U7 74HCT688

Commit message: fix part selection for i2c card
Parts:
- U6: LCSC Part # C460495 -> C7465
Changed lines of the file:
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@@
 			)
 		)
-		(property "LCSC Part #" "C460495"
+		(property "LCSC Part #" "C7465"
 			(at 251.46 44.45 0)
 			(effects

Commit message: no more SMT for isa_i2c, tweak motherboard multiplex logic, handful of other tweaks
Parts:
- removed J1: Conn_01x02, Connector_PinHeader_2.54mm:PinHeader_1x02_P2.54mm_Vertical, symbol Connector_Generic:Conn_01x02
- removed J2, J3, J4, J5, J6, J7: Conn_01x03, Connector_PinHeader_2.54mm:PinHeader_1x03_P2.54mm_Vertical, symbol Connector_Generic:Conn_01x03
- removed U1: PCF8584, Package_SO:SO-20_12.8x7.5mm_P1.27mm, symbol Interface_Expansion:PCF8584
- removed U6: 74AHC1GU04, Package_TO_SOT_SMD:SOT-23-5, symbol 74xGxx:74AHC1GU04
- added C3: 10 uF, Capacitor_THT:C_Disc_D3.0mm_W1.6mm_P2.50mm, symbol Device:C_Small
- added C4: 0.1 uF, Capacitor_THT:C_Disc_D3.0mm_W1.6mm_P2.50mm, symbol Device:C_Small
- added J10, J12, J13, J14, J15, J16: Conn_01x04, Connector_JST:JST_PH_S4B-PH-K_1x04_P2.00mm_Horizontal, symbol Connector_Generic:Conn_01x04
- added Q1: BS170, Package_TO_SOT_THT:TO-92_Inline, symbol Transistor_FET:BS170
- added Q2: BS250, Package_TO_SOT_THT:TO-92_Inline, symbol Transistor_FET:BS250
- added U1: PCA9564N, Package_DIP:DIP-20_W7.62mm_Socket, symbol Custom:PCA9564
- added U4: LD1117V33, Package_TO_SOT_THT:TO-220-3_Horizontal_TabDown, symbol SamacSys_Parts:LD1117V33
- C1, C2, C6, C7: footprint Capacitor_SMD:C_0603_1608Metric -> Capacitor_THT:C_Disc_D3.0mm_W1.6mm_P2.50mm; Manufacturer_Name (none) -> KYOCERA AVX; Manufacturer_Part_Number (none) -> 0603ZC104K4T2A; Mouser Part Number (none) -> 581-0603ZC104K4T2A
- R1, R2: value 2.2k -> 2.2k 1/8W; footprint Resistor_SMD:R_0603_1608Metric -> Resistor_THT:R_Axial_DIN0204_L3.6mm_D1.6mm_P5.08mm_Horizontal
Connections:
- net +5V: now also C4.1, J10.3 (Pin_3), J12.3 (Pin_3), J13.3 (Pin_3), J14.3 (Pin_3), J15.3 (Pin_3), J16.3 (Pin_3), Q2.3 (S), U4.3 (VIN); no longer C1.1
- net BA00: now also U1.14 (A0)
- net BA01: now also U1.15 (A1)
- net D0: now also U1.1 (D0)
- net D1: now also U1.2 (D1)
- net D2: now also U1.3 (D2)
- net D3: now also U1.4 (D3)
- net D4: now also U1.5 (D4)
- net D5: now also U1.6 (D5)
- net D6: now also U1.7 (D6)
- net D7: now also U1.8 (D7)
- net GND: now also C3.2, C4.2, J10.4 (Pin_4), J12.4 (Pin_4), J13.4 (Pin_4), J14.4 (Pin_4), J15.4 (Pin_4), J16.4 (Pin_4), Q1.3 (S), U1.10 (VSS), U4.1 (ADJ/GND)
- net RESET: now also Q1.2 (G), Q2.2 (G)
- net SCL: now also J10.1 (Pin_1), J12.1 (Pin_1), J13.1 (Pin_1), J14.1 (Pin_1), J15.1 (Pin_1), J16.1 (Pin_1), U1.18 (SCL)
- net SDA: now also J10.2 (Pin_2), J12.2 (Pin_2), J13.2 (Pin_2), J14.2 (Pin_2), J15.2 (Pin_2), J16.2 (Pin_2), U1.19 (SDA)
- net ~{CS}: now also U1.13 (~{CE})
- net ~{IOR}: now also U1.12 (~{RD})
- net ~{IOW}: now also U1.11 (~{WR})
- net ~{RESET}: now also Q1.1 (D), Q2.1 (D), U1.17 (~{RESET})
- net CLK: no longer names the net of J8.20 (CLK)
- new net +3.3V: C1.1, C3.1, U1.20 (VDD), U4.2 (VOUT)
Other:
- note added: "Active-high RESET to Active-low RESET CMOS Inverter, through-hole, single gate"
- note added: "Horizontal STEMMA QT x6"
- note added: "NB: using 10 address lines for I/O, ignoring higher bits"
- note removed: "NB: ISA bus is specified to use 10 address lines for I/O"
- moved on the sheet: C1, C2, C6, C7, R1, R2, RN1, RN2, SW1, U2, U7

Commit message: i2c card tweaks, manual tweaks
Parts:
- removed C3: 10 uF, Capacitor_THT:C_Disc_D3.0mm_W1.6mm_P2.50mm, symbol Device:C_Small
- removed C4: 0.1 uF, Capacitor_THT:C_Disc_D3.0mm_W1.6mm_P2.50mm, symbol Device:C_Small
- removed U1: PCA9564N, Package_DIP:DIP-20_W7.62mm_Socket, symbol Custom:PCA9564
- removed U4: LD1117V33, Package_TO_SOT_THT:TO-220-3_Horizontal_TabDown, symbol SamacSys_Parts:LD1117V33
- added U3: PCF8584, Package_DIP:DIP-20_W7.62mm_Socket, symbol Interface_Expansion:PCF8584
- C1, C2, C6, C7: LCSC Part # C14663 -> C1619948; Manufacturer_Name KYOCERA AVX -> KEMET; Manufacturer_Part_Number 0603ZC104K4T2A -> C320C104K1R5TA; Mouser Part Number 581-0603ZC104K4T2A -> (none)
- J10, J12, J13, J14, J15, J16: LCSC Part # (none) -> C157926; Manufacturer_Name (none) -> JST; Manufacturer_Part_Number (none) -> S4B-PH-K-S(LF)(SN)
- J8: now left out of the parts list
- Q1: LCSC Part # (none) -> C111691; Manufacturer_Name (none) -> onsemi; Manufacturer_Part_Number (none) -> BS170
- Q2: LCSC Part # (none) -> C151450; Manufacturer_Name (none) -> Diodes Incorporated; Manufacturer_Part_Number (none) -> BS250P
- R1, R2: LCSC Part # C4190 -> C274498; Manufacturer_Name (none) -> Futaba Elec; Manufacturer_Part_Number (none) -> RNS14F2201A520NH
Connections:
- net +3.3V is gone; now on net +5V: C1.1
- net +5V: now also U3.20 (VDD), U3.4 (~{IACK})
- net BA00: now also U3.6 (A0)
- net D0: now also U3.7 (D0)
- net D1: now also U3.8 (D1)
- net D2: now also U3.9 (D2)
- net D3: now also U3.11 (D3)
- net D4: now also U3.12 (D4)
- net D5: now also U3.13 (D5)
- net D6: now also U3.14 (D6)
- net D7: now also U3.15 (D7)
- net GND: now also U3.10 (VSS)
- net SCL: now also U3.3 (SCL)
- net SDA: now also U3.2 (SDA)
- net ~{CS}: now also U3.17 (~{CS})
- net ~{IOR}: now also U3.16 (~{RD})
- net ~{IOW}: now also U3.18 (~{WR})
- net ~{RESET}: now also U3.19 (~{RST})
- net CLK: now reaches J8.20 (CLK)
- net CLK: now also U3.1 (CLK)
Other:
- moved on the sheet: C1, C6, Q1, Q2

Commit message: simplify m88 logic further, reduce ICs, reorient the POST display, use an oscillator for 14.31818 MHz, update isa-i2c bridge BOM
Parts:
- added C3: 10-100uF 16V Electrolytic, Capacitor_THT:CP_Radial_D5.0mm_P2.00mm, symbol Device:C_Polarized_US
- C1, C2, C6, C7: Manufacturer_Name KEMET -> Vishay / BC Components; Manufacturer_Part_Number C320C104K1R5TA -> K104M15X7RF53K2; Mouser Part Number (none) -> 594-K104M15X7RF53K2
- J10, J12, J13, J14, J15, J16: Mouser Part Number (none) -> 306-S4BPHKSLFSN
- Q1: Mouser Part Number (none) -> 512-BS170
- Q2: Mouser Part Number (none) -> 522-BS250P
- R1, R2: Mouser Part Number (none) -> 279-LR0204F2K2
- RN1, RN2: Mouser Part Number (none) -> 652-4609X-1LF-10K
- SW1: Mouser Part Number (none) -> 710-418117270908
- U2, U3, U7: Mouser Part Number (none) -> 571-1-2199298-6
Connections:
- net +5V: now also C3.1
- net GND: now also C3.2

Commit message: isa_i2c: current-limit the reset line inverter
Parts:
- added R3: 680 1/8W, Resistor_THT:R_Axial_DIN0204_L3.6mm_D1.6mm_P5.08mm_Horizontal, symbol Device:R_Small_US
Connections:
- net +5V: now also R3.2; no longer Q2.3 (S)
- new net: Q2.3 (S), R3.1
Changed lines of the file:
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@@
+	(wire
+		(pts
+			(xy 264.16 31.75) (xy 264.16 34.29)
+		)
+		(stroke
+			(width 0)
+			(type default)
+		)
+	)
 	(wire
 		(pts
@@
 	(wire
 		(pts
-			(xy 264.16 24.13) (xy 264.16 34.29)
+			(xy 264.16 24.13) (xy 264.16 26.67)
 		)
 		(stroke
@@
 					(unit 1)
 				)
+			)
+		)
+	)
+	(symbol
+		(lib_id "Device:R_Small_US")
+		(at 264.16 29.21 0)
+		(mirror x)
+		(unit 1)
+		(exclude_from_sim no)
+		(in_bom yes)
+		(on_board yes)
+		(dnp no)
+		(property "Reference" "R3"
+			(at 261.62 27.9399 0)
+			(effects
+				(font
+					(size 1.27 1.27)
+				)
+				(justify right)
+			)
+		)
+		(property "Value" "680 1/8W"
+			(at 261.62 30.4799 0)
+			(effects
+				(font
+					(size 1.27 1.27)
+				)
+				(justify right)
+			)
+		)
+		(property "Footprint" "Resistor_THT:R_Axial_DIN0204_L3.6mm_D1.6mm_P5.08mm_Horizontal"
+			(at 264.16 29.21 0)
+			(effects
+				(font
+					(size 1.27 1.27)
+				)
+				(hide yes)
+			)
+		)
+		(property "Datasheet" "~"
+			(at 264.16 29.21 0)
+			(effects
+				(font
+					(size 1.27 1.27)
+				)
+				(hide yes)
+			)
+		)
+		(property "Description" "Limit to <8mA draw"
+			(at 251.968 32.766 0)
+			(effects
+				(font
+					(size 1.27 1.27)
+				)
+			)
+		)
+		(property "LCSC Part #" "C274498"
+			(at 264.16 29.21 0)
+			(effects
+				(font
+					(size 1.27 1.27)
+				)
+				(hide yes)
+			)
+		)
+		(property "Height" ""
+			(at 264.16 29.21 0)
+			(effects
+				(font
+					(size 1.27 1.27)
+				)
+				(hide yes)
+			)
+		)
+		(property "Manufacturer_Name" "Futaba Elec"
+			(at 264.16 29.21 0)
+			(effects
+				(font
+					(size 1.27 1.27)
+				)
+				(hide yes)
+			)
+		)
+		(property "Manufacturer_Part_Number" "RNS14F2201A520NH"
+			(at 264.16 29.21 0)
+			(effects
+				(font
+					(size 1.27 1.27)
+				)
+				(hide yes)
+			)
+		)
+		(property "Mouser Part Number" "279-LR0204F2K2"
+			(at 264.16 29.21 0)
+			(effects
+				(font
+					(size 1.27 1.27)
+				)
+				(hide yes)
+			)
+		)
+		(property "Mouser Price/Stock" ""
+			(at 264.16 29.21 0)
+			(effects
+				(font
+					(size 1.27 1.27)
+				)
+				(hide yes)
+			)
+		)
+		(pin "2"
+		)
+		(pin "1"
+		)
+		(instances
+			(project "isa_i2c"
+				(path "/65b312ef-48c6-4b8d-9854-6e1afa7c3490"
+					(reference "R3")
+					(unit 1)
+				)

Commit message: motherboard tweaks for manufacturing run, i2c card tweaks for manufacturing run, de9 -> stemma adapter idea for the i2c card
Parts:
- removed C6: 0.1 uF, Capacitor_THT:C_Disc_D3.0mm_W1.6mm_P2.50mm, symbol Device:C_Small
- removed H1: MountingHole, MountingHole:MountingHole_3.2mm_M3, symbol Mechanical:MountingHole
- removed H2: MountingHole_Pad, MountingHole:MountingHole_3.2mm_M3_Pad_Via, symbol Mechanical:MountingHole_Pad
- removed J12, J13, J14, J15, J16: Conn_01x04, Connector_JST:JST_PH_S4B-PH-K_1x04_P2.00mm_Horizontal, symbol Connector_Generic:Conn_01x04
- removed Q1: BS170, Package_TO_SOT_THT:TO-92_Inline, symbol Transistor_FET:BS170
- removed Q2: BS250, Package_TO_SOT_THT:TO-92_Inline, symbol Transistor_FET:BS250
- removed R3: 680 1/8W, Resistor_THT:R_Axial_DIN0204_L3.6mm_D1.6mm_P5.08mm_Horizontal, symbol Device:R_Small_US
- added C4: 0.1 uF, Capacitor_SMD:C_0603_1608Metric, symbol Device:C_Small
- added J1: DE9_Receptacle, SamacSys_Parts:L77SDE09SA4CH4F, symbol Connector:DE9_Receptacle_MountingHoles
- added R4, R5: 47 1/8W, Resistor_THT:R_Axial_DIN0204_L3.6mm_D1.6mm_P5.08mm_Horizontal, symbol Device:R_Small_US
- added U1: 74AHC1G04, Package_TO_SOT_SMD:SOT-23-5, symbol 74xGxx:74AHC1G04
- RN1, RN2: Manufacturer_Name (none) -> Bourns; Manufacturer_Part_Number (none) -> 4609X-101-103LF
- SW1: Manufacturer_Name (none) -> Wurth Elektronik; Manufacturer_Part_Number (none) -> 418117270908
- U2: LCSC Part # C2899 -> (none); Manufacturer_Name (none) -> Texas Instruments; Manufacturer_Part_Number (none) -> SN74HC245N; Mouser Part Number 571-1-2199298-6 -> 595-SN74HC245N
- U3: footprint Package_DIP:DIP-20_W7.62mm_Socket -> Package_SO:SOIC-20W_7.5x12.8mm_P1.27mm; LCSC Part # C72118 -> C2678126; Manufacturer_Name (none) -> NXP Semiconductors; Manufacturer_Part_Number (none) -> PCF8584T/2,518; Mouser Part Number 571-1-2199298-6 -> 771-PCF8584TD-T
- U7: LCSC Part # C1523711 -> (none); Manufacturer_Name (none) -> Texas Instruments; Manufacturer_Part_Number (none) -> CD74HCT688E; Mouser Part Number 571-1-2199298-6 -> 595-CD74HCT688E
Connections:
- net +5V: now also C4.1, J1.7, U1.5 (VCC)
- net GND: now also C4.2, J1.0 (PAD), J1.1, J1.2, J1.3, J1.4, U1.3 (GND)
- net RESET: now also U1.2
- net SCL: now also J1.8, R5.2; no longer R1.1, U3.3 (SCL)
- net SDA: now also J1.6, R4.2; no longer R2.1, U3.2 (SDA)
- net ~{RESET}: now also U1.4
- new net PCF_SCL: R1.1, R5.1, U3.3 (SCL)
- new net PCF_SDA: R2.1, R4.1, U3.2 (SDA)
- no-connect marks 36 -> 38
Other:
- note added: "DE-9 Socket For external connection & bracket mounting to a Keystone 9200-1 bracket"
- note added: "Horizontal STEMMA (for devices inside the PC case)"
- note removed: "Horizontal STEMMA QT x6"
- moved on the sheet: J10
